File: KiCad/_autosave-AstroWeather.kicad_pcb (KiCad board)
At the start: 2 copper layers, 243 x 28 mm, 52 parts, among them Q501 IRLML2502, Q502 Si2365EDS, Q503 Si2365EDS, Q504 Si2365EDS, Q505 Si2365EDS, Q506 Si2365EDS, Q507 IRLML2502, U301 STM32G0B1KCTx, U501 SCT2024, U502 MCP6006T-E/OT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

Commit message: KiCad work
Parts:
- removed U301: STM32G0B1KCTx, Package_QFP:LQFP-32_7x7mm_P0.8mm
- added C302: 4u7, Capacitor_SMD:C_0603_1608Metric, F.Cu at (97.2, 23.0)
- added C303: 10p, Capacitor_SMD:C_0603_1608Metric, F.Cu at (97.2, 25.5)
- added C304: 10p, Capacitor_SMD:C_0603_1608Metric, F.Cu at (97.2, 28.0)
- added C305: 100n, Capacitor_SMD:C_0603_1608Metric, F.Cu at (97.2, 30.5)
- added U302: AT24CS01-STUM, Package_TO_SOT_SMD:SOT-23-5, F.Cu at (86.4, 35.5)
- added U303: STM32G0B1CETx, Package_QFP:LQFP-48_7x7mm_P0.5mm, B.Cu at (65.8, 66.2)
