File: KiCad/AstroWeather.kicad_sch (KiCad schematic)
At the start: 0 parts

Commit message: KiCad work
Parts:
- added J101: USB_C_Receptacle_USB2.0_14P, symbol Connector:USB_C_Receptacle_USB2.0_14P
- added J102: SWD, symbol Connector_Generic_MountingPin:Conn_01x06_MountingPin
- added J103: I2C, symbol Connector_Generic_MountingPin:Conn_01x04_MountingPin
Connections:
- new net: J101.A1 (GND), J101.A12 (GND), J101.B1 (GND), J101.B12 (GND)
- new net: J101.A4 (VBUS), J101.A9 (VBUS), J101.B4 (VBUS), J101.B9 (VBUS)
Other:
- added sheet Power Supply (PowerSupply.kicad_sch)
- sheet Display ports: added LED_BRIGHTNESS, LOW_POWER_ENABLE; removed none
- sheet Host Controller ports: added +3.3V, DIS1_EN, DIS2_EN, DIS3_EN, DIS4_EN, DIS5_EN, GND, I2C_SCL, I2C_SDA, LOW_POWER_ENABLE, NRST, SCT_CLK, SCT_SDI, ST67_MISO, ST67_MOSI, ST67_RX, ST67_SCK, ST67_TX, SWCLK, SWDIO, UCPD_CC1, UCPD_CC2, USB+, USB-, ~{SCT_EN}, ~{SCT_LA}; removed none

Commit message: KiCad work
Parts:
- removed J102: SWD, symbol Connector_Generic_MountingPin:Conn_01x06_MountingPin
- removed J103: I2C, symbol Connector_Generic_MountingPin:Conn_01x04_MountingPin
- added D101, D102: D_TVS, symbol Device:D_TVS
- added J102, J103: Conn_01x10, symbol Connector_Generic:Conn_01x10
- added J104: AUX_POWER, symbol Connector_Generic:Conn_01x02
- added J105: SWD, symbol Connector_Generic:Conn_01x06
- added J106: I2C, symbol Connector_Generic:Conn_01x04
Connections:
- net Host Controller/NRST: now also J105.5 (Pin_5)
- net Host Controller/SWCLK: now also J105.2 (Pin_2)
- net Host Controller/SWDIO: now also J105.4 (Pin_4)
- net Host Controller/UCPD_CC1: now also J101.A5 (CC1)
- net Host Controller/UCPD_CC2: now also J101.B5 (CC2)
- net Host Controller/USB+: now also J101.A6 (D+), J101.B6 (D+), D102.2 (A2)
- net Host Controller/USB-: now also J101.A7 (D-), J101.B7 (D-), D101.2 (A2)
- net GND: now reaches J101.A1 (GND), J101.A12 (GND), J101.B1 (GND), J101.B12 (GND)
- net GND: now also D101.1 (A1), D102.1 (A1), J105.3 (Pin_3)
- net VBUS: now reaches J101.A4 (VBUS), J101.A9 (VBUS), J101.B4 (VBUS), J101.B9 (VBUS)
- new net +3.3V: J105.1 (Pin_1)
- no-connect marks 0 -> 2
Other:
- sheet Display ports: added GND, VLED, ~{SCT_EN}, ~{SCT_LA}; removed !SCT_EN, !SCT_LA, Gnd, Vdd
- sheet ST67W611M1 ports: added GND, ST67_CLK, ST67_CS, ST67_MISO, ST67_MOSI, ST67_RDY, ST67_RX, ST67_TX; removed none
- moved on the sheet: J101

Commit message: KiCad work
Other:
- added sheet Power Supply +3.3V (PowerSupply3.3V.kicad_sch)
- sheet Host Controller ports: added ST67_BOOT, ST67_CHIP_EN, ST67_CS, ST67_RDY; removed none
- sheet ST67W611M1 ports: added +3.3V, BOOT, CHIP_EN; removed none
- note added: "Power consumption ----------------- ST67W611M1 <1mA / ~400mA peak STM32G0B1xx 10mA max SCT2024 10mA max x 4"

Commit message: KiCad work
Parts:
- removed J102, J103: Conn_01x10, symbol Connector_Generic:Conn_01x10
- added C609: 100n, symbol Device:C
- added J102, J108: Conn_01x16, symbol Connector_Generic:Conn_01x16
- added J107: POWER_SELECT, symbol Connector:Conn_01x03_Pin
- added R606: 105k, symbol Device:R
- added U604: INA180A2, Package_TO_SOT_SMD:SOT-23-5, symbol Amplifier_Current:INA180A2
Connections:
- net +3.3V: now also J106.1 (Pin_1), C609.1, U604.5 (V+)
- net Display/DIS1_EN: now also J102.11 (Pin_11), J108.11 (Pin_11)
- net Display/DIS2_EN: now also J102.12 (Pin_12), J108.12 (Pin_12)
- net Display/DIS3_EN: now also J102.13 (Pin_13), J108.13 (Pin_13)
- net Display/DIS4_EN: now also J102.14 (Pin_14), J108.14 (Pin_14)
- net Display/DIS5_EN: now also J102.15 (Pin_15), J108.15 (Pin_15)
- net Display/LOW_POWER_ENABLE: now also J102.16 (Pin_16), J108.16 (Pin_16)
- net Display/SCT_CLK: now also J102.7 (Pin_7), J108.7 (Pin_7)
- net Display/~{SCT_EN}: now also J102.10 (Pin_10), J108.10 (Pin_10)
- net Display/~{SCT_LA}: now also J102.9 (Pin_9), J108.9 (Pin_9)
- net GND: now also J104.1 (Pin_1), J106.2 (Pin_2), C609.2, J102.1 (Pin_1), J102.3 (Pin_3), J102.6 (Pin_6), J102.8 (Pin_8), J108.1 (Pin_1), J108.3 (Pin_3), J108.6 (Pin_6), J108.8 (Pin_8), U604.2 (GND)
- net Host Controller/I2C_SCL: now also J106.3 (Pin_3)
- net Host Controller/I2C_SDA: now also J106.4 (Pin_4)
- net VBUS: now also J102.2 (Pin_2), J102.4 (Pin_4), J108.2 (Pin_2), J108.4 (Pin_4), R606.2, U604.4 (-); no longer J101.A4 (VBUS), J101.A9 (VBUS), J101.B4 (VBUS), J101.B9 (VBUS)
- net at J104.2 (Pin_2): now also J107.1 (Pin_1)
- new net: J101.A4 (VBUS), J101.A9 (VBUS), J101.B4 (VBUS), J101.B9 (VBUS), J107.3 (Pin_3)
- new net Display/SCT_SDI: J102.5 (Pin_5), J108.5 (Pin_5)
- new net Host Controller/CURRENT_SENSE: U604.1
- new net Host Controller/VOLTAGE_SENSE: J107.2 (Pin_2), R606.1, U604.3 (+)
Other:
- removed sheet Power Supply +3.3V
- sheet Display ports: added SCT_SDI; removed STC_SDI
- sheet Host Controller ports: added CURRENT_SENSE, VOLTAGE_SENSE; removed none
- sheet Power Supply ports: added +3.3V, +3.7V, GND, VDD; removed none
- note added: "INA180AX: Imax = 3A Usense(max) = 3V G=20 -> Rsense = 3V/20/3A = 0.05 Ohm | 0.15V drop G=50 -> Rsense = 0.02 Ohm | 0.06V G=100 -> Rsesne = 0.01 Ohm | 0.03V"
- moved on the sheet: D101, D102, J101, J104, J105, J106

Commit message: KiCad work
Parts:
- R606: value 105k -> 0.05
Connections:
- net Display/DIS1_EN renamed Controller/DIS1_EN
- net Display/DIS2_EN renamed Controller/DIS2_EN
- net Display/DIS3_EN renamed Controller/DIS3_EN
- net Display/DIS4_EN renamed Controller/DIS4_EN
- net Display/DIS5_EN renamed Controller/DIS5_EN
- net Display/LOW_POWER_ENABLE renamed Controller/LOW_POWER_ENABLE
- net Display/SCT_CLK renamed Controller/SCT_CLK
- net Display/SCT_SDI renamed Controller/SCT_SDI
- net Display/~{SCT_EN} renamed Controller/~{SCT_EN}
- net Display/~{SCT_LA} renamed Controller/~{SCT_LA}
- net Host Controller/I2C_SCL renamed Controller/I2C_SCL
- net Host Controller/I2C_SDA renamed Controller/I2C_SDA
- net Host Controller/NRST renamed Controller/NRST
- net Host Controller/SWCLK renamed Controller/SWCLK
- net Host Controller/SWDIO renamed Controller/SWDIO
Other:
- sheet Controller ports: added +3.3V, DIS1_EN, DIS2_EN, DIS3_EN, DIS4_EN, DIS5_EN, GND, I2C_SCL, I2C_SDA, LOW_POWER_ENABLE, NRST, SCT_CLK, SCT_SDI, SWCLK, SWDIO, ~{SCT_EN}, ~{SCT_LA}; removed none
- note added: "INA180AX ----------- Imax = 3A Usense(max) = 3V G=20 -> Rsense = 3V/20/3A = 0.05 Ohm | 0.15V drop G=50 -> Rsense = 0.02 Ohm | 0.06V G=100 -> Rsesne = 0.01 Ohm | 0.03V"
- note removed: "INA180AX: Imax = 3A Usense(max) = 3V G=20 -> Rsense = 3V/20/3A = 0.05 Ohm | 0.15V drop G=50 -> Rsense = 0.02 Ohm | 0.06V G=100 -> Rsesne = 0.01 Ohm | 0.03V"
- moved on the sheet: C609, D101, D102, J101, J102, J104, J105, J106, J107, J108, R606, U604

Commit message: KiCad work
Parts:
- removed J102, J108: Conn_01x16, symbol Connector_Generic:Conn_01x16
- added J101: OUTPUT, Connector_PinSocket_2.54mm:PinSocket_1x21_P2.54mm_Horizontal, symbol Connector_Generic:Conn_01x21
- added J105: INPUT, Connector_PinHeader_2.54mm:PinHeader_1x21_P2.54mm_Horizontal, symbol Connector_Generic:Conn_01x21
- C101: renamed from C609; footprint (none) -> Capacitor_SMD:C_0603_1608Metric
- D101, D102: footprint (none) -> Diode_SMD:D_SOD-323
- J102: renamed from J106; footprint (none) -> Connector_PinHeader_2.54mm:PinHeader_1x04_P2.54mm_Vertical
- J103: renamed from J105; footprint (none) -> Connector_JST:JST_PH_S6B-PH-SM4-TB_1x06-1MP_P2.00mm_Horizontal
- J104: footprint (none) -> Connector_PinSocket_2.54mm:PinSocket_1x02_P2.54mm_Vertical
- J106: renamed from J107; footprint (none) -> Connector_PinSocket_2.54mm:PinSocket_1x03_P2.54mm_Vertical
- J107: renamed from J101; footprint (none) -> Connector_USB:USB_C_Receptacle_GCT_USB4135-GF-A_6P_TopMnt_Horizontal
- R101: renamed from R606; footprint (none) -> Resistor_SMD:R_1206_3216Metric
- renumbered U604 to U101
Connections:
- net Controller/DIS1_EN: now also J101.17 (Pin_17), J105.17 (Pin_17)
- net Controller/DIS2_EN: now also J101.18 (Pin_18), J105.18 (Pin_18)
- net Controller/DIS3_EN: now also J101.19 (Pin_19), J105.19 (Pin_19)
- net Controller/DIS4_EN: now also J101.20 (Pin_20), J105.20 (Pin_20)
- net Controller/DIS5_EN: now also J101.21 (Pin_21), J105.21 (Pin_21)
- net Controller/I2C_SCL: now also J101.2 (Pin_2), J105.2 (Pin_2)
- net Controller/I2C_SDA: now also J101.4 (Pin_4), J105.4 (Pin_4)
- net Controller/SCT_CLK: now also J101.13 (Pin_13), J105.13 (Pin_13)
- net Controller/SCT_SDI: now also J101.11 (Pin_11), J105.11 (Pin_11)
- net Controller/~{SCT_EN}: now also J101.16 (Pin_16), J105.16 (Pin_16)
- net Controller/~{SCT_LA}: now also J101.15 (Pin_15), J105.15 (Pin_15)
- net Display/LED_BRIGHTNESS: now also J101.10 (Pin_10), J105.10 (Pin_10)
- net GND: now also J101.1 (Pin_1), J101.12 (Pin_12), J101.14 (Pin_14), J101.3 (Pin_3), J101.5 (Pin_5), J101.7 (Pin_7), J105.1 (Pin_1), J105.12 (Pin_12), J105.14 (Pin_14), J105.3 (Pin_3), J105.5 (Pin_5), J105.7 (Pin_7)
- net VBUS: now also J101.6 (Pin_6), J101.8 (Pin_8), J105.6 (Pin_6), J105.8 (Pin_8)
- new net Host Controller/LOW_POWER_ENABLE: J101.9 (Pin_9), J105.9 (Pin_9)
Other:
- added sheet Light Sensor (LightSensor.kicad_sch)
- sheet Controller ports: added none; removed LOW_POWER_ENABLE
- sheet Display ports: added none; removed LOW_POWER_ENABLE
- moved on the sheet: J102, J103

Commit message: KiCad work
Parts:
- added R102, R103: 5k1, Resistor_SMD:R_0805_2012Metric, symbol Device:R
Connections:
- net Controller/SCT_SDI: no longer J101.11 (Pin_11)
- net GND: now also R102.2, R103.2
- net Host Controller/UCPD_CC1: now also R103.1
- net Host Controller/UCPD_CC2: now also R102.1
- new net Display/SCT_SDO: J101.11 (Pin_11)
Other:
- sheet Display ports: added SCT_SDO; removed none

Commit message: Work
Parts:
- J103: footprint Connector_JST:JST_PH_S6B-PH-SM4-TB_1x06-1MP_P2.00mm_Horizontal -> Connector_JST:JST_PH_B6B-PH-K_1x06_P2.00mm_Vertical
- J107: value USB_C_Receptacle_USB2.0_14P -> USB; footprint Connector_USB:USB_C_Receptacle_GCT_USB4135-GF-A_6P_TopMnt_Horizontal -> JPConnectors:USB_C_Receptacle_GCT_USB4216
Connections:
- net Controller/DIS1_EN renamed Controller/DISPLAY1_EN
- net Controller/DIS2_EN renamed Controller/DISPLAY2_EN
- net Controller/DIS3_EN renamed Controller/DISPLAY3_EN
- net Controller/DIS4_EN renamed Controller/DISPLAY4_EN
- net Controller/DIS5_EN renamed Controller/DISPLAY5_EN
Other:
- sheet Controller ports: added DISPLAY1_EN, DISPLAY2_EN, DISPLAY3_EN, DISPLAY4_EN, DISPLAY5_EN; removed DIS1_EN, DIS2_EN, DIS3_EN, DIS4_EN, DIS5_EN
- sheet Display ports: added DISPLAY1_EN, DISPLAY2_EN, DISPLAY3_EN, DISPLAY4_EN, DISPLAY5_EN; removed DIS1_EN, DIS2_EN, DIS3_EN, DIS4_EN, DIS5_EN
- sheet Host Controller ports: added DISPLAY1_EN, DISPLAY2_EN, DISPLAY3_EN, DISPLAY4_EN, DISPLAY5_EN; removed DIS1_EN, DIS2_EN, DIS3_EN, DIS4_EN, DIS5_EN
Changed lines of the file:
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@@
 			)
 		)
-		(property "Footprint" "Connector_JST:JST_PH_S6B-PH-SM4-TB_1x06-1MP_P2.00mm_Horizontal"
+		(property "Footprint" "Connector_JST:JST_PH_B6B-PH-K_1x06_P2.00mm_Vertical"
 			(at 140.97 83.82 0)
 			(effects
@@
 			)
 		)
-		(property "Value" "USB_C_Receptacle_USB2.0_14P"
+		(property "Value" "USB"
 			(at 129.54 201.93 0)
 			(effects
@@
 			)
 		)
-		(property "Footprint" "Connector_USB:USB_C_Receptacle_GCT_USB4135-GF-A_6P_TopMnt_Horizontal"
+		(property "Footprint" "JPConnectors:USB_C_Receptacle_GCT_USB4216"
 			(at 133.35 220.98 0)
 			(effects
@@
 			)
 		)
-		(pin "DIS1_EN" output
-			(at 217.17 69.85 0)
+		(pin "GND" input
+			(at 193.04 87.63 270)
 			(effects
 				(font
 					(size 1.27 1.27)
 				)
-				(justify right)
+				(justify left)
 			)
 		)
-		(pin "DIS2_EN" output
-			(at 217.17 72.39 0)
+		(pin "I2C_SCL" output
+			(at 181.61 64.77 180)
 			(effects
 				(font
 					(size 1.27 1.27)
 				)
-				(justify right)
+				(justify left)
 			)
 		)
-		(pin "DIS3_EN" output
-			(at 217.17 74.93 0)
+		(pin "I2C_SDA" bidirectional
+			(at 181.61 62.23 180)
 			(effects
 				(font
 					(size 1.27 1.27)
 				)
-				(justify right)
+				(justify left)
 			)
 		)
-		(pin "DIS4_EN" output
-			(at 217.17 77.47 0)
+		(pin "NRST" input
+			(at 181.61 72.39 180)
 			(effects
 				(font
 					(size 1.27 1.27)
 				)
-				(justify right)
+				(justify left)
 			)
 		)
-		(pin "DIS5_EN" output
-			(at 217.17 80.01 0)
+		(pin "SCT_CLK" output
+			(at 217.17 59.69 0)
 			(effects
 				(font
@@
 			)
 		)
-		(pin "GND" input
-			(at 193.04 87.63 270)
+		(pin "SCT_SDI" output
+			(at 217.17 57.15 0)
 			(effects
 				(font
 					(size 1.27 1.27)
 				)
-				(justify left)
+				(justify right)
 			)
 		)
-		(pin "I2C_SCL" output
-			(at 181.61 64.77 180)
+		(pin "SWCLK" input
+			(at 181.61 77.47 180)
 			(effects
 				(font
@@
 			)
 		)
-		(pin "I2C_SDA" bidirectional
-			(at 181.61 62.23 180)
+		(pin "SWDIO" input
+			(at 181.61 74.93 180)
 			(effects
 				(font
@@
 			)
 		)
-		(pin "NRST" input
-			(at 181.61 72.39 180)
+		(pin "~{SCT_EN}" output
+			(at 217.17 66.04 0)
 			(effects
 				(font
 					(size 1.27 1.27)
 				)
-				(justify left)
+				(justify right)
 			)
 		)
-		(pin "SCT_CLK" output
-			(at 217.17 59.69 0)
+		(pin "~{SCT_LA}" output
+			(at 217.17 63.5 0)
 			(effects
 				(font
@@
 			)
 		)
-		(pin "SCT_SDI" output
-			(at 217.17 57.15 0)
+		(pin "DISPLAY1_EN" output
+			(at 217.17 69.85 0)
 			(effects
 				(font
@@
 			)
 		)
-		(pin "SWCLK" input
-			(at 181.61 77.47 180)
+		(pin "DISPLAY2_EN" output
+			(at 217.17 72.39 0)
 			(effects
 				(font
 					(size 1.27 1.27)
 				)
-				(justify left)
+				(justify right)
 			)
 		)
-		(pin "SWDIO" input
-			(at 181.61 74.93 180)
+		(pin "DISPLAY3_EN" output
+			(at 217.17 74.93 0)
 			(effects
 				(font
 					(size 1.27 1.27)
 				)
-				(justify left)
+				(justify right)
 			)
 		)
-		(pin "~{SCT_EN}" output
-			(at 217.17 66.04 0)
+		(pin "DISPLAY4_EN" output
+			(at 217.17 77.47 0)
 			(effects
 				(font
@@
 			)
 		)
-		(pin "~{SCT_LA}" output
-			(at 217.17 63.5 0)
+		(pin "DISPLAY5_EN" output
+			(at 217.17 80.01 0)
 			(effects
 				(font
@@
 			)
 		)
-		(pin "DIS1_EN" input
-			(at 295.91 133.35 180)
+		(pin "SCT_CLK" input
+			(at 295.91 123.19 180)
 			(effects
 				(font
@@
 			)
 		)
-		(pin "DIS2_EN" input
-			(at 295.91 135.89 180)
+		(pin "~{SCT_EN}" input
+			(at 295.91 129.54 180)
 			(effects
 				(font
@@
 			)
 		)
-		(pin "DIS3_EN" input
-			(at 295.91 138.43 180)
+		(pin "~{SCT_LA}" input
+			(at 295.91 127 180)
 			(effects
 				(font
@@
 			)
 		)
-		(pin "DIS4_EN" input
-			(at 295.91 140.97 180)
+		(pin "GND" input
+			(at 322.58 153.67 270)
 			(effects
 				(font
@@
 			)
 		)
-		(pin "DIS5_EN" input
-			(at 295.91 143.51 180)
+		(pin "VLED" input
+			(at 322.58 115.57 90)
 			(effects
 				(font
 					(size 1.27 1.27)
 				)
-				(justify left)
+				(justify right)
 			)
 		)
-		(pin "SCT_CLK" input
-			(at 295.91 123.19 180)
+		(pin "SCT_SDI" input
+			(at 295.91 118.11 180)
 			(effects
 				(font
@@
 			)
 		)
-		(pin "~{SCT_EN}" input
-			(at 295.91 129.54 180)
+		(pin "LED_BRIGHTNESS" input
+			(at 295.91 149.86 180)
 			(effects
 				(font
@@
 			)
 		)
-		(pin "~{SCT_LA}" input
-			(at 295.91 127 180)
+		(pin "SCT_SDO" output
+			(at 295.91 120.65 180)
 			(effects
 				(font
@@
 			)
 		)
-		(pin "GND" input
-			(at 322.58 153.67 270)
+		(pin "DISPLAY1_EN" input
+			(at 295.91 133.35 180)
 			(effects
 				(font
@@
 			)
 		)
-		(pin "VLED" input
-			(at 322.58 115.57 90)
+		(pin "DISPLAY2_EN" input
+			(at 295.91 135.89 180)
 			(effects
 				(font
 					(size 1.27 1.27)
 				)
-				(justify right)
+				(justify left)
 			)
 		)
-		(pin "SCT_SDI" input
-			(at 295.91 118.11 180)
+		(pin "DISPLAY3_EN" input
+			(at 295.91 138.43 180)
 			(effects
 				(font
@@
 			)
 		)
-		(pin "LED_BRIGHTNESS" input
-			(at 295.91 149.86 180)
+		(pin "DISPLAY4_EN" input
+			(at 295.91 140.97 180)
 			(effects
 				(font
@@
 			)
 		)
-		(pin "SCT_SDO" output
-			(at 295.91 120.65 180)
+		(pin "DISPLAY5_EN" input
+			(at 295.91 143.51 180)
 			(effects
 				(font
@@
 			)
 		)
-		(pin "DIS1_EN" output
-			(at 217.17 133.35 0)
+		(pin "SCT_CLK" output
+			(at 217.17 123.19 0)
 			(effects
 				(font
@@
 			)
 		)
-		(pin "DIS2_EN" output
-			(at 217.17 135.89 0)
+		(pin "~{SCT_EN}" output
+			(at 217.17 129.54 0)
 			(effects
 				(font
@@
 			)
 		)
-		(pin "DIS3_EN" output
-			(at 217.17 138.43 0)
+		(pin "~{SCT_LA}" output
+			(at 217.17 127 0)
 			(effects
 				(font
@@
 			)
 		)
-		(pin "DIS4_EN" output
-			(at 217.17 140.97 0)
+		(pin "LOW_POWER_ENABLE" output
+			(at 217.17 147.32 0)
 			(effects
 				(font
@@
 			)
 		)
-		(pin "DIS5_EN" output
-			(at 217.17 143.51 0)
+		(pin "SCT_SDI" output
+			(at 217.17 120.65 0)
 			(effects
 				(font
@@
 			)
 		)
-		(pin "SCT_CLK" output
-			(at 217.17 123.19 0)
+		(pin "ST67_BOOT" output
+			(at 160.02 149.86 180)
 			(effects
 				(font
 					(size 1.27 1.27)
 				)
-				(justify right)
+				(justify left)
 			)
 		)
-		(pin "~{SCT_EN}" output
-			(at 217.17 129.54 0)
+		(pin "ST67_CHIP_EN" output
+			(at 160.02 147.32 180)
 			(effects
 				(font
 					(size 1.27 1.27)
 				)
-				(justify right)
+				(justify left)
 			)
 		)
-		(pin "~{SCT_LA}" output
-			(at 217.17 127 0)
+		(pin "ST67_CS" output
+			(at 160.02 135.89 180)
 			(effects
 				(font
 					(size 1.27 1.27)
 				)
-				(justify right)
+				(justify left)
 			)
 		)
-		(pin "LOW_POWER_ENABLE" output
-			(at 217.17 147.32 0)
+		(pin "ST67_RDY" input
+			(at 160.02 139.7 180)
 			(effects
 				(font
 					(size 1.27 1.27)
 				)
-				(justify right)
+				(justify left)
 			)
 		)
-		(pin "SCT_SDI" output
-			(at 217.17 120.65 0)
+		(pin "CURRENT_SENSE" input
+			(at 180.34 156.21 270)
 			(effects
 				(font
 					(size 1.27 1.27)
 				)
-				(justify right)
+				(justify left)
 			)
 		)
-		(pin "ST67_BOOT" output
-			(at 160.02 149.86 180)
+		(pin "VOLTAGE_SENSE" input
+			(at 177.8 156.21 270)
 			(effects
 				(font
@@
 			)
 		)
-		(pin "ST67_CHIP_EN" output
-			(at 160.02 147.32 180)
+		(pin "DISPLAY1_EN" output
+			(at 217.17 133.35 0)
 			(effects
 				(font
 					(size 1.27 1.27)
 				)
-				(justify left)
+				(justify right)
 			)
 		)
-		(pin "ST67_CS" output
-			(at 160.02 135.89 180)
+		(pin "DISPLAY2_EN" output
+			(at 217.17 135.89 0)
 			(effects
 				(font
 					(size 1.27 1.27)
 				)
-				(justify left)
+				(justify right)
 			)
 		)
-		(pin "ST67_RDY" input
-			(at 160.02 139.7 180)
+		(pin "DISPLAY3_EN" output
+			(at 217.17 138.43 0)
 			(effects
 				(font
 					(size 1.27 1.27)
 				)
-				(justify left)
+				(justify right)
 			)
 		)
-		(pin "CURRENT_SENSE" input
-			(at 180.34 156.21 270)
+		(pin "DISPLAY4_EN" output
+			(at 217.17 140.97 0)
 			(effects
 				(font
 					(size 1.27 1.27)
 				)
-				(justify left)
+				(justify right)
 			)
 		)
-		(pin "VOLTAGE_SENSE" input
-			(at 177.8 156.21 270)
+		(pin "DISPLAY5_EN" output
+			(at 217.17 143.51 0)
 			(effects
 				(font
 					(size 1.27 1.27)
 				)
-				(justify left)
+				(justify right)
 			)
 		)
