File: KiCad/AstroWeather.kicad_sch (KiCad schematic)
At the start: 14 parts, among them J101 OUTPUT, J102 I2C, J103 SWD, J104 AUX_POWER, J105 INPUT, J106 POWER_SELECT, J107 USB, U101 INA180A2

Commit message: KiCad work
Parts:
- removed J106: POWER_SELECT, Connector_PinSocket_2.54mm:PinSocket_1x03_P2.54mm_Vertical, symbol Connector:Conn_01x03_Pin
- J104: footprint Connector_PinSocket_2.54mm:PinSocket_1x02_P2.54mm_Vertical -> Connector_PinHeader_2.54mm:PinHeader_1x02_P2.54mm_Vertical
Connections:
- net Host Controller/VOLTAGE_SENSE: now also J104.2 (Pin_2), J107.A4 (VBUS), J107.A9 (VBUS), J107.B4 (VBUS), J107.B9 (VBUS)
- net Controller/DISPLAY1_EN renamed Display/DISPLAY1_EN
- net Controller/DISPLAY2_EN renamed Display/DISPLAY2_EN
- net Controller/DISPLAY3_EN renamed Display/DISPLAY3_EN
- net Controller/DISPLAY4_EN renamed Display/DISPLAY4_EN
- net Controller/DISPLAY5_EN renamed Display/DISPLAY5_EN
- net Controller/I2C_SCL renamed Host Controller/I2C_SCL
- net Controller/I2C_SDA renamed Host Controller/I2C_SDA
- net Controller/NRST renamed Host Controller/NRST
- net Controller/SCT_CLK renamed Display/SCT_CLK
- net Controller/SCT_SDI renamed Display/SCT_SDI
- net Controller/SWCLK renamed Host Controller/SWCLK
- net Controller/SWDIO renamed Host Controller/SWDIO
- net Controller/~{SCT_EN} renamed Display/~{SCT_EN}
- net Controller/~{SCT_LA} renamed Display/~{SCT_LA}
Other:
- removed sheet Controller
- moved on the sheet: J104

Commit message: KiCad work
Parts:
- removed J101: OUTPUT, Connector_PinSocket_2.54mm:PinSocket_1x21_P2.54mm_Horizontal, symbol Connector_Generic:Conn_01x21
- removed J105: INPUT, Connector_PinHeader_2.54mm:PinHeader_1x21_P2.54mm_Horizontal, symbol Connector_Generic:Conn_01x21
- added H101, H102, H103: MountingHole, symbol Mechanical:MountingHole
- added J101: Conn_01x10, Connector_PinSocket_2.54mm:PinSocket_1x10_P2.54mm_Horizontal, symbol Connector_Generic:Conn_01x10
- added J105: Conn_01x10, Connector_PinHeader_2.54mm:PinHeader_1x10_P2.54mm_Horizontal, symbol Connector_Generic:Conn_01x10
Connections:
- net Display/LED_BRIGHTNESS: now also J101.10 (Pin_10), J105.10 (Pin_10)
- net GND: now also J101.1 (Pin_1), J101.3 (Pin_3), J101.5 (Pin_5), J101.7 (Pin_7), J105.1 (Pin_1), J105.3 (Pin_3), J105.5 (Pin_5), J105.7 (Pin_7)
- net Host Controller/I2C_SCL: now also J101.2 (Pin_2), J105.2 (Pin_2)
- net Host Controller/I2C_SDA: now also J101.4 (Pin_4), J105.4 (Pin_4)
- net Host Controller/LOW_POWER_ENABLE: now also J101.9 (Pin_9), J105.9 (Pin_9)
- net VBUS: now also J101.6 (Pin_6), J101.8 (Pin_8), J105.6 (Pin_6), J105.8 (Pin_8)

Commit message: KiCad work
Parts:
- H101, H102, H103: footprint (none) -> MountingHole:MountingHole_3.2mm_M3
- renumbered J102 to J101, J101 to J102, J105 to J104, J104 to J105, J107 to J106

Commit message: KiCad work
Other:
- moved on the sheet: J101
Changed lines of the file:
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@@
 	(wire
 		(pts
-			(xy 146.05 69.85) (xy 149.86 69.85)
-		)
-		(stroke
-			(width 0)
-			(type default)
-		)
-	)
-	(wire
-		(pts
-			(xy 146.05 64.77) (xy 175.26 64.77)
+			(xy 170.18 62.23) (xy 170.18 66.04)
 		)
 		(stroke
@@
 	(wire
 		(pts
-			(xy 146.05 67.31) (xy 147.32 67.31)
+			(xy 172.72 62.23) (xy 172.72 63.5)
 		)
 		(stroke
@@
 	(wire
 		(pts
+			(xy 175.26 62.23) (xy 175.26 96.52)
+		)
+		(stroke
+			(width 0)
+			(type default)
+		)
+	)
+	(wire
+		(pts
 			(xy 144.78 220.98) (xy 147.32 220.98)
 		)
@@
 	(wire
 		(pts
-			(xy 146.05 62.23) (xy 177.8 62.23)
-		)
-		(stroke
-			(width 0)
-			(type default)
-		)
-	)
-	(wire
-		(pts
 			(xy 322.58 182.88) (xy 322.58 184.15)
 		)
@@
 		(pts
 			(xy 322.58 167.64) (xy 322.58 168.91)
-		)
-		(stroke
-			(width 0)
-			(type default)
-		)
-	)
-	(wire
-		(pts
-			(xy 175.26 64.77) (xy 175.26 96.52)
 		)
 		(stroke
@@
 	(symbol
 		(lib_id "power:GND")
-		(at 147.32 67.31 90)
+		(at 172.72 63.5 0)
 		(unit 1)
 		(exclude_from_sim no)
@@
 		(fields_autoplaced yes)
 		(property "Reference" "#PWR0102"
-			(at 153.67 67.31 0)
+			(at 172.72 69.85 0)
 			(effects
 				(font
@@
 		)
 		(property "Value" "GND"
-			(at 152.4 67.31 0)
+			(at 172.72 68.58 0)
 			(effects
 				(font
@@
 		)
 		(property "Footprint" ""
-			(at 147.32 67.31 0)
+			(at 172.72 63.5 0)
 			(effects
 				(font
@@
 		)
 		(property "Datasheet" ""
-			(at 147.32 67.31 0)
+			(at 172.72 63.5 0)
 			(effects
 				(font
@@
 		)
 		(property "Description" "Power symbol creates a global label with name \"GND\" , ground"
-			(at 147.32 67.31 0)
+			(at 172.72 63.5 0)
 			(effects
 				(font
@@
 	(symbol
 		(lib_id "Connector_Generic:Conn_01x04")
-		(at 140.97 67.31 180)
+		(at 172.72 57.15 90)
 		(unit 1)
 		(exclude_from_sim no)
@@
 		(fields_autoplaced yes)
 		(property "Reference" "J101"
-			(at 134.62 66.04 90)
+			(at 173.99 50.8 90)
 			(effects
 				(font
@@
 		)
 		(property "Value" "I2C"
-			(at 137.16 66.04 90)
+			(at 173.99 53.34 90)
 			(effects
 				(font
@@
 		)
 		(property "Footprint" "Connector_PinHeader_2.54mm:PinHeader_1x04_P2.54mm_Vertical"
-			(at 140.97 67.31 0)
+			(at 172.72 57.15 0)
 			(effects
 				(font
@@
 		)
 		(property "Datasheet" "~"
-			(at 140.97 67.31 0)
+			(at 172.72 57.15 0)
 			(effects
 				(font
@@
 		)
 		(property "Description" "Generic connector, single row, 01x04, script generated (kicad-library-utils/schlib/autogen/connector/)"
-			(at 140.97 67.31 0)
+			(at 172.72 57.15 0)
 			(effects
 				(font
@@
 	(symbol
 		(lib_id "power:+3.3V")
-		(at 149.86 69.85 270)
+		(at 170.18 66.04 180)
 		(unit 1)
 		(exclude_from_sim no)
@@
 		(fields_autoplaced yes)
 		(property "Reference" "#PWR0103"
-			(at 146.05 69.85 0)
+			(at 170.18 62.23 0)
 			(effects
 				(font
@@
 		)
 		(property "Value" "+3.3V"
-			(at 154.94 69.85 0)
+			(at 170.18 71.12 0)
 			(effects
 				(font
@@
 		)
 		(property "Footprint" ""
-			(at 149.86 69.85 0)
+			(at 170.18 66.04 0)
 			(effects
 				(font
@@
 		)
 		(property "Datasheet" ""
-			(at 149.86 69.85 0)
+			(at 170.18 66.04 0)
 			(effects
 				(font
@@
 		)
 		(property "Description" "Power symbol creates a global label with name \"+3.3V\""
-			(at 149.86 69.85 0)
-			(effects
-				(font
+			(at 170.18 66.04 0)
+			(effects
+				(font

Commit message: KiCad finishing touches, gerber
Connections:
- net Host Controller/VOLTAGE_SENSE renamed VBUS_IN
Changed lines of the file:
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@@
+		)
+	)
+	(label "VBUS_IN"
+		(at 156.21 193.04 0)
+		(effects
+			(font
+				(size 1.27 1.27)
+			)
+			(justify left bottom)
 		)
 	)
