File: KiCad/AstroWeather.kicad_sch (KiCad schematic)
At the start: 16 parts, among them J101 I2C, J102 Conn_01x10, J103 SWD, J104 Conn_01x10, J105 AUX_POWER, J106 USB, U101 INA180A2

Commit message: bug mentioned
Other:
- note added: "Bugs: Missing voltage divider on input voltage sense"
Changed lines of the file:
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@@
+		)
+	)
+	(text "Bugs:\nMissing voltage divider on input voltage sense"
+		(exclude_from_sim no)
+		(at 18.796 24.13 0)
+		(effects
+			(font
+				(size 3 3)
+			)
+			(justify left)
 		)
 	)

Commit message: Bug added: wrong sense pins
Other:
- note added: "Bugs: Missing voltage divider on input voltage sense SENSE inputs connected to non-ADC pins"
- note removed: "Bugs: Missing voltage divider on input voltage sense"
Changed lines of the file:
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@@
 		)
 	)
-	(text "Bugs:\nMissing voltage divider on input voltage sense"
+	(text "Bugs:\nMissing voltage divider on input voltage sense\nSENSE inputs connected to non-ADC pins"
 		(exclude_from_sim no)
 		(at 18.796 24.13 0)
@@
 				(size 3 3)
 			)
-			(justify left)
+			(justify left top)
 		)
 	)

Commit message: Sensors initial commit
Other:
- note added: "Bugs: Missing voltage divider on input voltage sense SENSE inputs connected to non-ADC pins Vref shorted to GND"
- note removed: "Bugs: Missing voltage divider on input voltage sense SENSE inputs connected to non-ADC pins"
Changed lines of the file:
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@@
 		)
 	)
-	(text "Bugs:\nMissing voltage divider on input voltage sense\nSENSE inputs connected to non-ADC pins"
+	(text "Bugs:\nMissing voltage divider on input voltage sense\nSENSE inputs connected to non-ADC pins\nVref shorted to GND"
 		(exclude_from_sim no)
 		(at 18.796 24.13 0)
