File: KiCad/Controller.kicad_sch (KiCad schematic)
At the start: 0 parts

Commit message: KiCad work
Parts:
- added C401: 100n, symbol Device:C
- added C402: 4u7, symbol Device:C
- added C403: 100n, Capacitor_SMD:C_0603_1608Metric, symbol Device:C
- added R401: R, symbol Device:R
- added SW401: Reset, symbol Switch:SW_Push
- added U401: STM32G030F6Px, Package_SO:TSSOP-20_4.4x6.5mm_P0.65mm, symbol MCU_ST_STM32G0:STM32G030F6Px
Connections:
- new net +3.3V: C401.1, C402.1, U401.4 (VDD)
- new net GND: C401.2, C402.2, C403.2, SW401.1, U401.5 (VSS)
- new net I2C_SCL: U401.16 (PA9/PA11)
- new net I2C_SDA: U401.17 (PA10/PA12)
- new net NRST: C403.1, SW401.2, U401.6 (NRST)
- new net SCT_CLK: U401.8 (PA1)
- new net SCT_SDI: U401.9 (PA2)
- new net SWCLK: U401.19 (PA14/PA15)
- new net SWDIO: U401.18 (PA13)

Commit message: KiCad work
Parts:
- removed R401: R, symbol Device:R
- C401: footprint (none) -> Capacitor_SMD:C_0603_1608Metric
- C402: footprint (none) -> Capacitor_SMD:C_0805_2012Metric
- SW401: footprint (none) -> Button_Switch_SMD:SW_Tactile_SPST_NO_Straight_CK_PTS636Sx25SMTRLFS
Changed lines of the file:
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@@
-		)
-	)
-	(hierarchical_label "LOW_POWER_ENABLE"
-		(shape output)
-		(at 185.42 87.63 0)
-		(effects
-			(font
-				(size 1.27 1.27)
-			)
-			(justify left)
 		)
 	)
@@
 			)
 		)
-		(property "Footprint" ""
+		(property "Footprint" "Capacitor_SMD:C_0805_2012Metric"
 			(at 169.8752 40.64 0)
 			(effects
@@
 		(dnp no)
 		(fields_autoplaced yes)
-		(property "Reference" "#PWR0406"
+		(property "Reference" "#PWR0403"
 			(at 156.21 49.53 0)
 			(effects
@@
 			(project "AstroWeather"
 				(path "/8561283c-f5b3-4542-8880-7f435c3a9f7c/4c8e54d0-2d5b-47d4-b46b-1559d4095c20"
-					(reference "#PWR0406")
+					(reference "#PWR0403")
 					(unit 1)
 				)
@@
 		(dnp no)
 		(fields_autoplaced yes)
-		(property "Reference" "#PWR0405"
+		(property "Reference" "#PWR0401"
 			(at 156.21 34.29 0)
 			(effects
@@
 			(project "AstroWeather"
 				(path "/8561283c-f5b3-4542-8880-7f435c3a9f7c/4c8e54d0-2d5b-47d4-b46b-1559d4095c20"
-					(reference "#PWR0405")
+					(reference "#PWR0401")
 					(unit 1)
 				)
@@
 		(dnp no)
 		(fields_autoplaced yes)
-		(property "Reference" "#PWR0402"
+		(property "Reference" "#PWR0408"
 			(at 139.7 113.03 0)
 			(effects
@@
 			(project ""
 				(path "/8561283c-f5b3-4542-8880-7f435c3a9f7c/4c8e54d0-2d5b-47d4-b46b-1559d4095c20"
-					(reference "#PWR0402")
+					(reference "#PWR0408")
 					(unit 1)
 				)
@@
 			)
 		)
-		(property "Footprint" ""
+		(property "Footprint" "Capacitor_SMD:C_0603_1608Metric"
 			(at 157.1752 40.64 0)
 			(effects
@@
 		(dnp no)
 		(fields_autoplaced yes)
-		(property "Reference" "#PWR0404"
+		(property "Reference" "#PWR0405"
 			(at 139.7 62.23 0)
 			(effects
@@
 			(project "AstroWeather"
 				(path "/8561283c-f5b3-4542-8880-7f435c3a9f7c/4c8e54d0-2d5b-47d4-b46b-1559d4095c20"
-					(reference "#PWR0404")
-					(unit 1)
-				)
-			)
-		)
-	)
-	(symbol
-		(lib_id "Device:R")
-		(at 86.36 59.69 0)
-		(unit 1)
-		(exclude_from_sim no)
-		(in_bom yes)
-		(on_board yes)
-		(dnp no)
-		(fields_autoplaced yes)
-		(property "Reference" "R401"
-			(at 88.9 58.4199 0)
-			(effects
-				(font
-					(size 1.27 1.27)
-				)
-				(justify left)
-			)
-		)
-		(property "Value" "R"
-			(at 88.9 60.9599 0)
-			(effects
-				(font
-					(size 1.27 1.27)
-				)
-				(justify left)
-			)
-		)
-		(property "Footprint" ""
-			(at 84.582 59.69 90)
-			(effects
-				(font
-					(size 1.27 1.27)
-				)
-				(hide yes)
-			)
-		)
-		(property "Datasheet" "~"
-			(at 86.36 59.69 0)
-			(effects
-				(font
-					(size 1.27 1.27)
-				)
-				(hide yes)
-			)
-		)
-		(property "Description" "Resistor"
-			(at 86.36 59.69 0)
-			(effects
-				(font
-					(size 1.27 1.27)
-				)
-				(hide yes)
-			)
-		)
-		(pin "2"
-		)
-		(pin "1"
-		)
-		(instances
-			(project ""
-				(path "/8561283c-f5b3-4542-8880-7f435c3a9f7c/4c8e54d0-2d5b-47d4-b46b-1559d4095c20"
-					(reference "R401")
+					(reference "#PWR0405")
 					(unit 1)
 				)
@@
 		(dnp no)
 		(fields_autoplaced yes)
-		(property "Reference" "#PWR0408"
+		(property "Reference" "#PWR0407"
 			(at 100.33 87.63 0)
 			(effects
@@
 			(project "AstroWeather"
 				(path "/8561283c-f5b3-4542-8880-7f435c3a9f7c/4c8e54d0-2d5b-47d4-b46b-1559d4095c20"
-					(reference "#PWR0408")
+					(reference "#PWR0407")
 					(unit 1)
 				)
@@
 		(dnp no)
 		(fields_autoplaced yes)
-		(property "Reference" "#PWR0407"
+		(property "Reference" "#PWR0406"
 			(at 88.9 87.63 0)
 			(effects
@@
 			(project "AstroWeather"
 				(path "/8561283c-f5b3-4542-8880-7f435c3a9f7c/4c8e54d0-2d5b-47d4-b46b-1559d4095c20"
-					(reference "#PWR0407")
+					(reference "#PWR0406")
 					(unit 1)
 				)
@@
 			)
 		)
-		(property "Footprint" ""
+		(property "Footprint" "Button_Switch_SMD:SW_Tactile_SPST_NO_Straight_CK_PTS636Sx25SMTRLFS"
 			(at 83.82 74.93 0)
 			(effects
@@
 		(dnp no)
 		(fields_autoplaced yes)
-		(property "Reference" "#PWR0403"
+		(property "Reference" "#PWR0404"
 			(at 57.15 50.8 0)
 			(effects
@@
 			(project "AstroWeather"
 				(path "/8561283c-f5b3-4542-8880-7f435c3a9f7c/4c8e54d0-2d5b-47d4-b46b-1559d4095c20"
-					(reference "#PWR0403")
+					(reference "#PWR0404")
 					(unit 1)
 				)
@@
 		(dnp no)
 		(fields_autoplaced yes)
-		(property "Reference" "#PWR0401"
+		(property "Reference" "#PWR0402"
 			(at 57.15 38.1 0)
 			(effects
@@
 			(project ""
 				(path "/8561283c-f5b3-4542-8880-7f435c3a9f7c/4c8e54d0-2d5b-47d4-b46b-1559d4095c20"
-					(reference "#PWR0401")
-					(unit 1)
-				)
+					(reference "#PWR0402")
+					(unit 1)
+				)

Commit message: Work
Changed lines of the file:
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@@
+		)
+	)
+	(hierarchical_label "DISPLAY2_EN"
+		(shape output)
+		(at 207.01 78.74 0)
+		(effects
+			(font
+				(size 1.27 1.27)
+			)
+			(justify left)
 		)
 	)
@@
 		)
 	)
-	(hierarchical_label "DIS2_EN"
-		(shape output)
-		(at 185.42 77.47 0)
-		(effects
-			(font
-				(size 1.27 1.27)
-			)
-			(justify left)
-		)
-	)
 	(hierarchical_label "GND"
 		(shape input)
@@
 			)
 			(justify right)
-		)
-	)
-	(hierarchical_label "DIS3_EN"
-		(shape output)
-		(at 185.42 80.01 0)
-		(effects
-			(font
-				(size 1.27 1.27)
-			)
-			(justify left)
-		)
-	)
-	(hierarchical_label "DIS1_EN"
-		(shape output)
-		(at 185.42 74.93 0)
-		(effects
-			(font
-				(size 1.27 1.27)
-			)
-			(justify left)
 		)
 	)
@@
 		)
 	)
-	(hierarchical_label "DIS5_EN"
-		(shape output)
-		(at 185.42 85.09 0)
-		(effects
-			(font
-				(size 1.27 1.27)
-			)
-			(justify left)
-		)
-	)
 	(hierarchical_label "I2C_SDA"
 		(shape bidirectional)
 		(at 171.45 92.71 0)
-		(effects
-			(font
-				(size 1.27 1.27)
-			)
-			(justify left)
-		)
-	)
-	(hierarchical_label "DIS4_EN"
-		(shape output)
-		(at 185.42 82.55 0)
 		(effects
 			(font
@@
 		)
 	)
+	(hierarchical_label "DISPLAY3_EN"
+		(shape output)
+		(at 207.01 81.28 0)
+		(effects
+			(font
+				(size 1.27 1.27)
+			)
+			(justify left)
+		)
+	)
 	(hierarchical_label "SCT_CLK"
 		(shape output)
@@
 		(effects
 			(font
+				(size 1.27 1.27)
+			)
+			(justify left)
+		)
+	)
+	(hierarchical_label "DISPLAY5_EN"
+		(shape output)
+		(at 207.01 86.36 0)
+		(effects
+			(font
+				(size 1.27 1.27)
+			)
+			(justify left)
+		)
+	)
+	(hierarchical_label "DISPLAY1_EN"
+		(shape output)
+		(at 207.01 76.2 0)
+		(effects
+			(font
+				(size 1.27 1.27)
+			)
+			(justify left)
+		)
+	)
+	(hierarchical_label "DISPLAY4_EN"
+		(shape output)
+		(at 207.01 83.82 0)
+		(effects
+			(font
