File: KiCad/HostController.kicad_sch (KiCad schematic)
At the start: 4 parts, among them U301 STM32G0B1KCTx, Y301 Crystal_Small

Commit message: work
Parts:
- removed U301: STM32G0B1KCTx, Package_QFP:LQFP-32_7x7mm_P0.8mm, symbol MCU_ST_STM32G0:STM32G0B1KCTx
- added C303, C304: 10p, Capacitor_SMD:C_0603_1608Metric, symbol Device:C
- added C305: 100n, Capacitor_SMD:C_0603_1608Metric, symbol Device:C
- added SW301: Reset, symbol Switch:SW_Push
- added U302: AT24CS01-STUM, Package_TO_SOT_SMD:SOT-23-5, symbol Memory_EEPROM:AT24CS01-STUM
- added U303: STM32G0B1CETx, Package_QFP:LQFP-48_7x7mm_P0.5mm, symbol MCU_ST_STM32G0:STM32G0B1CETx
- Y301: value Crystal_Small -> 24M
Connections:
- net +3.3V: now also U302.4 (VCC), U303.4 (VBAT), U303.6 (VDD)
- net GND: now also C303.1, C304.1, C305.2, SW301.1, U302.2 (GND), U303.7 (VSS)
- net at Y301.1: now also C304.2, U303.9 (PF1)
- net at Y301.2: now also C303.2, U303.8 (PF0)
- new net DISPL_MOSI: U303.44 (PB5)
- new net DISPL_SCK: U303.42 (PB3)
- new net I2C_SCL: U302.1 (SCL), U303.29 (PA9/UCPD1_DBCC1)
- new net I2C_SDA: U302.3 (SDA), U303.32 (PA10/UCPD1_DBCC2)
- new net NRST: C305.1, SW301.2, U303.10 (PF2)
- new net ST67_MISO: U303.17 (PA6)
- new net ST67_MOSI: U303.18 (PA7)
- new net ST67_RX: U303.14 (PA3)
- new net ST67_SCK: U303.12 (PA1)
- new net ST67_TX: U303.13 (PA2)
- new net SWCLK: U303.36 (PA14)
- new net SWDIO: U303.35 (PA13)
Other:
- moved on the sheet: C301, C302, Y301

Commit message: KiCad work
Parts:
- added D301, D302: LED, symbol Device:LED
- added R301, R302: dnp, symbol Device:R
- added SW302, SW303: Reset, symbol Switch:SW_Push
- added U301: INA169, Package_TO_SOT_SMD:SOT-23-5, symbol Amplifier_Current:INA169
Connections:
- net +3.3V: now also R301.1, R302.1
- net GND: now also U302.5 (WP), U303.5 (VREF+)
- net I2C_SCL: now also R302.2
- net I2C_SDA: now also R301.2
- net DISPL_MOSI renamed SCT_SDI
- net DISPL_SCK renamed SCT_CLK
Other:
- moved on the sheet: C301, C302, U302

Commit message: KiCad work
Changed lines of the file:
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@@
+		)
+	)
+	(hierarchical_label "ST67_CHIP_EN"
+		(shape output)
+		(at 210.82 76.2 0)
+		(effects
+			(font
+				(size 1.27 1.27)
+			)
+			(justify left)
 		)
 	)
@@
 		)
 	)
+	(hierarchical_label "ST67_RDY"
+		(shape input)
+		(at 214.63 67.31 0)
+		(effects
+			(font
+				(size 1.27 1.27)
+			)
+			(justify left)
+		)
+	)
 	(hierarchical_label "ST67_RX"
 		(shape input)
@@
 			)
 			(justify right)
+		)
+	)
+	(hierarchical_label "ST67_BOOT"
+		(shape output)
+		(at 210.82 78.74 0)
+		(effects
+			(font
+				(size 1.27 1.27)
+			)
+			(justify left)
 		)
 	)
@@
 		(effects
 			(font
+				(size 1.27 1.27)
+			)
+			(justify left)
+		)
+	)
+	(hierarchical_label "ST67_CS"
+		(shape output)
+		(at 208.28 72.39 0)
+		(effects
+			(font

Commit message: KiCad work
Parts:
- removed SW303: Reset, symbol Switch:SW_Push
- removed U301: INA169, Package_TO_SOT_SMD:SOT-23-5, symbol Amplifier_Current:INA169
- added C18, C306: 100n, Capacitor_SMD:C_0603_1608Metric, symbol Device:C
- added R10, R14, R305, R306: 10k, Resistor_SMD:R_0603_1608Metric, symbol Device:R
- added R303, R304: 2k2, symbol Device:R
- added SW2: SW_Push, Button_Switch_SMD:SW_SPST_PTS645, symbol Switch:SW_Push
- D301: value LED -> LED1
- D302: value LED -> LED2
- SW302: value Reset -> SW_Push; footprint (none) -> Button_Switch_SMD:SW_SPST_PTS645
Connections:
- net GND: now also D301.1 (K), D302.1 (K), SW302.1, C18.2, C306.2, SW2.1
- net at D301.2 (A): now also R303.1
- net at D302.2 (A): now also R304.1
- net at SW302.2: now also R305.2, R306.2
- new net: R10.2, R14.2, SW2.2
- new net +3V3: R10.1, R305.1
- new net LED1: R303.2
- new net LED2: R304.2
- new net SWITCH_1: C18.1, R14.1
- new net SWITCH_2: C306.1, R306.1
Other:
- moved on the sheet: D301

Commit message: KiCad work
Other:
- moved on the sheet: D301, D302, R303, R304
Changed lines of the file:
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@@
 	(wire
 		(pts
-			(xy 85.09 143.51) (xy 85.09 144.78)
+			(xy 90.17 143.51) (xy 90.17 144.78)
 		)
 		(stroke
@@
 	(wire
 		(pts
-			(xy 85.09 129.54) (xy 97.79 129.54)
+			(xy 90.17 129.54) (xy 102.87 129.54)
 		)
 		(stroke
@@
 	(wire
 		(pts
-			(xy 96.52 132.08) (xy 97.79 132.08)
+			(xy 101.6 132.08) (xy 102.87 132.08)
 		)
 		(stroke
@@
 	(wire
 		(pts
-			(xy 85.09 152.4) (xy 85.09 153.67)
+			(xy 90.17 152.4) (xy 90.17 153.67)
 		)
 		(stroke
@@
 	(wire
 		(pts
-			(xy 96.52 143.51) (xy 96.52 144.78)
+			(xy 101.6 143.51) (xy 101.6 144.78)
 		)
 		(stroke
@@
 	(wire
 		(pts
-			(xy 96.52 152.4) (xy 96.52 153.67)
+			(xy 101.6 152.4) (xy 101.6 153.67)
 		)
 		(stroke
@@
 	(wire
 		(pts
-			(xy 96.52 135.89) (xy 96.52 132.08)
+			(xy 101.6 135.89) (xy 101.6 132.08)
 		)
 		(stroke
@@
 	(wire
 		(pts
-			(xy 85.09 135.89) (xy 85.09 129.54)
+			(xy 90.17 135.89) (xy 90.17 129.54)
 		)
 		(stroke
@@
 	)
 	(label "LED2"
-		(at 97.79 132.08 0)
+		(at 102.87 132.08 0)
 		(effects
 			(font
@@
 	)
 	(label "LED1"
-		(at 97.79 129.54 0)
+		(at 102.87 129.54 0)
 		(effects
 			(font
@@
 	(symbol
 		(lib_id "power:GND")
-		(at 85.09 153.67 0)
+		(at 90.17 153.67 0)
 		(unit 1)
 		(exclude_from_sim no)
@@
 		(fields_autoplaced yes)
 		(property "Reference" "#PWR0316"
-			(at 85.09 160.02 0)
+			(at 90.17 160.02 0)
 			(effects
 				(font
@@
 		)
 		(property "Value" "GND"
-			(at 85.09 158.75 0)
+			(at 90.17 158.75 0)
 			(effects
 				(font
@@
 		)
 		(property "Footprint" ""
-			(at 85.09 153.67 0)
+			(at 90.17 153.67 0)
 			(effects
 				(font
@@
 		)
 		(property "Datasheet" ""
-			(at 85.09 153.67 0)
+			(at 90.17 153.67 0)
 			(effects
 				(font
@@
 		)
 		(property "Description" "Power symbol creates a global label with name \"GND\" , ground"
-			(at 85.09 153.67 0)
+			(at 90.17 153.67 0)
 			(effects
 				(font
@@
 	(symbol
 		(lib_id "Device:LED")
-		(at 96.52 148.59 90)
+		(at 101.6 148.59 90)
 		(unit 1)
 		(exclude_from_sim no)
@@
 		(fields_autoplaced yes)
 		(property "Reference" "D302"
-			(at 100.33 148.9074 90)
+			(at 105.41 148.9074 90)
 			(effects
 				(font
@@
 		)
 		(property "Value" "LED2"
-			(at 100.33 151.4474 90)
+			(at 105.41 151.4474 90)
 			(effects
 				(font
@@
 		)
 		(property "Footprint" ""
-			(at 96.52 148.59 0)
+			(at 101.6 148.59 0)
 			(effects
 				(font
@@
 		)
 		(property "Datasheet" "~"
-			(at 96.52 148.59 0)
+			(at 101.6 148.59 0)
 			(effects
 				(font
@@
 		)
 		(property "Description" "Light emitting diode"
-			(at 96.52 148.59 0)
+			(at 101.6 148.59 0)
 			(effects
 				(font
@@
 		)
 		(property "Sim.Pins" "1=K 2=A"
-			(at 96.52 148.59 0)
+			(at 101.6 148.59 0)
 			(effects
 				(font
@@
 	(symbol
 		(lib_id "Device:R")
-		(at 96.52 139.7 180)
+		(at 101.6 139.7 180)
 		(unit 1)
 		(exclude_from_sim no)
@@
 		(fields_autoplaced yes)
 		(property "Reference" "R304"
-			(at 99.06 138.4299 0)
+			(at 104.14 138.4299 0)
 			(effects
 				(font
@@
 		)
 		(property "Value" "2k2"
-			(at 99.06 140.9699 0)
+			(at 104.14 140.9699 0)
 			(effects
 				(font
@@
 		)
 		(property "Footprint" ""
-			(at 98.298 139.7 90)
+			(at 103.378 139.7 90)
 			(effects
 				(font
@@
 		)
 		(property "Datasheet" "~"
-			(at 96.52 139.7 0)
+			(at 101.6 139.7 0)
 			(effects
 				(font
@@
 		)
 		(property "Description" "Resistor"
-			(at 96.52 139.7 0)
+			(at 101.6 139.7 0)
 			(effects
 				(font
@@
 	(symbol
 		(lib_id "Device:R")
-		(at 85.09 139.7 180)
+		(at 90.17 139.7 180)
 		(unit 1)
 		(exclude_from_sim no)
@@
 		(fields_autoplaced yes)
 		(property "Reference" "R303"
-			(at 87.63 138.4299 0)
+			(at 92.71 138.4299 0)
 			(effects
 				(font
@@
 		)
 		(property "Value" "2k2"
-			(at 87.63 140.9699 0)
+			(at 92.71 140.9699 0)
 			(effects
 				(font
@@
 		)
 		(property "Footprint" ""
-			(at 86.868 139.7 90)
+			(at 91.948 139.7 90)
 			(effects
 				(font
@@
 		)
 		(property "Datasheet" "~"
-			(at 85.09 139.7 0)
+			(at 90.17 139.7 0)
 			(effects
 				(font
@@
 		)
 		(property "Description" "Resistor"
-			(at 85.09 139.7 0)
+			(at 90.17 139.7 0)
 			(effects
 				(font
@@
 	(symbol
 		(lib_id "Device:LED")
-		(at 85.09 148.59 90)
+		(at 90.17 148.59 90)
 		(unit 1)
 		(exclude_from_sim no)
@@
 		(fields_autoplaced yes)
 		(property "Reference" "D301"
-			(at 88.9 148.9074 90)
+			(at 93.98 148.9074 90)
 			(effects
 				(font
@@
 		)
 		(property "Value" "LED1"
-			(at 88.9 151.4474 90)
+			(at 93.98 151.4474 90)
 			(effects
 				(font
@@
 		)
 		(property "Footprint" ""
-			(at 85.09 148.59 0)
+			(at 90.17 148.59 0)
 			(effects
 				(font
@@
 		)
 		(property "Datasheet" "~"
-			(at 85.09 148.59 0)
+			(at 90.17 148.59 0)
 			(effects
 				(font
@@
 		)
 		(property "Description" "Light emitting diode"
-			(at 85.09 148.59 0)
+			(at 90.17 148.59 0)
 			(effects
 				(font
@@
 		)
 		(property "Sim.Pins" "1=K 2=A"
-			(at 85.09 148.59 0)
+			(at 90.17 148.59 0)
 			(effects
 				(font
@@
 	(symbol
 		(lib_id "power:GND")
-		(at 96.52 153.67 0)
+		(at 101.6 153.67 0)
 		(unit 1)
 		(exclude_from_sim no)
@@
 		(fields_autoplaced yes)
 		(property "Reference" "#PWR0317"
-			(at 96.52 160.02 0)
+			(at 101.6 160.02 0)
 			(effects
 				(font
@@
 		)
 		(property "Value" "GND"
-			(at 96.52 158.75 0)
+			(at 101.6 158.75 0)
 			(effects
 				(font
@@
 		)
 		(property "Footprint" ""
-			(at 96.52 153.67 0)
+			(at 101.6 153.67 0)
 			(effects
 				(font
@@
 		)
 		(property "Datasheet" ""
-			(at 96.52 153.67 0)
+			(at 101.6 153.67 0)
 			(effects
 				(font
@@
 		)
 		(property "Description" "Power symbol creates a global label with name \"GND\" , ground"
-			(at 96.52 153.67 0)
+			(at 101.6 153.67 0)
 			(effects
 				(font

Commit message: KiCad work
Parts:
- added C308: 100n, Capacitor_SMD:C_0603_1608Metric, symbol Device:C
- added R309: dnp, Resistor_SMD:R_0805_2012Metric, symbol Device:R
- C302, C303, C304: footprint Capacitor_SMD:C_0603_1608Metric -> Capacitor_SMD:C_0805_2012Metric
- D301, D302: footprint (none) -> Diode_SMD:D_0805_2012Metric
- R301, R302: footprint (none) -> Resistor_SMD:R_0805_2012Metric
- R307: renamed from R303; footprint (none) -> Resistor_SMD:R_0805_2012Metric
- R308: renamed from R304; footprint (none) -> Resistor_SMD:R_0805_2012Metric
- SW301: footprint (none) -> Button_Switch_SMD:SW_Tactile_SPST_NO_Straight_CK_PTS636Sx25SMTRLFS
- SW302: footprint Button_Switch_SMD:SW_SPST_PTS645 -> Button_Switch_SMD:SW_Tactile_SPST_NO_Straight_CK_PTS636Sx25SMTRLFS
- SW303: renamed from SW2; footprint Button_Switch_SMD:SW_SPST_PTS645 -> Button_Switch_SMD:SW_Tactile_SPST_NO_Straight_CK_PTS636Sx25SMTRLFS
- Y301: footprint (none) -> Crystal:Crystal_SMD_Abracon_ABM3-2Pin_5.0x3.2mm
- renumbered C18 to C307, R305 to R303, R10 to R304, R306 to R305, R14 to R306, U302 to U301, U303 to U302
Connections:
- net GND: now also C308.2
- new net: C308.1, R309.1

Commit message: KiCad work
Changed lines of the file:
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@@
 	(hierarchical_label "DIS1_EN"
 		(shape output)
-		(at 223.52 114.3 0)
+		(at 204.47 125.73 0)
 		(effects
 			(font
@@
 	(hierarchical_label "~{SCT_LA}"
 		(shape output)
-		(at 223.52 104.14 0)
+		(at 204.47 115.57 0)
 		(effects
 			(font
@@
 	(hierarchical_label "DIS5_EN"
 		(shape output)
-		(at 223.52 124.46 0)
+		(at 204.47 135.89 0)
 		(effects
 			(font
@@
 	(hierarchical_label "~{SCT_EN}"
 		(shape output)
-		(at 223.52 107.95 0)
+		(at 204.47 118.11 0)
 		(effects
 			(font
@@
 	(hierarchical_label "LOW_POWER_ENABLE"
 		(shape output)
-		(at 223.52 129.54 0)
+		(at 204.47 140.97 0)
 		(effects
 			(font
@@
 	(hierarchical_label "DIS4_EN"
 		(shape output)
-		(at 223.52 121.92 0)
+		(at 204.47 133.35 0)
 		(effects
 			(font
@@
 	(hierarchical_label "DIS3_EN"
 		(shape output)
-		(at 223.52 119.38 0)
+		(at 204.47 130.81 0)
 		(effects
 			(font
@@
 	(hierarchical_label "DIS2_EN"
 		(shape output)
-		(at 223.52 116.84 0)
-		(effects
-			(font
+		(at 204.47 128.27 0)
+		(effects
+			(font

Commit message: Work
Parts:
- added R310: x, Resistor_SMD:R_0805_2012Metric, symbol Device:R
Connections:
- net OSC_OUT: now also U302.21 (PB2), U302.9 (PF1), R310.1
- net UCPD_CC1: now also U302.28 (PA8)
- net UCPD_CC2: now also U302.27 (PB15)
- net USB+: now also U302.34 (PA10/PA12)
- net USB-: now also U302.33 (PA9/PA11)
- net at C304.2, Y301.1: now also R310.2; no longer U302.9 (PF1)
- net OSC_IN: now reaches C303.2, U302.8 (PF0), Y301.2
- net DISPLAY2_EN: now reaches U302.37 (PA15)
- net DISPLAY5_EN: now reaches U302.38 (PD0)
- net DISPLAY3_EN: now reaches U302.39 (PD1)
- net DISPLAY4_EN: now reaches U302.40 (PD2)
- net DISPLAY1_EN: now reaches U302.41 (PD3)
Other:
- moved on the sheet: C303, C304, C305, SW301, Y301
