File: KiCad/HostController.kicad_sch (KiCad schematic)
At the start: 26 parts, among them SW301 Reset, SW302 SW_Push, SW303 SW_Push, U301 AT24CS01-STUM, U302 STM32G0B1CETx, Y301 24M

Commit message: KiCad work
Parts:
- added SW304: SW_DIP_x03, Button_Switch_SMD:SW_DIP_SPSTx03_Slide_KingTek_DSHP03TJ_W5.25mm_P1.27mm_JPin, symbol Switch:SW_DIP_x03
Changed lines of the file:
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@@
+	)
+	(symbol
+		(lib_id "Switch:SW_DIP_x03")
+		(at 233.68 125.73 0)
+		(unit 1)
+		(exclude_from_sim no)
+		(in_bom yes)
+		(on_board yes)
+		(dnp no)
+		(fields_autoplaced yes)
+		(property "Reference" "SW304"
+			(at 233.68 115.57 0)
+			(effects
+				(font
+					(size 1.27 1.27)
+				)
+			)
+		)
+		(property "Value" "SW_DIP_x03"
+			(at 233.68 118.11 0)
+			(effects
+				(font
+					(size 1.27 1.27)
+				)
+			)
+		)
+		(property "Footprint" "Button_Switch_SMD:SW_DIP_SPSTx03_Slide_KingTek_DSHP03TJ_W5.25mm_P1.27mm_JPin"
+			(at 233.68 128.27 0)
+			(effects
+				(font
+					(size 1.27 1.27)
+				)
+				(hide yes)
+			)
+		)
+		(property "Datasheet" "~"
+			(at 233.68 128.27 0)
+			(effects
+				(font
+					(size 1.27 1.27)
+				)
+				(hide yes)
+			)
+		)
+		(property "Description" "3x DIP Switch, Single Pole Single Throw (SPST) switch, small symbol"
+			(at 233.68 125.73 0)
+			(effects
+				(font
+					(size 1.27 1.27)
+				)
+				(hide yes)
+			)
+		)
+		(pin "1"
+		)
+		(pin "3"
+		)
+		(pin "2"
+		)
+		(pin "6"
+		)
+		(pin "5"
+		)
+		(pin "4"
+		)
+		(instances
+			(project ""
+				(path "/8561283c-f5b3-4542-8880-7f435c3a9f7c/d62dd27e-49e2-449e-88dd-01d5559c6bc2"
+					(reference "SW304")
+					(unit 1)
+				)
+			)
+		)
 	)
 	(symbol

Commit message: KiCad work
Parts:
- removed SW301: Reset, Button_Switch_SMD:SW_Tactile_SPST_NO_Straight_CK_PTS636Sx25SMTRLFS, symbol Switch:SW_Push
- added TP301: TestPoint, TestPoint:TestPoint_Pad_D1.5mm, symbol Connector:TestPoint
Connections:
- net LOW_POWER_ENABLE: now also U302.47 (PB8)
- net OSC_OUT: no longer U302.21 (PB2)
- net ST67_BOOT: now also U302.20 (PB1)
- net ST67_CHIP_EN: now also U302.11 (PA0)
- net ST67_CS: now also U302.16 (PA5)
- net ST67_RDY: now also U302.15 (PA4)
- net ~{SCT_EN}: now also U302.46 (PB7)
- net ~{SCT_LA}: now also U302.45 (PB6)
- new net OSC_OUT_PIN: TP301.1, U302.21 (PB2)
Changed lines of the file:
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@@
 	)
 	(junction
-		(at 82.55 69.85)
-		(diameter 0)
-		(color 0 0 0 0)
-	)
-	(junction
 		(at 87.63 54.61)
 		(diameter 0)
@@
 	(wire
 		(pts
-			(xy 76.2 69.85) (xy 82.55 69.85)
+			(xy 182.88 78.74) (xy 189.23 78.74)
 		)
 		(stroke
@@
 	(wire
 		(pts
-			(xy 182.88 78.74) (xy 189.23 78.74)
+			(xy 121.92 73.66) (xy 127 73.66)
 		)
 		(stroke
@@
 	(wire
 		(pts
-			(xy 121.92 73.66) (xy 127 73.66)
+			(xy 26.67 151.13) (xy 33.02 151.13)
 		)
 		(stroke
@@
 	(wire
 		(pts
-			(xy 26.67 151.13) (xy 33.02 151.13)
+			(xy 149.86 38.1) (xy 138.43 38.1)
 		)
 		(stroke
@@
 	(wire
 		(pts
-			(xy 149.86 38.1) (xy 138.43 38.1)
+			(xy 125.73 58.42) (xy 127 58.42)
 		)
 		(stroke
@@
 	(wire
 		(pts
-			(xy 125.73 58.42) (xy 127 58.42)
+			(xy 233.68 82.55) (xy 233.68 80.01)
 		)
 		(stroke
@@
 	(wire
 		(pts
-			(xy 233.68 82.55) (xy 233.68 80.01)
+			(xy 182.88 71.12) (xy 189.23 71.12)
 		)
 		(stroke
@@
 	(wire
 		(pts
-			(xy 82.55 82.55) (xy 82.55 83.82)
-		)
-		(stroke
-			(width 0)
-			(type default)
-		)
-	)
-	(wire
-		(pts
 			(xy 36.83 30.48) (xy 36.83 26.67)
 		)
@@
 	(wire
 		(pts
-			(xy 182.88 106.68) (xy 189.23 106.68)
+			(xy 182.88 106.68) (xy 209.55 106.68)
 		)
 		(stroke
@@
 	(wire
 		(pts
-			(xy 82.55 69.85) (xy 95.25 69.85)
+			(xy 182.88 68.58) (xy 189.23 68.58)
+		)
+		(stroke
+			(width 0)
+			(type default)
+		)
+	)
+	(wire
+		(pts
+			(xy 76.2 69.85) (xy 95.25 69.85)
 		)
 		(stroke
@@
 	(wire
 		(pts
+			(xy 182.88 121.92) (xy 189.23 121.92)
+		)
+		(stroke
+			(width 0)
+			(type default)
+		)
+	)
+	(wire
+		(pts
 			(xy 255.27 31.75) (xy 255.27 34.29)
 		)
@@
 	(wire
 		(pts
+			(xy 182.88 104.14) (xy 189.23 104.14)
+		)
+		(stroke
+			(width 0)
+			(type default)
+		)
+	)
+	(wire
+		(pts
 			(xy 182.88 66.04) (xy 189.23 66.04)
 		)
@@
 	(wire
 		(pts
+			(xy 209.55 106.68) (xy 209.55 104.14)
+		)
+		(stroke
+			(width 0)
+			(type default)
+		)
+	)
+	(wire
+		(pts
 			(xy 264.16 31.75) (xy 264.16 34.29)
 		)
@@
 	(wire
 		(pts
+			(xy 182.88 119.38) (xy 189.23 119.38)
+		)
+		(stroke
+			(width 0)
+			(type default)
+		)
+	)
+	(wire
+		(pts
 			(xy 157.48 48.26) (xy 157.48 50.8)
 		)
@@
 	(wire
 		(pts
+			(xy 182.88 116.84) (xy 189.23 116.84)
+		)
+		(stroke
+			(width 0)
+			(type default)
+		)
+	)
+	(wire
+		(pts
+			(xy 182.88 58.42) (xy 189.23 58.42)
+		)
+		(stroke
+			(width 0)
+			(type default)
+		)
+	)
+	(wire
+		(pts
 			(xy 55.88 134.62) (xy 55.88 137.16)
 		)
@@
 	(wire
 		(pts
-			(xy 82.55 69.85) (xy 82.55 72.39)
-		)
-		(stroke
-			(width 0)
-			(type default)
-		)
-	)
-	(wire
-		(pts
 			(xy 33.02 151.13) (xy 39.37 151.13)
 		)
@@
 		)
 	)
-	(label "OSC_OUT"
+	(label "OSC_OUT_PIN"
 		(at 189.23 106.68 0)
 		(effects
@@
 	(hierarchical_label "ST67_CHIP_EN"
 		(shape output)
-		(at 210.82 76.2 0)
+		(at 189.23 58.42 0)
 		(effects
 			(font
@@
 	(hierarchical_label "~{SCT_LA}"
 		(shape output)
-		(at 204.47 115.57 0)
+		(at 189.23 116.84 0)
 		(effects
 			(font
@@
 	(hierarchical_label "ST67_RDY"
 		(shape input)
-		(at 214.63 67.31 0)
+		(at 189.23 68.58 0)
 		(effects
 			(font
@@
 	(hierarchical_label "ST67_BOOT"
 		(shape output)
-		(at 210.82 78.74 0)
+		(at 189.23 104.14 0)
 		(effects
 			(font
@@
 	(hierarchical_label "~{SCT_EN}"
 		(shape output)
-		(at 204.47 118.11 0)
+		(at 189.23 119.38 0)
 		(effects
 			(font
@@
 	(hierarchical_label "LOW_POWER_ENABLE"
 		(shape output)
-		(at 204.47 140.97 0)
+		(at 189.23 121.92 0)
 		(effects
 			(font
@@
 	(hierarchical_label "ST67_CS"
 		(shape output)
-		(at 208.28 72.39 0)
+		(at 189.23 71.12 0)
 		(effects
 			(font
@@
 	)
 	(symbol
-		(lib_id "Switch:SW_Push")
-		(at 82.55 77.47 90)
-		(unit 1)
-		(exclude_from_sim no)
-		(in_bom yes)
-		(on_board yes)
-		(dnp no)
-		(fields_autoplaced yes)
-		(property "Reference" "SW301"
-			(at 83.82 76.1999 90)
-			(effects
-				(font
-					(size 1.27 1.27)
-				)
-				(justify right)
-			)
-		)
-		(property "Value" "Reset"
-			(at 83.82 78.7399 90)
-			(effects
-				(font
-					(size 1.27 1.27)
-				)
-				(justify right)
-			)
-		)
-		(property "Footprint" "Button_Switch_SMD:SW_Tactile_SPST_NO_Straight_CK_PTS636Sx25SMTRLFS"
-			(at 77.47 77.47 0)
-			(effects
-				(font
-					(size 1.27 1.27)
-				)
-				(hide yes)
-			)
-		)
-		(property "Datasheet" "~"
-			(at 77.47 77.47 0)
-			(effects
-				(font
-					(size 1.27 1.27)
-				)
-				(hide yes)
-			)
-		)
-		(property "Description" "Push button switch, generic, two pins"
-			(at 82.55 77.47 0)
-			(effects
-				(font
-					(size 1.27 1.27)
-				)
-				(hide yes)
-			)
-		)
-		(pin "2"
-		)
-		(pin "1"
-		)
-		(instances
-			(project ""
-				(path "/8561283c-f5b3-4542-8880-7f435c3a9f7c/d62dd27e-49e2-449e-88dd-01d5559c6bc2"
-					(reference "SW301")
-					(unit 1)
-				)
-			)
-		)
-	)
-	(symbol
 		(lib_id "Device:R")
 		(at 264.16 38.1 0)
@@
 	)
 	(symbol
+		(lib_id "Connector:TestPoint")
+		(at 209.55 104.14 0)
+		(unit 1)
+		(exclude_from_sim no)
+		(in_bom yes)
+		(on_board yes)
+		(dnp no)
+		(fields_autoplaced yes)
+		(property "Reference" "TP301"
+			(at 212.09 99.5679 0)
+			(effects
+				(font
+					(size 1.27 1.27)
+				)
+				(justify left)
+			)
+		)
+		(property "Value" "TestPoint"
+			(at 212.09 102.1079 0)
+			(effects
+				(font
+					(size 1.27 1.27)
+				)
+				(justify left)
+			)
+		)
+		(property "Footprint" "TestPoint:TestPoint_Pad_D1.5mm"
+			(at 214.63 104.14 0)
+			(effects
+				(font
+					(size 1.27 1.27)
+				)
+				(hide yes)
+			)
+		)
+		(property "Datasheet" "~"
+			(at 214.63 104.14 0)
+			(effects
+				(font
+					(size 1.27 1.27)
+				)
+				(hide yes)
+			)
+		)
+		(property "Description" "test point"
+			(at 209.55 104.14 0)
+			(effects
+				(font
+					(size 1.27 1.27)
+				)
+				(hide yes)
+			)
+		)
+		(pin "1"
+		)
+		(instances
+			(project ""
+				(path "/8561283c-f5b3-4542-8880-7f435c3a9f7c/d62dd27e-49e2-449e-88dd-01d5559c6bc2"
+					(reference "TP301")
+					(unit 1)
+				)
+			)
+		)
+	)
+	(symbol
 		(lib_id "power:GND")
 		(at 95.25 83.82 0)
@@
 					(unit 1)
 				)
-			)
-		)
-	)
-	(symbol
-		(lib_id "power:GND")
-		(at 82.55 83.82 0)
-		(unit 1)
-		(exclude_from_sim no)
-		(in_bom yes)
-		(on_board yes)
-		(dnp no)
-		(fields_autoplaced yes)
-		(property "Reference" "#PWR0313"
-			(at 82.55 90.17 0)
-			(effects
-				(font
-					(size 1.27 1.27)
-				)
-				(hide yes)
-			)
-		)
-		(property "Value" "GND"
-			(at 82.55 88.9 0)
-			(effects
-				(font
-					(size 1.27 1.27)
-				)
-			)
-		)
-		(property "Footprint" ""
-			(at 82.55 83.82 0)
-			(effects
-				(font
-					(size 1.27 1.27)
-				)
-				(hide yes)
-			)
-		)
-		(property "Datasheet" ""
-			(at 82.55 83.82 0)
-			(effects
-				(font
-					(size 1.27 1.27)
-				)
-				(hide yes)
-			)
-		)
-		(property "Description" "Power symbol creates a global label with name \"GND\" , ground"
-			(at 82.55 83.82 0)
-			(effects
-				(font
-					(size 1.27 1.27)
-				)
-				(hide yes)
-			)
-		)
-		(pin "1"
-		)
-		(instances
-			(project "AstroWeather"
-				(path "/8561283c-f5b3-4542-8880-7f435c3a9f7c/d62dd27e-49e2-449e-88dd-01d5559c6bc2"
-					(reference "#PWR0313")
-					(unit 1)
-				)

Commit message: some work
Connections:
- net +3V3 is gone; now on net +3.3V: R303.1, R304.1
- net LED1: now also U302.1 (PC13)
- net LED2: now also U302.48 (PB9)
- net SWITCH_1: now also U302.25 (PB13)
- net SWITCH_2: now also U302.24 (PB12)
Changed lines of the file:
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@@
 	(wire
 		(pts
+			(xy 182.88 132.08) (xy 189.23 132.08)
+		)
+		(stroke
+			(width 0)
+			(type default)
+		)
+	)
+	(wire
+		(pts
 			(xy 62.23 153.67) (xy 62.23 151.13)
 		)
@@
 	(wire
 		(pts
+			(xy 182.88 124.46) (xy 189.23 124.46)
+		)
+		(stroke
+			(width 0)
+			(type default)
+		)
+	)
+	(wire
+		(pts
 			(xy 252.73 53.34) (xy 255.27 53.34)
 		)
@@
 	(wire
 		(pts
+			(xy 182.88 134.62) (xy 189.23 134.62)
+		)
+		(stroke
+			(width 0)
+			(type default)
+		)
+	)
+	(wire
+		(pts
 			(xy 252.73 48.26) (xy 255.27 48.26)
 		)
@@
 	(wire
 		(pts
+			(xy 121.92 91.44) (xy 127 91.44)
+		)
+		(stroke
+			(width 0)
+			(type default)
+		)
+	)
+	(wire
+		(pts
 			(xy 242.57 59.69) (xy 242.57 60.96)
 		)
@@
 		)
 	)
-	(label "LED1"
-		(at 105.41 115.57 0)
+	(label "LED2"
+		(at 189.23 124.46 0)
 		(effects
 			(font
@@
 	)
 	(label "SWITCH_1"
-		(at 90.17 113.03 0)
+		(at 189.23 134.62 0)
 		(effects
 			(font
@@
 	)
 	(label "LED1"
-		(at 105.41 113.03 0)
+		(at 121.92 91.44 180)
 		(effects
 			(font
 				(size 1.27 1.27)
 			)
-			(justify left bottom)
+			(justify right bottom)
 		)
 	)
 	(label "SWITCH_2"
-		(at 90.17 116.84 0)
+		(at 189.23 132.08 0)
 		(effects
 			(font
@@
 	)
 	(symbol
+		(lib_id "power:+3.3V")
+		(at 26.67 127 0)
+		(unit 1)
+		(exclude_from_sim no)
+		(in_bom yes)
+		(on_board yes)
+		(dnp no)
+		(fields_autoplaced yes)
+		(property "Reference" "#PWR0313"
+			(at 26.67 130.81 0)
+			(effects
+				(font
+					(size 1.27 1.27)
+				)
+				(hide yes)
+			)
+		)
+		(property "Value" "+3.3V"
+			(at 26.67 121.92 0)
+			(effects
+				(font
+					(size 1.27 1.27)
+				)
+			)
+		)
+		(property "Footprint" ""
+			(at 26.67 127 0)
+			(effects
+				(font
+					(size 1.27 1.27)
+				)
+				(hide yes)
+			)
+		)
+		(property "Datasheet" ""
+			(at 26.67 127 0)
+			(effects
+				(font
+					(size 1.27 1.27)
+				)
+				(hide yes)
+			)
+		)
+		(property "Description" "Power symbol creates a global label with name \"+3.3V\""
+			(at 26.67 127 0)
+			(effects
+				(font
+					(size 1.27 1.27)
+				)
+				(hide yes)
+			)
+		)
+		(pin "1"
+		)
+		(instances
+			(project "AstroWeather"
+				(path "/8561283c-f5b3-4542-8880-7f435c3a9f7c/d62dd27e-49e2-449e-88dd-01d5559c6bc2"
+					(reference "#PWR0313")
+					(unit 1)
+				)
+			)
+		)
+	)
+	(symbol
 		(lib_id "Switch:SW_Push")
 		(at 55.88 144.78 90)
@@
 	)
 	(symbol
+		(lib_id "power:+3.3V")
+		(at 55.88 127 0)
+		(unit 1)
+		(exclude_from_sim no)
+		(in_bom yes)
+		(on_board yes)
+		(dnp no)
+		(fields_autoplaced yes)
+		(property "Reference" "#PWR0315"
+			(at 55.88 130.81 0)
+			(effects
+				(font
+					(size 1.27 1.27)
+				)
+				(hide yes)
+			)
+		)
+		(property "Value" "+3.3V"
+			(at 55.88 121.92 0)
+			(effects
+				(font
+					(size 1.27 1.27)
+				)
+			)
+		)
+		(property "Footprint" ""
+			(at 55.88 127 0)
+			(effects
+				(font
+					(size 1.27 1.27)
+				)
+				(hide yes)
+			)
+		)
+		(property "Datasheet" ""
+			(at 55.88 127 0)
+			(effects
+				(font
+					(size 1.27 1.27)
+				)
+				(hide yes)
+			)
+		)
+		(property "Description" "Power symbol creates a global label with name \"+3.3V\""
+			(at 55.88 127 0)
+			(effects
+				(font
+					(size 1.27 1.27)
+				)
+				(hide yes)
+			)
+		)
+		(pin "1"
+		)
+		(instances
+			(project "AstroWeather"
+				(path "/8561283c-f5b3-4542-8880-7f435c3a9f7c/d62dd27e-49e2-449e-88dd-01d5559c6bc2"
+					(reference "#PWR0315")
+					(unit 1)
+				)
+			)
+		)
+	)
+	(symbol
 		(lib_id "Connector:TestPoint")
 		(at 209.55 104.14 0)
@@
 	)
 	(symbol
-		(lib_id "EnvSensor-v2-rescue:+3.3V-power")
-		(at 55.88 127 0)
-		(unit 1)
-		(exclude_from_sim no)
-		(in_bom yes)
-		(on_board yes)
-		(dnp no)
-		(property "Reference" "#PWR0316"
-			(at 55.88 130.81 0)
-			(effects
-				(font
-					(size 1.27 1.27)
-				)
-				(hide yes)
-			)
-		)
-		(property "Value" "+3V3"
-			(at 56.261 122.6058 0)
-			(effects
-				(font
-					(size 1.27 1.27)
-				)
-			)
-		)
-		(property "Footprint" ""
-			(at 55.88 127 0)
-			(effects
-				(font
-					(size 1.27 1.27)
-				)
-				(hide yes)
-			)
-		)
-		(property "Datasheet" ""
-			(at 55.88 127 0)
-			(effects
-				(font
-					(size 1.27 1.27)
-				)
-				(hide yes)
-			)
-		)
-		(property "Description" ""
-			(at 55.88 127 0)
-			(effects
-				(font
-					(size 1.27 1.27)
-				)
-				(hide yes)
-			)
-		)
-		(pin "1"
-		)
-		(instances
-			(project "AstroWeather"
-				(path "/8561283c-f5b3-4542-8880-7f435c3a9f7c/d62dd27e-49e2-449e-88dd-01d5559c6bc2"
-					(reference "#PWR0316")
-					(unit 1)
-				)
-			)
-		)
-	)
-	(symbol
 		(lib_id "power:GND")
 		(at 62.23 153.67 0)
@@
 					(unit 1)
 				)
-			)
-		)
-	)
-	(symbol
-		(lib_id "EnvSensor-v2-rescue:+3.3V-power")
-		(at 26.67 127 0)
-		(unit 1)
-		(exclude_from_sim no)
-		(in_bom yes)
-		(on_board yes)
-		(dnp no)
-		(property "Reference" "#PWR0315"
-			(at 26.67 130.81 0)
-			(effects
-				(font
-					(size 1.27 1.27)
-				)
-				(hide yes)
-			)
-		)
-		(property "Value" "+3V3"
-			(at 27.051 122.6058 0)
-			(effects
-				(font
-					(size 1.27 1.27)
-				)
-			)
-		)
-		(property "Footprint" ""
-			(at 26.67 127 0)
-			(effects
-				(font
-					(size 1.27 1.27)
-				)
-				(hide yes)
-			)
-		)
-		(property "Datasheet" ""
-			(at 26.67 127 0)
-			(effects
-				(font
-					(size 1.27 1.27)
-				)
-				(hide yes)
-			)
-		)
-		(property "Description" ""
-			(at 26.67 127 0)
-			(effects
-				(font
-					(size 1.27 1.27)
-				)
-				(hide yes)
-			)
-		)
-		(pin "1"
-		)
-		(instances
-			(project "AstroWeather"
-				(path "/8561283c-f5b3-4542-8880-7f435c3a9f7c/d62dd27e-49e2-449e-88dd-01d5559c6bc2"
-					(reference "#PWR0315")
-					(unit 1)
-				)

Commit message: KiCad work
Parts:
- removed SW304: SW_DIP_x03, Button_Switch_SMD:SW_DIP_SPSTx03_Slide_KingTek_DSHP03TJ_W5.25mm_P1.27mm_JPin, symbol Switch:SW_DIP_x03
- added C309: 100n, Capacitor_SMD:C_0805_2012Metric, symbol Device:C
- added JP301: A0, Jumper:SolderJumper-3_P1.3mm_Open_RoundedPad1.0x1.5mm, symbol Jumper:SolderJumper_3_Open
- added JP302: A1, Jumper:SolderJumper-3_P1.3mm_Open_RoundedPad1.0x1.5mm, symbol Jumper:SolderJumper_3_Open
- added JP303: A2, Jumper:SolderJumper-3_P1.3mm_Open_RoundedPad1.0x1.5mm, symbol Jumper:SolderJumper_3_Open
- added R311: ?, Resistor_SMD:R_0805_2012Metric, symbol Device:R
- C308: footprint Capacitor_SMD:C_0603_1608Metric -> Capacitor_SMD:C_0805_2012Metric
- R309: value dnp -> ?
Connections:
- net +3.3V: now also JP301.1 (A), JP302.1 (A), JP303.1 (A)
- net CURRENT_SENSE: now also R311.2
- net GND: now also R307.1, R308.1, C309.2, JP301.3 (B), JP302.3 (B), JP303.3 (B); no longer D301.1 (K), D302.1 (K)
- net LED1: now also D301.2 (A); no longer R307.2
- net LED2: now also D302.2 (A); no longer R308.2
- net VOLTAGE_SENSE: now also R309.2
- net VOLTAGE_SENS_FLTR: now reaches C308.1, R309.1
- net VOLTAGE_SENS_FLTR: now also U302.31 (PC7)
- net ADDR_0: now reaches U302.22 (PB10)
- net ADDR_0: now also JP301.2 (C)
- net ADDR_1: now reaches U302.23 (PB11)
- net ADDR_1: now also JP302.2 (C)
- net ADDR_2: now reaches U302.26 (PB14)
- net ADDR_2: now also JP303.2 (C)
- net CURRENT_SENSE_FLTR: now reaches U302.30 (PC6)
- net CURRENT_SENSE_FLTR: now also C309.1, R311.1
- new net: D302.1 (K), R308.2
- new net: D301.1 (K), R307.2
Other:
- moved on the sheet: C308, D301, D302, R307, R308, R309

Commit message: KiCad work
Parts:
- renumbered C308 to C306, C309 to C307, C306 to C308, C307 to C309, R310 to R303, R309 to R304, R311 to R305, R303 to R306, R304 to R307, R305 to R308, R306 to R309, R307 to R310, R308 to R311, SW302 to SW301, SW303 to SW302
