File: KiCad/HostController.kicad_sch (KiCad schematic)
At the start: 31 parts, among them SW301 SW_Push, SW302 SW_Push, U301 AT24CS01-STUM, U302 STM32G0B1CETx, Y301 24M

Commit message: KiCad work
Parts:
- removed Y301: 24M, Crystal:Crystal_SMD_Abracon_ABM3-2Pin_5.0x3.2mm, symbol Device:Crystal_Small
- added Y301: Crystal_GND24_Small, Crystal:Crystal_SMD_Abracon_ABM3B-4Pin_5.0x3.2mm, symbol Device:Crystal_GND24_Small
- C303, C304: value 10p -> 20p
- C306, C307: value 100n -> 1u
- R304, R305: value ? -> 100k
Connections:
- net GND: now also Y301.2 (G), Y301.4 (G)
- net OSC_IN: now also Y301.1
- net at C304.2, R303.2: now also Y301.3
Changed lines of the file:
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@@
 	)
 	(junction
+		(at 76.2 59.69)
+		(diameter 0)
+		(color 0 0 0 0)
+	)
+	(junction
 		(at 157.48 48.26)
 		(diameter 0)
@@
 	(wire
 		(pts
+			(xy 76.2 66.04) (xy 76.2 59.69)
+		)
+		(stroke
+			(width 0)
+			(type default)
+		)
+	)
+	(wire
+		(pts
 			(xy 182.88 106.68) (xy 209.55 106.68)
 		)
@@
 	(wire
 		(pts
-			(xy 76.2 69.85) (xy 95.25 69.85)
+			(xy 91.44 69.85) (xy 95.25 69.85)
 		)
 		(stroke
@@
 	(wire
 		(pts
+			(xy 76.2 54.61) (xy 76.2 59.69)
+		)
+		(stroke
+			(width 0)
+			(type default)
+		)
+	)
+	(wire
+		(pts
 			(xy 255.27 31.75) (xy 255.27 34.29)
 		)
@@
 	(wire
 		(pts
+			(xy 74.93 59.69) (xy 76.2 59.69)
+		)
+		(stroke
+			(width 0)
+			(type default)
+		)
+	)
+	(wire
+		(pts
+			(xy 76.2 59.69) (xy 85.09 59.69)
+		)
+		(stroke
+			(width 0)
+			(type default)
+		)
+	)
+	(wire
+		(pts
 			(xy 182.88 114.3) (xy 189.23 114.3)
 		)
@@
 	(hierarchical_label "NRST"
 		(shape input)
-		(at 76.2 69.85 180)
+		(at 91.44 69.85 180)
 		(effects
 			(font
@@
 			)
 		)
-		(property "Value" "100n"
+		(property "Value" "1u"
 			(at 242.57 90.1699 0)
 			(effects
@@
 	)
 	(symbol
-		(lib_id "Device:Crystal_Small")
-		(at 87.63 59.69 90)
-		(unit 1)
-		(exclude_from_sim no)
-		(in_bom yes)
-		(on_board yes)
-		(dnp no)
-		(fields_autoplaced yes)
-		(property "Reference" "Y301"
-			(at 90.17 58.4199 90)
-			(effects
-				(font
-					(size 1.27 1.27)
-				)
-				(justify right)
-			)
-		)
-		(property "Value" "24M"
-			(at 90.17 60.9599 90)
-			(effects
-				(font
-					(size 1.27 1.27)
-				)
-				(justify right)
-			)
-		)
-		(property "Footprint" "Crystal:Crystal_SMD_Abracon_ABM3-2Pin_5.0x3.2mm"
-			(at 87.63 59.69 0)
-			(effects
-				(font
-					(size 1.27 1.27)
-				)
-				(hide yes)
-			)
-		)
-		(property "Datasheet" "~"
-			(at 87.63 59.69 0)
-			(effects
-				(font
-					(size 1.27 1.27)
-				)
-				(hide yes)
-			)
-		)
-		(property "Description" "Two pin crystal, small symbol"
-			(at 87.63 59.69 0)
-			(effects
-				(font
-					(size 1.27 1.27)
-				)
-				(hide yes)
-			)
-		)
-		(pin "2"
-		)
-		(pin "1"
-		)
-		(instances
-			(project ""
-				(path "/8561283c-f5b3-4542-8880-7f435c3a9f7c/d62dd27e-49e2-449e-88dd-01d5559c6bc2"
-					(reference "Y301")
-					(unit 1)
-				)
-			)
-		)
-	)
-	(symbol
 		(lib_id "Device:R")
 		(at 97.79 66.04 270)
@@
 	)
 	(symbol
+		(lib_id "Device:Crystal_GND24_Small")
+		(at 87.63 59.69 270)
+		(unit 1)
+		(exclude_from_sim no)
+		(in_bom yes)
+		(on_board yes)
+		(dnp no)
+		(fields_autoplaced yes)
+		(property "Reference" "Y301"
+			(at 90.17 58.4199 90)
+			(effects
+				(font
+					(size 1.27 1.27)
+				)
+				(justify left)
+			)
+		)
+		(property "Value" "Crystal_GND24_Small"
+			(at 90.17 60.9599 90)
+			(effects
+				(font
+					(size 1.27 1.27)
+				)
+				(justify left)
+			)
+		)
+		(property "Footprint" "Crystal:Crystal_SMD_Abracon_ABM3B-4Pin_5.0x3.2mm"
+			(at 87.63 59.69 0)
+			(effects
+				(font
+					(size 1.27 1.27)
+				)
+				(hide yes)
+			)
+		)
+		(property "Datasheet" "~"
+			(at 87.63 59.69 0)
+			(effects
+				(font
+					(size 1.27 1.27)
+				)
+				(hide yes)
+			)
+		)
+		(property "Description" "Four pin crystal, GND on pins 2 and 4, small symbol"
+			(at 87.63 59.69 0)
+			(effects
+				(font
+					(size 1.27 1.27)
+				)
+				(hide yes)
+			)
+		)
+		(property private "KLC_S3.3" "The rectangle is not a symbol body but a graphical element"
+			(at 77.47 59.69 0)
+			(show_name yes)
+			(effects
+				(font
+					(size 1.27 1.27)
+				)
+				(hide yes)
+			)
+		)
+		(property private "KLC_S4.1" "Some pins are on 50mil grid to make the symbol small"
+			(at 74.93 59.69 0)
+			(show_name yes)
+			(effects
+				(font
+					(size 1.27 1.27)
+				)
+				(hide yes)
+			)
+		)
+		(pin "4"
+		)
+		(pin "1"
+		)
+		(pin "3"
+		)
+		(pin "2"
+		)
+		(instances
+			(project ""
+				(path "/8561283c-f5b3-4542-8880-7f435c3a9f7c/d62dd27e-49e2-449e-88dd-01d5559c6bc2"
+					(reference "Y301")
+					(unit 1)
+				)
+			)
+		)
+	)
+	(symbol
 		(lib_id "power:+3.3V")
 		(at 26.67 127 0)
@@
 			)
 		)
-		(property "Value" "100n"
+		(property "Value" "1u"
 			(at 251.46 111.7599 0)
 			(effects
@@
 		(dnp no)
 		(property "Reference" "C304"
-			(at 81.28 58.42 90)
+			(at 81.28 72.136 90)
 			(effects
 				(font
@@
 			)
 		)
-		(property "Value" "10p"
-			(at 81.28 60.96 90)
+		(property "Value" "20p"
+			(at 81.28 69.85 90)
 			(effects
 				(font
@@
 	)
 	(symbol
-		(lib_id "power:GND")
-		(at 76.2 66.04 270)
-		(unit 1)
-		(exclude_from_sim no)
-		(in_bom yes)
-		(on_board yes)
-		(dnp no)
-		(fields_autoplaced yes)
-		(property "Reference" "#PWR0312"
-			(at 69.85 66.04 0)
-			(effects
-				(font
-					(size 1.27 1.27)
-				)
-				(hide yes)
-			)
-		)
-		(property "Value" "GND"
-			(at 72.39 66.0399 90)
-			(effects
-				(font
-					(size 1.27 1.27)
-				)
-				(justify right)
-			)
-		)
-		(property "Footprint" ""
-			(at 76.2 66.04 0)
-			(effects
-				(font
-					(size 1.27 1.27)
-				)
-				(hide yes)
-			)
-		)
-		(property "Datasheet" ""
-			(at 76.2 66.04 0)
-			(effects
-				(font
-					(size 1.27 1.27)
-				)
-				(hide yes)
-			)
-		)
-		(property "Description" "Power symbol creates a global label with name \"GND\" , ground"
-			(at 76.2 66.04 0)
-			(effects
-				(font
-					(size 1.27 1.27)
-				)
-				(hide yes)
-			)
-		)
-		(pin "1"
-		)
-		(instances
-			(project "AstroWeather"
-				(path "/8561283c-f5b3-4542-8880-7f435c3a9f7c/d62dd27e-49e2-449e-88dd-01d5559c6bc2"
-					(reference "#PWR0312")
-					(unit 1)
-				)
-			)
-		)
-	)
-	(symbol
 		(lib_id "Device:C")
 		(at 81.28 54.61 90)
@@
 			)
 		)
-		(property "Value" "10p"
+		(property "Value" "20p"
 			(at 81.28 49.53 90)
 			(effects
@@
 			)
 		)
-		(property "Value" "?"
+		(property "Value" "100k"
 			(at 254 100.33 90)
 			(effects
@@
 	(symbol
 		(lib_id "power:GND")
-		(at 76.2 54.61 270)
+		(at 74.93 59.69 270)
 		(unit 1)
 		(exclude_from_sim no)
@@
 		(fields_autoplaced yes)
 		(property "Reference" "#PWR0309"
-			(at 69.85 54.61 0)
+			(at 68.58 59.69 0)
 			(effects
 				(font
@@
 		)
 		(property "Value" "GND"
-			(at 72.39 54.6099 90)
+			(at 71.12 59.6899 90)
 			(effects
 				(font
@@
 		)
 		(property "Footprint" ""
-			(at 76.2 54.61 0)
+			(at 74.93 59.69 0)
 			(effects
 				(font
@@
 		)
 		(property "Datasheet" ""
-			(at 76.2 54.61 0)
+			(at 74.93 59.69 0)
 			(effects
 				(font
@@
 		)
 		(property "Description" "Power symbol creates a global label with name \"GND\" , ground"
-			(at 76.2 54.61 0)
+			(at 74.93 59.69 0)
 			(effects
 				(font
@@
 			)
 		)
-		(property "Value" "?"
+		(property "Value" "100k"
 			(at 245.11 78.74 90)
 			(effects
