File: KiCad/HostController.kicad_sch (KiCad schematic)
At the start: 31 parts, among them SW301 SW_Push, SW302 SW_Push, U301 AT24CS01-STUM, U302 STM32G0B1CETx, Y301 Crystal_GND24_Small

Commit message: KiCad work
Other:
- note added: "25.07.2026 - 22p"
Changed lines of the file:
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@@
 	(generator_version "9.0")
 	(paper "A4")
+	(text "25.07.2026 - 22p"
+		(exclude_from_sim no)
+		(at 81.534 42.418 0)
+		(effects
+			(font
+				(size 1.27 1.27)
+			)
+		)
+	)
 	(junction
 		(at 33.02 151.13)
