File: KiCad/HostController.kicad_sch (KiCad schematic)
At the start: 31 parts, among them SW301 SW_Push, SW302 SW_Push, U301 AT24CS01-STUM, U302 STM32G0B1CETx, Y301 Crystal_GND24_Small

Commit message: 24AA01 EEPROM driver and console probe commands
Add Device::Eeprom24AA01 for the 24AA01T-I/OT settings EEPROM on I2C1,
with page-aware writes and internal write-cycle (t_WC) ack polling, plus
'eeprom probe/scan/read/write/erase/dump' console commands to bring it up.

Verified on hardware: the chip answers at 0x50 (aliasing to 0x57, since
its address pins are not bonded), page-straddling writes read back exact,
and a full erase and 128-byte dump both complete.

Bringing the bus up needed 2.2k pull-up resistors on SCL/SDA, which were
missing. Without them the lines could never be released high, so the
peripheral latched BUSY on its first START and no device ever answered.
The resistors are sized for the eventual bus: one EEPROM plus up to ten
external boards is roughly 300-450 pF, where 4.7k would exceed the 1 us
rise time that 100 kHz standard mode allows.

Also here:
- Restore Core/Src/main.c and stm32g0xx_hal_msp.c to stock CubeMX output.
  An earlier iteration configured the I2C pull-ups and timing directly in
  these generated files, which the stm32-development skill does not allow
  even inside USER CODE markers; the pull-up and speed settings now come
  from the .ioc.
- Parse eeprom command offsets and lengths as hex, so an address read off
  a dump line can be typed straight back in. They were decimal, which made
  'eeprom read 70' silently mean offset 0x46.
- Size the driver's timeouts for a slow bus. A 2 ms ack poll was too tight
  and failed mid-erase during bring-up at reduced clock.

Co-Authored-By: Claude Opus 5 <noreply@anthropic.com>
Other:
- note added: "Using 2.2k because ~10 board + 1 eeprom chip"
Changed lines of the file:
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@@
 	(generator_version "9.0")
 	(paper "A4")
+	(text "Using 2.2k because ~10 board + 1 eeprom chip"
+		(exclude_from_sim no)
+		(at 264.16 20.066 0)
+		(effects
+			(font
+				(size 1.27 1.27)
+			)
+		)
+	)
 	(text "25.07.2026 - 22p"
 		(exclude_from_sim no)
