File: KiCad/AstroWeather.kicad_pcb (KiCad board)
At the start: 2 copper layers, 243 x 28 mm, 41 parts, among them Q501 IRLML2502, Q502 Si2365EDS, Q503 Si2365EDS, Q504 Si2365EDS, Q505 Si2365EDS, Q506 Si2365EDS, U301 STM32G0B1KCTx, U501 SCT2024, U502 MCP6006T-E/OT, U503 LFD028BUE-103A, U504 LFD028BUE-103A, U505 LFD028BUE-103A, U506 LFD028BUE-103A, U507 KW3-281AVA, U508 KW3-281AVA, U509 KW3-281AVA, U510 KW3-281AVA

Commit message: KiCad work
Parts:
- removed U301: STM32G0B1KCTx, Package_QFP:LQFP-32_7x7mm_P0.8mm
- added C301: 100n, Capacitor_SMD:C_0603_1608Metric, F.Cu at (66.3, 25.7)
- added C302: 4u7, Capacitor_SMD:C_0603_1608Metric, F.Cu at (97.2, 23.0)
- added C303: 10p, Capacitor_SMD:C_0603_1608Metric, F.Cu at (97.2, 25.5)
- added C304: 10p, Capacitor_SMD:C_0603_1608Metric, F.Cu at (97.2, 28.0)
- added C305: 100n, Capacitor_SMD:C_0603_1608Metric, F.Cu at (97.2, 30.5)
- added C501: 1u, Capacitor_SMD:C_0805_2012Metric, F.Cu at (60.0, 25.9)
- added C502: 4u7, Capacitor_SMD:C_0805_2012Metric, F.Cu at (60.0, 28.9)
- added C503: 10p, Capacitor_SMD:C_0805_2012Metric, F.Cu at (60.0, 32.0)
- added C504: 10u, Capacitor_SMD:C_0805_2012Metric, F.Cu at (60.0, 35.0)
- added C505: 10p, Capacitor_SMD:C_0805_2012Metric, F.Cu at (60.0, 38.0)
- added C506: 4u7, Capacitor_SMD:C_0805_2012Metric, F.Cu at (60.0, 41.0)
- added C507: 1u, Capacitor_SMD:C_0805_2012Metric, F.Cu at (60.0, 44.0)
- added Q507: IRLML2502, Package_TO_SOT_SMD:SOT-23, F.Cu at (41.1, 40.0)
- added U302: AT24CS01-STUM, Package_TO_SOT_SMD:SOT-23-5, F.Cu at (86.4, 35.5)
- added U303: STM32G0B1CETx, Package_QFP:LQFP-48_7x7mm_P0.5mm, B.Cu at (65.8, 66.2)
- added U511: MCP6006T-E/OT, Package_TO_SOT_SMD:SOT-23-5, F.Cu at (41.2, 35.6)
- added U512: SCT2024, Package_SO:SSOP-24_3.9x8.7mm_P0.635mm, B.Cu at (34.6, 38.3)
Connections:
- D502 pad 1: unconnected-(D502-K-Pad1) -> /Display/LINE1_1
- D502 pad 2: unconnected-(D502-A-Pad2) -> Net-(D502-A)
- D503 pad 1: unconnected-(D503-K-Pad1) -> /Display/LINE1_2
- D503 pad 2: unconnected-(D503-A-Pad2) -> Net-(D502-A)
- D504 pad 1: unconnected-(D504-K-Pad1) -> /Display/LINE1_3
- D504 pad 2: unconnected-(D504-A-Pad2) -> Net-(D502-A)
- D505 pad 1: unconnected-(D505-K-Pad1) -> /Display/LINE1_4
- D505 pad 2: unconnected-(D505-A-Pad2) -> Net-(D502-A)
- D506 pad 1: unconnected-(D506-K-Pad1) -> /Display/LINE1_5
- D506 pad 2: unconnected-(D506-A-Pad2) -> Net-(D502-A)
- D507 pad 1: unconnected-(D507-K-Pad1) -> /Display/LINE1_6
- D507 pad 2: unconnected-(D507-A-Pad2) -> Net-(D502-A)
- D508 pad 1: unconnected-(D508-K-Pad1) -> /Display/LINE1_7
- D508 pad 2: unconnected-(D508-A-Pad2) -> Net-(D502-A)
- D509 pad 1: unconnected-(D509-K-Pad1) -> /Display/LINE1_8
- D509 pad 2: unconnected-(D509-A-Pad2) -> Net-(D502-A)
- D510 pad 1: unconnected-(D510-K-Pad1) -> /Display/LINE1_9
- D510 pad 2: unconnected-(D510-A-Pad2) -> Net-(D502-A)
- D511 pad 1: unconnected-(D511-K-Pad1) -> /Display/LINE1_10
- D511 pad 2: unconnected-(D511-A-Pad2) -> Net-(D502-A)
- D512 pad 1: unconnected-(D512-K-Pad1) -> /Display/LINE1_11
- D512 pad 2: unconnected-(D512-A-Pad2) -> Net-(D502-A)
- D513 pad 1: unconnected-(D513-K-Pad1) -> /Display/LINE1_12
- D513 pad 2: unconnected-(D513-A-Pad2) -> Net-(D502-A)
- D514 pad 1: unconnected-(D514-K-Pad1) -> /Display/LINE1_13
- D514 pad 2: unconnected-(D514-A-Pad2) -> Net-(D502-A)
- D515 pad 1: unconnected-(D515-K-Pad1) -> /Display/LINE1_14
- D515 pad 2: unconnected-(D515-A-Pad2) -> Net-(D502-A)
- D516 pad 1: unconnected-(D516-K-Pad1) -> /Display/LINE1_15
- D516 pad 2: unconnected-(D516-A-Pad2) -> Net-(D502-A)
- D517 pad 1: unconnected-(D517-K-Pad1) -> /Display/LINE1_16
- D517 pad 2: unconnected-(D517-A-Pad2) -> Net-(D502-A)
- D518 pad 1: unconnected-(D518-K-Pad1) -> /Display/LINE1_17
- D518 pad 2: unconnected-(D518-A-Pad2) -> Net-(D502-A)
- D519 pad 1: unconnected-(D519-K-Pad1) -> /Display/LINE1_18
- D519 pad 2: unconnected-(D519-A-Pad2) -> Net-(D502-A)
- D520 pad 1: unconnected-(D520-K-Pad1) -> /Display/LINE1_19
- D520 pad 2: unconnected-(D520-A-Pad2) -> Net-(D502-A)
- D521 pad 1: unconnected-(D521-K-Pad1) -> /Display/LINE1_20
- D521 pad 2: unconnected-(D521-A-Pad2) -> Net-(D502-A)
- D522 pad 1: unconnected-(D522-K-Pad1) -> /Display/LINE1_21
- D522 pad 2: unconnected-(D522-A-Pad2) -> Net-(D502-A)
- D523 pad 1: unconnected-(D523-K-Pad1) -> /Display/LINE1_22
- D523 pad 2: unconnected-(D523-A-Pad2) -> Net-(D502-A)
- D524 pad 1: unconnected-(D524-K-Pad1) -> /Display/LINE1_23
- D524 pad 2: unconnected-(D524-A-Pad2) -> Net-(D502-A)
- D525 pad 1: unconnected-(D525-K-Pad1) -> /Display/LINE1_24
- D525 pad 2: unconnected-(D525-A-Pad2) -> Net-(D502-A)
- Q502 pad 3: Net-(Q502-D) -> Net-(D502-A)
- U503 pad 1: Net-(Q502-D) -> Net-(D502-A)
- U504 pad 1: Net-(Q502-D) -> Net-(D502-A)

Commit message: KiCad work
Parts:
- removed D502, D503, D504, D505, D506, D507, D508, D509, D510, D511, D512, D513, D514, D515, D516, D517, D518, D519, D520, D521, D522, D523, D524, D525: LED, LED_THT:LED_D3.0mm
- removed the Q501 at (96.4, 68.7)
- removed the U505 at (199.6, 56.2)
- removed the U507 at (229.3, 56.2)
- added C101: 100n, Capacitor_SMD:C_0603_1608Metric, F.Cu at (84.7, -32.6)
- added C201: 10u, Capacitor_SMD:C_0805_2012Metric, F.Cu at (130.5, -22.3)
- added C202: 10u, Capacitor_SMD:C_0805_2012Metric, F.Cu at (130.5, -19.3)
- added C203: 10u, Capacitor_SMD:C_0805_2012Metric, F.Cu at (130.5, -16.2)
- added C204: 5p1, Capacitor_SMD:C_0805_2012Metric, F.Cu at (130.5, -13.2)
- added C205: 5p1, Capacitor_SMD:C_0805_2012Metric, F.Cu at (130.5, -10.2)
- added C206: 100n, Capacitor_SMD:C_0201_0603Metric, F.Cu at (129.5, -4.90)
- added C306: 100n, Capacitor_SMD:C_0603_1608Metric, F.Cu at (63.4, -7.87)
- added C307: 100n, Capacitor_SMD:C_0603_1608Metric, F.Cu at (63.4, -5.36)
- added C401: 100n, Capacitor_SMD:C_0603_1608Metric, F.Cu at (83.0, -2.62)
- added C402: 4u7, Capacitor_SMD:C_0805_2012Metric, F.Cu at (83.2, 2.65)
- added C403: 100n, Capacitor_SMD:C_0603_1608Metric, F.Cu at (83.0, -0.11)
- added C508: 4u7, Capacitor_SMD:C_0805_2012Metric, F.Cu at (100.0, -50.0)
- added C509: 1u, Capacitor_SMD:C_0805_2012Metric, F.Cu at (100.0, -47.0)
- added C510: 4u7, Capacitor_SMD:C_0805_2012Metric, F.Cu at (100.0, -44.0)
- added C601: 100n, Capacitor_SMD:C_0201_0603Metric, F.Cu at (109.1, -6.95)
- added C602: 10u, Capacitor_SMD:C_0805_2012Metric, F.Cu at (105.7, -13.4)
- added C603: 100n, Capacitor_SMD:C_0603_1608Metric, F.Cu at (109.2, -16.6)
- added C604: 22u, Capacitor_SMD:C_1206_3216Metric, F.Cu at (100.6, -13.2)
- added C605: 22u, Capacitor_SMD:C_1206_3216Metric, F.Cu at (100.6, -9.90)
- added C606: 4u7, Capacitor_SMD:C_0805_2012Metric, F.Cu at (105.7, -10.4)
- added C607: 1u, Capacitor_SMD:C_0805_2012Metric, F.Cu at (105.7, -7.40)
- added C608: 47p, Capacitor_SMD:C_0805_2012Metric, F.Cu at (105.7, -4.39)
- added D101: D_TVS, Diode_SMD:D_SOD-323, F.Cu at (93.5, -44.5)
- added D102: D_TVS, Diode_SMD:D_SOD-323, F.Cu at (93.5, -41.6)
- added D301: LED1, Diode_SMD:D_0805_2012Metric, F.Cu at (67.6, 4.20)
- added D302: LED2, Diode_SMD:D_0805_2012Metric, F.Cu at (67.6, 7.24)
- added D501: 1.5V-2V (short), Diode_SMD:D_SMA, F.Cu at (128.0, -30.9)
- added J101: OUTPUT, Connector_PinSocket_2.54mm:PinSocket_1x21_P2.54mm_Horizontal, F.Cu at (164.4, 52.4)
- added J102: I2C, Connector_PinHeader_2.54mm:PinHeader_1x04_P2.54mm_Vertical, F.Cu at (42.5, 76.0)
- added J103: SWD, Connector_JST:JST_PH_S6B-PH-SM4-TB_1x06-1MP_P2.00mm_Horizontal, F.Cu at (50.4, 52.9)
- added J104: AUX_POWER, Connector_PinSocket_2.54mm:PinSocket_1x02_P2.54mm_Vertical, F.Cu at (89.0, -43.7)
- added J105: INPUT, Connector_PinHeader_2.54mm:PinHeader_1x21_P2.54mm_Horizontal, F.Cu at (167.2, 75.0)
- added J106: POWER_SELECT, Connector_PinSocket_2.54mm:PinSocket_1x03_P2.54mm_Vertical, F.Cu at (84.4, -43.7)
- added J107: USB_C_Receptacle_USB2.0_14P, Connector_USB:USB_C_Receptacle_GCT_USB4135-GF-A_6P_TopMnt_Horizontal, F.Cu at (105.5, 76.0)
- added L601: 6u8, Inductor_SMD:L_7.3x7.3_H4.5, F.Cu at (134.8, 100.0)
- added Q506: BC847, Package_TO_SOT_SMD:SOT-23, F.Cu at (61.1, 60.0)
- added Q508: BC847, Package_TO_SOT_SMD:SOT-23, F.Cu at (99.1, 69.0)
- added Q509: BC847, Package_TO_SOT_SMD:SOT-23, F.Cu at (177.1, 51.0)
- added Q701: IRLML2502, Package_TO_SOT_SMD:SOT-23, F.Cu at (120.5, 3.35)
- added R101: 0.05, Resistor_SMD:R_1206_3216Metric, F.Cu at (89.5, -37.2)
- added R201: 33k, Resistor_SMD:R_0805_2012Metric, F.Cu at (130.5, -7.25)
- added R301: dnp, Resistor_SMD:R_0805_2012Metric, F.Cu at (67.6, -7.65)
- added R302: dnp, Resistor_SMD:R_0805_2012Metric, F.Cu at (67.6, -4.70)
- added R303: 10k, Resistor_SMD:R_0603_1608Metric, F.Cu at (63.4, -2.85)
- added R304: 10k, Resistor_SMD:R_0603_1608Metric, F.Cu at (63.4, -0.34)
- added R305: 10k, Resistor_SMD:R_0603_1608Metric, F.Cu at (63.4, 2.17)
- added R306: 10k, Resistor_SMD:R_0603_1608Metric, F.Cu at (63.4, 4.68)
- added R307: 2k2, Resistor_SMD:R_0805_2012Metric, F.Cu at (67.6, -1.75)
- added R308: 2k2, Resistor_SMD:R_0805_2012Metric, F.Cu at (67.6, 1.20)
- added R501: 10, Resistor_SMD:R_0805_2012Metric, F.Cu at (109.3, -42.1)
- added R502: 1k, Resistor_SMD:R_0805_2012Metric, F.Cu at (109.3, -39.1)
- added R503: dnp, Resistor_SMD:R_0805_2012Metric, F.Cu at (109.3, -36.2)
- added R504: 1k, Resistor_SMD:R_0805_2012Metric, F.Cu at (109.3, -33.2)
- added R505: 4k7 / 10k, Resistor_SMD:R_0805_2012Metric, F.Cu at (109.3, -30.3)
- added R506: 10, Resistor_SMD:R_0805_2012Metric, F.Cu at (109.3, -27.4)
- added R507: dnp, Resistor_SMD:R_0805_2012Metric, F.Cu at (113.8, -42.1)
- added R508: 1k, Resistor_SMD:R_0805_2012Metric, F.Cu at (113.8, -39.1)
- added R509: 4k7 / 10k, Resistor_SMD:R_0805_2012Metric, F.Cu at (113.8, -36.2)
- added R510: 10, Resistor_SMD:R_0805_2012Metric, F.Cu at (113.8, -33.2)
- added R511: dnp, Resistor_SMD:R_0805_2012Metric, F.Cu at (113.8, -30.3)
- added R512: 1k, Resistor_SMD:R_0805_2012Metric, F.Cu at (113.8, -27.4)
- added R513: 4k7 / 10k, Resistor_SMD:R_0805_2012Metric, F.Cu at (118.2, -42.1)
- added R514: 10, Resistor_SMD:R_0805_2012Metric, F.Cu at (118.2, -39.1)
- added R515: dnp, Resistor_SMD:R_0805_2012Metric, F.Cu at (118.2, -36.2)
- added R516: 1k, Resistor_SMD:R_0805_2012Metric, F.Cu at (118.2, -33.2)
- added R517: 4k7 / 10k, Resistor_SMD:R_0805_2012Metric, F.Cu at (118.2, -30.3)
- added R601: 100k, Resistor_SMD:R_0805_2012Metric, F.Cu at (109.4, -22.3)
- added R602: 19k2, Resistor_SMD:R_0805_2012Metric, F.Cu at (109.4, -19.4)
- added R701: 4k7, Resistor_SMD:R_0805_2012Metric, F.Cu at (115.8, -0.55)
- added R702: 470k, Resistor_SMD:R_0805_2012Metric, F.Cu at (115.8, 2.40)
- added R703: 4k-2M, Resistor_THT:R_Axial_DIN0204_L3.6mm_D1.6mm_P1.90mm_Vertical, F.Cu at (119.6, -0.45)
- added R704: 1k5, Resistor_SMD:R_0805_2012Metric, F.Cu at (115.8, 5.35)
- added R705: 3k2, Resistor_SMD:R_0805_2012Metric, F.Cu at (115.8, 8.30)
- added SW301: Reset, Button_Switch_SMD:SW_Tactile_SPST_NO_Straight_CK_PTS636Sx25SMTRLFS, F.Cu at (56.1, -6.50)
- added SW302: SW_Push, Button_Switch_SMD:SW_Tactile_SPST_NO_Straight_CK_PTS636Sx25SMTRLFS, F.Cu at (56.1, -1.25)
- added SW303: SW_Push, Button_Switch_SMD:SW_Tactile_SPST_NO_Straight_CK_PTS636Sx25SMTRLFS, F.Cu at (56.1, 4.00)
- added SW401: Reset, Button_Switch_SMD:SW_Tactile_SPST_NO_Straight_CK_PTS636Sx25SMTRLFS, F.Cu at (77.1, -6.50)
- added TP501: TestPoint, TestPoint:TestPoint_THTPad_D1.5mm_Drill0.7mm, F.Cu at (122.1, -41.8)
- added TP502: TestPoint, TestPoint:TestPoint_THTPad_D1.5mm_Drill0.7mm, F.Cu at (122.1, -38.2)
- added TP503: TestPoint, TestPoint:TestPoint_THTPad_D1.5mm_Drill0.7mm, F.Cu at (122.1, -34.7)
- added TP504: TestPoint, TestPoint:TestPoint_THTPad_D1.5mm_Drill0.7mm, F.Cu at (122.1, -31.1)
- added TP601: TestPoint, TestPoint:TestPoint_THTPad_D1.5mm_Drill0.7mm, F.Cu at (109.7, -13.2)
- added TP602: TestPoint, TestPoint:TestPoint_THTPad_D1.5mm_Drill0.7mm, F.Cu at (109.7, -9.60)
- added TP701: TestPoint, TestPoint:TestPoint_THTPad_D1.5mm_Drill0.7mm, F.Cu at (119.8, 7.35)
- added U101: INA180A2, Package_TO_SOT_SMD:SOT-23-5, F.Cu at (80.1, -31.4)
- added U201: ST67W611, JPComms:ST67W611M1, F.Cu at (32.2, 64.7)
- added U401: STM32G030F6Px, Package_SO:TSSOP-20_4.4x6.5mm_P0.65mm, F.Cu at (59.1, 73.1)
- added U511: MCP6006T-E/OT, Package_TO_SOT_SMD:SOT-23-5, F.Cu at (140.0, 31.0)
- added U512: LFD028BUE-103A, JPDisplays:LFD028BUE-103A, F.Cu at (199.5, 57.2)
- added U513: SCT2024, Package_SO:SSOP-24_3.9x8.7mm_P0.635mm, F.Cu at (177.4, 63.9)
- added U514: LFD028BUE-103A, JPDisplays:LFD028BUE-103A, F.Cu at (199.5, 69.8)
- added U515: MCP6006T-E/OT, Package_TO_SOT_SMD:SOT-23-5, F.Cu at (134.4, -36.5)
- added U601: TPS54302, Package_TO_SOT_SMD:SOT-23-6, F.Cu at (100.3, -5.83)
- added U602: MCP1825S, Package_TO_SOT_SMD:SOT-223-3_TabPin2, F.Cu at (115.0, 99.0)
- added Y201: 32.768k, Crystal:Crystal_SMD_7050-2Pin_7.0x5.0mm, F.Cu at (182.7, -12.6)
- added Y301: 24M, Crystal:Crystal_SMD_Abracon_ABM3-2Pin_5.0x3.2mm, F.Cu at (193.3, -13.5)
- C302, C303, C304: footprint Capacitor_SMD:C_0603_1608Metric -> Capacitor_SMD:C_0805_2012Metric
- C505: value 10p -> 1u
- Q507: value IRLML2502 -> BC847
- U506: value LFD028BUE-103A -> LED Matrix 5x7; footprint JPDisplays:LFD028BUE-103A -> JPDisplays:FYM-7571A
- U508, U509: value KW3-281AVA -> LED Matrix 5x7; footprint JPDisplays:KW3-281AVA -> JPDisplays:FYM-7571A
- U510: value KW3-281AVA -> SCT2167; footprint JPDisplays:KW3-281AVA -> Package_SO:SSOP-16_3.9x4.9mm_P0.635mm; moved to B.Cu
- moved U510 151.5 mm to (105.0, 65.0)
- moved C506 104.9 mm to (100.0, -56.0)
- moved C505 104.9 mm to (100.0, -59.0)
- moved C507 104.9 mm to (100.0, -53.0)
- moved C501 99.3 mm to (100.0, -65.0)
- moved C502 99.3 mm to (100.0, -62.0)
- moved U509 98.4 mm to (158.3, 64.2), turned to 90 degrees
- moved U508 90.2 mm to (139.3, 64.2), turned to 90 degrees
- moved U506 79.3 mm to (120.6, 64.0), turned to 90 degrees
- moved U505 72.9 mm to (105.0, 57.5)
- moved Q507 59.9 mm to (99.9, 51.0)
- moved U503 50.0 mm to (139.5, 42.0)
- moved Q503 38.6 mm to (81.3, 71.9)
- moved Q504 38.6 mm to (85.8, 71.9)
- moved U501 38.6 mm to (67.8, 63.0)
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- renumbered C504 to C503, C503 to C504, Q502 to Q501, Q503 to Q502, Q504 to Q503, Q505 to Q504, Q506 to Q505, U302 to U301, U303 to U302, U503 to U502, U502 to U503, U512 to U505, U511 to U507
Connections:
- net /Host Controller/NRST renamed /Controller/NRST
- net LED_BRIGHT renamed /Display/LED_BRIGHTNESS
- C505 pad 1: Net-(U512-CLK) -> +3.3V
- Q501 pad 1: /Display/DIS1_EN -> /Controller/DIS1_EN
- Q501 pad 3: Net-(D502-A) -> Net-(Q501-D)
- Q502 pad 1: /Display/DIS2_EN -> /Controller/DIS2_EN
- Q502 pad 3: Net-(Q503-D) -> Net-(Q502-D)
- Q503 pad 1: /Display/DIS3_EN -> /Controller/DIS3_EN
- Q503 pad 3: Net-(Q504-D) -> Net-(Q503-D)
- Q504 pad 1: /Display/DIS4_EN -> /Controller/DIS4_EN
- Q504 pad 3: Net-(Q505-D) -> Net-(Q504-D)
- Q505 pad 1: /Display/DIS5_EN -> /Controller/DIS5_EN
- Q505 pad 3: Net-(Q506-D) -> Net-(Q505-D)
- U301 pad 5: unconnected-(U302-WP-Pad5) -> GND
- U302 pad 35: /Host Controller/SWDIO -> /Controller/SWDIO
- U302 pad 36: /Host Controller/SWCLK -> /Controller/SWCLK
- U302 pad 42: /Host Controller/DISPL_SCK -> /Controller/SCT_CLK
- U302 pad 44: /Host Controller/DISPL_MOSI -> /Controller/SCT_SDI
- U302 pad 5: unconnected-(U303-VREF+-Pad5) -> GND
- U501 pad 2: /Display/STC_SDI -> /Controller/SCT_SDI
- U501 pad 21: /Display/!SCT_EN -> /Controller/~{SCT_EN}
- U501 pad 22: unconnected-(U501-SDO-Pad22) -> Net-(U501-SDO)
- U501 pad 4: /Display/!SCT_LA -> /Controller/~{SCT_LA}
- U502 pad 1: Net-(D502-A) -> Net-(Q501-D)
- U502 pad 11: Net-(Q504-D) -> Net-(Q503-D)
- U502 pad 12: Net-(Q506-D) -> Net-(Q505-D)
- U502 pad 14: Net-(Q503-D) -> Net-(Q502-D)
- U502 pad 8: Net-(Q505-D) -> Net-(Q504-D)
- U503 pad 5: VDD -> +3.3V
- U504 pad 1: Net-(D502-A) -> Net-(Q501-D)
- U504 pad 11: Net-(Q504-D) -> Net-(Q503-D)
- U504 pad 12: Net-(Q506-D) -> Net-(Q505-D)
- U504 pad 14: Net-(Q503-D) -> Net-(Q502-D)
- U504 pad 8: Net-(Q505-D) -> Net-(Q504-D)
- U505 pad 10: /Display/LINE1_6 -> /Display/DIS3_6
- U505 pad 11: /Display/LINE1_7 -> /Display/DIS3_7
- U505 pad 12: /Display/LINE1_8 -> /Display/DIS3_8
- U505 pad 13: /Display/LINE1_9 -> /Display/DIS3_9
- U505 pad 14: /Display/LINE1_10 -> /Display/DIS3_10
- U505 pad 15: /Display/LINE1_11 -> /Display/DIS3_11
- U505 pad 16: /Display/LINE1_12 -> /Display/DIS3_12
- U505 pad 17: /Display/LINE1_13 -> /Display/DIS3_13
- U505 pad 18: /Display/LINE1_14 -> /Display/DIS3_14
- U505 pad 19: /Display/LINE1_15 -> /Display/DIS3_15
- U505 pad 2: /Display/STC_SDI -> Net-(U501-SDO)
- U505 pad 20: /Display/LINE1_16 -> /Display/DIS3_16
- U505 pad 21: /Display/!SCT_EN -> /Controller/~{SCT_EN}
- U505 pad 22: unconnected-(U512-SDO-Pad22) -> Net-(U505-SDO)
- U505 pad 3: Net-(U512-CLK) -> Net-(U501-CLK)
- U505 pad 4: /Display/!SCT_LA -> /Controller/~{SCT_LA}
- U505 pad 5: /Display/LINE1_1 -> /Display/DIS3_1
- U505 pad 6: /Display/LINE1_2 -> /Display/DIS3_2
- U505 pad 7: /Display/LINE1_3 -> /Display/DIS3_3
- U505 pad 8: /Display/LINE1_4 -> /Display/DIS3_4
- U505 pad 9: /Display/LINE1_5 -> /Display/DIS3_5
- U506 pad 1: unconnected-(U506-Dig1-Pad1) -> Net-(Q501-D)
- U506 pad 11: unconnected-(U506-Dig3-Pad11) -> /Display/DIS3_2
- U506 pad 12: unconnected-(U506-L-Pad12) -> /Display/DIS3_1
- U506 pad 2: unconnected-(U506-C-Pad2) -> /Display/DIS3_3
- U506 pad 3: unconnected-(U506-DP-Pad3) -> Net-(Q502-D)
- U506 pad 4: (no net) -> /Display/DIS3_5
- U506 pad 5: unconnected-(U506-E-Pad5) -> /Display/DIS3_6
- U506 pad 6: unconnected-(U506-D-Pad6) -> /Display/DIS3_7
- U506 pad 7: unconnected-(U506-G-Pad7) -> Net-(Q504-D)
- U506 pad 8: unconnected-(U506-Dig4-Pad8) -> Net-(Q505-D)
- U506 pad 9: (no net) -> /Display/DIS3_4
- U507 pad 5: VDD -> +3.3V
- U508 pad 1: unconnected-(U508-E-Pad1) -> Net-(Q501-D)
- U508 pad 10: unconnected-(U508-F-Pad10) -> Net-(Q503-D)
- U508 pad 11: unconnected-(U508-A-Pad11) -> /Display/DIS3_9
- U508 pad 12: unconnected-(U508-Dig1-Pad12) -> /Display/DIS3_8
- U508 pad 2: unconnected-(U508-D-Pad2) -> /Display/DIS3_10
- U508 pad 3: unconnected-(U508-DP-Pad3) -> Net-(Q502-D)
- U508 pad 4: unconnected-(U508-C-Pad4) -> /Display/DIS3_12
- U508 pad 5: unconnected-(U508-G-Pad5) -> /Display/DIS3_13
- U508 pad 7: unconnected-(U508-B-Pad7) -> Net-(Q504-D)
- U508 pad 8: unconnected-(U508-Dig3-Pad8) -> Net-(Q505-D)
- U508 pad 9: unconnected-(U508-Dig2-Pad9) -> /Display/DIS3_11
- U509 pad 1: unconnected-(U509-E-Pad1) -> Net-(Q501-D)
- U509 pad 10: unconnected-(U509-F-Pad10) -> Net-(Q503-D)
- U509 pad 11: unconnected-(U509-A-Pad11) -> /Display/DIS3_16
- U509 pad 12: unconnected-(U509-Dig1-Pad12) -> /Display/DIS3_15
- U509 pad 2: unconnected-(U509-D-Pad2) -> /Display/DIS3_17
- U509 pad 3: unconnected-(U509-DP-Pad3) -> Net-(Q502-D)
- U509 pad 4: unconnected-(U509-C-Pad4) -> /Display/DIS3_19
- U509 pad 5: unconnected-(U509-G-Pad5) -> /Display/DIS3_20
- U509 pad 7: unconnected-(U509-B-Pad7) -> Net-(Q504-D)
- U509 pad 8: unconnected-(U509-Dig3-Pad8) -> Net-(Q505-D)
- U509 pad 9: unconnected-(U509-Dig2-Pad9) -> /Display/DIS3_18
- U510 pad 1: unconnected-(U510-E-Pad1) -> GND
- U510 pad 2: unconnected-(U510-D-Pad2) -> Net-(U505-SDO)
- U510 pad 3: unconnected-(U510-DP-Pad3) -> Net-(U501-CLK)
- U510 pad 4: unconnected-(U510-C-Pad4) -> /Controller/~{SCT_LA}
- U510 pad 5: unconnected-(U510-G-Pad5) -> /Display/DIS3_17
- U510 pad 7: unconnected-(U510-B-Pad7) -> /Display/DIS3_19
- U510 pad 8: unconnected-(U510-Dig3-Pad8) -> /Display/DIS3_20
- U510 pad 9: unconnected-(U510-Dig2-Pad9) -> /Display/DIS3_21

Commit message: KiCad work
Parts:
- added C308: 100n, Capacitor_SMD:C_0603_1608Metric, F.Cu at (56.2, 94.2)
- added R102: 5k1, Resistor_SMD:R_0805_2012Metric, F.Cu at (39.0, 85.0)
- added R103: 5k1, Resistor_SMD:R_0805_2012Metric, F.Cu at (99.1, 88.0)
- added R309: dnp, Resistor_SMD:R_0805_2012Metric, F.Cu at (56.5, 90.5)
- C501, C502, C504, Q506, R501, R502, R503, R504, R505, U513: moved to B.Cu
- C601: footprint Capacitor_SMD:C_0201_0603Metric -> Capacitor_SMD:C_0805_2012Metric
- U302: moved to F.Cu
- moved Y201 178.8 mm to (14.0, 46.5), turned to -90 degrees
- moved C501 134.2 mm to (60.4, 63.2), turned to 90 degrees
- moved C502 131.9 mm to (58.4, 63.2), turned to 90 degrees
- moved SW401 130.6 mm to (49.0, 121.0)
- moved TP501 129.9 mm to (60.6, 72.7)
- moved R201 129.7 mm to (31.0, 76.0)
- moved C201 129.0 mm to (28.0, 56.0), turned to 180 degrees
- moved C204 125.2 mm to (20.0, 45.5)
- moved C205 124.7 mm to (20.0, 47.5)
- moved C203 123.6 mm to (41.0, 69.0), turned to 90 degrees
- moved R502 123.2 mm to (63.9, 75.4), turned to 180 degrees
- moved C202 120.2 mm to (41.0, 61.0), turned to -90 degrees
- moved R501 119.1 mm to (59.8, 66.2)
- moved C401 118.4 mm to (48.0, 110.5)
- moved R503 117.2 mm to (68.6, 73.7)
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Connections:
- net Net-(Q506-C) renamed /Display/SCT1_REXT
- C501 pad 1: +3.3V -> /Display/SCT1_VDD
- C502 pad 1: +3.3V -> /Display/SCT1_VDD
- J101 pad 11: /Controller/SCT_SDI -> /Display/SCT_SDO
- R501 pad 2: Net-(U501-VDD) -> /Display/SCT1_VDD
- U501 pad 24: Net-(U501-VDD) -> /Display/SCT1_VDD
- U513 pad 22: unconnected-(U513-SDO-Pad22) -> /Display/SCT_SDO
Routing:
- net (no net): track 0.00 -> 1.21 mm
Other:
- copper layers 2 -> 4

Commit message: Work
Parts:
- added R310: x, Resistor_SMD:R_0805_2012Metric, F.Cu at (44.5, 61.0)
- C206: footprint Capacitor_SMD:C_0201_0603Metric -> Capacitor_SMD:C_0805_2012Metric
- C505, C506, C507, C508, C509, C510, Q507, Q508, Q509, R506, R507, R508, R509, R510, R511, R512, R513, R514, R515, R516, R517, U507, U511, U515: moved to B.Cu
- J103: footprint Connector_JST:JST_PH_S6B-PH-SM4-TB_1x06-1MP_P2.00mm_Horizontal -> Connector_JST:JST_PH_B6B-PH-K_1x06_P2.00mm_Vertical
- J107: value USB_C_Receptacle_USB2.0_14P -> USB; footprint Connector_USB:USB_C_Receptacle_GCT_USB4135-GF-A_6P_TopMnt_Horizontal -> JPConnectors:USB_C_Receptacle_GCT_USB4216
- L601: footprint Inductor_SMD:L_7.3x7.3_H4.5 -> Inductor_SMD:L_Wuerth_MAPI-4020
- R703: footprint Resistor_THT:R_Axial_DIN0204_L3.6mm_D1.6mm_P1.90mm_Vertical -> OptoDevice:R_LDR_4.9x4.2mm_P2.54mm_Vertical
- TP501, TP502, TP503, TP504: footprint TestPoint:TestPoint_THTPad_D1.5mm_Drill0.7mm -> TestPoint:TestPoint_Pad_D1.5mm; moved to B.Cu
- TP601, TP602, TP701: footprint TestPoint:TestPoint_THTPad_D1.5mm_Drill0.7mm -> TestPoint:TestPoint_Pad_D1.5mm
- moved Y301 163.8 mm to (46.0, 58.0)
- moved J106 131.6 mm to (146.1, 72.6), turned to 90 degrees
- moved C607 126.5 mm to (178.5, 96.0), turned to 90 degrees
- moved J104 126.2 mm to (107.0, 81.2)
- moved D101 123.6 mm to (91.0, 79.0)
- moved C101 123.3 mm to (102.0, 89.5), turned to 180 degrees
- moved D102 122.6 mm to (91.0, 81.0)
- moved C509 122.6 mm to (169.6, 54.0), turned to 90 degrees
- moved TP602 121.8 mm to (177.5, 91.5)
- moved C606 121.1 mm to (163.5, 96.0), turned to 90 degrees
- moved C510 119.0 mm to (167.6, 54.0), turned to 90 degrees
- moved R101 116.9 mm to (155.6, 72.4)
- moved U101 116.4 mm to (100.4, 83.2)
- moved C507 115.6 mm to (95.2, 62.5), turned to 90 degrees
- moved C206 115.0 mm to (31.0, 54.5)
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Connections:
- net Net-(D501-A) renamed /Display/VDD_LED
- net Net-(Q501-D) renamed /Display/VDD_DIG1
- net Net-(Q502-D) renamed /Display/VDD_DIG2
- net Net-(Q503-D) renamed /Display/VDD_DIG3
- net Net-(Q504-D) renamed /Display/VDD_DIG4
- net Net-(Q505-D) renamed /Display/VDD_DIG5
- net Net-(Q507-C) renamed /Display/SCT2_REXT
- net Net-(Q508-C) renamed /Display/SCT3_REXT
- net Net-(Q509-C) renamed /Display/SCT4_REXT
- net Net-(U302-PF0) renamed /Host Controller/OSC_IN
- net Net-(U501-CLK) renamed /Display/SCT_CLK_F
- net Net-(U501-SDO) renamed /Display/SCT1_SDO
- C304 pad 2: Net-(U302-PF1) -> Net-(C304-Pad2)
- C505 pad 1: +3.3V -> /Display/SCT2_VDD
- C506 pad 1: +3.3V -> /Display/SCT2_VDD
- C507 pad 1: +3.3V -> /Display/SCT3_VDD
- C508 pad 1: +3.3V -> /Display/SCT3_VDD
- C509 pad 1: +3.3V -> /Display/SCT4_VDD
- C510 pad 1: +3.3V -> /Display/SCT4_VDD
- J101 pad 17: /Controller/DIS1_EN -> /Controller/DISPLAY1_EN
- J101 pad 18: /Controller/DIS2_EN -> /Controller/DISPLAY2_EN
- J101 pad 19: /Controller/DIS3_EN -> /Controller/DISPLAY3_EN
- J101 pad 20: /Controller/DIS4_EN -> /Controller/DISPLAY4_EN
- J101 pad 21: /Controller/DIS5_EN -> /Controller/DISPLAY5_EN
- J105 pad 17: /Controller/DIS1_EN -> /Controller/DISPLAY1_EN
- J105 pad 18: /Controller/DIS2_EN -> /Controller/DISPLAY2_EN
- J105 pad 19: /Controller/DIS3_EN -> /Controller/DISPLAY3_EN
- J105 pad 20: /Controller/DIS4_EN -> /Controller/DISPLAY4_EN
- J105 pad 21: /Controller/DIS5_EN -> /Controller/DISPLAY5_EN
- Q501 pad 1: /Controller/DIS1_EN -> /Controller/DISPLAY1_EN
- Q502 pad 1: /Controller/DIS2_EN -> /Controller/DISPLAY2_EN
- Q503 pad 1: /Controller/DIS3_EN -> /Controller/DISPLAY3_EN
- Q504 pad 1: /Controller/DIS4_EN -> /Controller/DISPLAY4_EN
- Q505 pad 1: /Controller/DIS5_EN -> /Controller/DISPLAY5_EN
- R506 pad 2: Net-(U505-VDD) -> /Display/SCT2_VDD
- R510 pad 2: Net-(U510-VDD) -> /Display/SCT3_VDD
- R514 pad 2: Net-(U513-VDD) -> /Display/SCT4_VDD
- U302 pad 21: unconnected-(U302-PB2-Pad21) -> /Host Controller/OSC_OUT
- U302 pad 27: unconnected-(U302-PB15-Pad27) -> /Host Controller/UCPD_CC2
- U302 pad 28: unconnected-(U302-PA8-Pad28) -> /Host Controller/UCPD_CC1
- U302 pad 33: unconnected-(U302-PA9/PA11-Pad33) -> /Host Controller/USB-
- U302 pad 34: unconnected-(U302-PA10/PA12-Pad34) -> /Host Controller/USB+
- U302 pad 37: unconnected-(U302-PA15-Pad37) -> /Controller/DISPLAY2_EN
- U302 pad 38: unconnected-(U302-PD0-Pad38) -> /Controller/DISPLAY5_EN
- U302 pad 39: unconnected-(U302-PD1-Pad39) -> /Controller/DISPLAY3_EN
- U302 pad 40: unconnected-(U302-PD2-Pad40) -> /Controller/DISPLAY4_EN
- U302 pad 41: unconnected-(U302-PD3-Pad41) -> /Controller/DISPLAY1_EN
- U302 pad 9: Net-(U302-PF1) -> /Host Controller/OSC_OUT
- U501 pad 10: /Display/DIS1_F -> /Display/DIS1_DP
- U501 pad 11: /Display/DIS1_G -> /Display/DIS1_E
- U501 pad 12: /Display/DIS1_DP -> /Display/DIS1_G
- U501 pad 13: /Display/DIS2_A -> /Display/DIS2_DP
- U501 pad 14: /Display/DIS2_B -> /Display/DIS2_C
- U501 pad 15: /Display/DIS2_C -> /Display/DIS2_E
- U501 pad 17: /Display/DIS2_E -> /Display/DIS2_G
- U501 pad 18: /Display/DIS2_F -> /Display/DIS2_A
- U501 pad 19: /Display/DIS2_G -> /Display/DIS2_B
- U501 pad 20: /Display/DIS2_DP -> /Display/DIS2_F
- U501 pad 5: /Display/DIS1_A -> /Display/DIS1_F
- U501 pad 7: /Display/DIS1_C -> /Display/DIS1_A
- U501 pad 9: /Display/DIS1_E -> /Display/DIS1_C
- U505 pad 22: Net-(U505-SDO) -> /Display/SCT2_SDO
- U505 pad 24: Net-(U505-VDD) -> /Display/SCT2_VDD
- U510 pad 14: unconnected-(U510-SDO-Pad14) -> /Display/SCT3_SDO
- U510 pad 16: Net-(U510-VDD) -> /Display/SCT3_VDD
- U510 pad 2: Net-(U505-SDO) -> /Display/SCT2_SDO
- U513 pad 10: /Display/DIS4_F -> /Display/DIS4_E
- U513 pad 11: /Display/DIS4_G -> /Display/DIS4_D
- U513 pad 12: /Display/DIS4_DP -> /Display/DIS4_G
- U513 pad 15: /Display/DIS5_C -> /Display/DIS5_F
- U513 pad 16: /Display/DIS5_D -> /Display/DIS5_G
- U513 pad 17: /Display/DIS5_E -> /Display/DIS5_D
- U513 pad 18: /Display/DIS5_F -> /Display/DIS5_E
- U513 pad 19: /Display/DIS5_G -> /Display/DIS5_DP
- U513 pad 2: Net-(U505-SDO) -> /Display/SCT3_SDO
- U513 pad 20: /Display/DIS5_DP -> /Display/DIS5_C
- U513 pad 24: Net-(U513-VDD) -> /Display/SCT4_VDD
- U513 pad 7: /Display/DIS4_C -> /Display/DIS4_F
- U513 pad 8: /Display/DIS4_D -> /Display/DIS4_C
- U513 pad 9: /Display/DIS4_E -> /Display/DIS4_DP
- Y301 pad 1: Net-(U302-PF1) -> Net-(C304-Pad2)
Routing:
- net /Display/VDD_DIG5: track 0.00 -> 197.8 mm, vias 0 -> 3
- net /Display/VDD_DIG2: track 0.00 -> 173.5 mm, vias 0 -> 1
- net /Display/VDD_DIG3: track 0.00 -> 173.1 mm, vias 0 -> 2
- net /Display/VDD_DIG4: track 0.00 -> 156.8 mm, vias 0 -> 1
- net /Controller/DISPLAY5_EN: track 0.00 -> 109.6 mm, vias 0 -> 1
- net /Controller/DISPLAY3_EN: track 0.00 -> 105.0 mm, vias 0 -> 1
- net /Controller/DISPLAY4_EN: track 0.00 -> 101.9 mm, vias 0 -> 1
- net /Display/VDD_DIG1: track 0.00 -> 101.3 mm, vias 0 -> 1
- net /Controller/DISPLAY1_EN: track 0.00 -> 89.5 mm, vias 0 -> 1
- net /Controller/DISPLAY2_EN: track 0.00 -> 83.3 mm, vias 0 -> 1
- net /Display/DIS3_18: track 0.00 -> 65.8 mm
- net /Display/DIS3_20: track 0.00 -> 62.9 mm
- net /Display/DIS3_19: track 0.00 -> 61.1 mm
- net /Display/DIS3_21: track 0.00 -> 60.9 mm
- net /Host Controller/USB+: track 0.00 -> 60.0 mm
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- added copper zone on F.Cu, net GND
- added copper zone on In1.Cu, net GND
- added copper zone on F.Cu, net VBUS
- added copper zone on F.Cu, net VDD
Other:
- board size 243 x 28 mm -> 185 x 28 mm

Commit message: KiCad work
Parts:
- removed C401, C403: 100n, Capacitor_SMD:C_0603_1608Metric
- removed C402: 4u7, Capacitor_SMD:C_0805_2012Metric
- removed J106: POWER_SELECT, Connector_PinSocket_2.54mm:PinSocket_1x03_P2.54mm_Vertical
- removed R503, R507, R511, R515: dnp, Resistor_SMD:R_0805_2012Metric
- removed SW401: Reset, Button_Switch_SMD:SW_Tactile_SPST_NO_Straight_CK_PTS636Sx25SMTRLFS
- removed U401: STM32G030F6Px, Package_SO:TSSOP-20_4.4x6.5mm_P0.65mm
- added SW304: SW_DIP_x03, Button_Switch_SMD:SW_DIP_SPSTx03_Slide_KingTek_DSHP03TJ_W5.25mm_P1.27mm_JPin, F.Cu at (43.9, 43.0)
- C101, R101, U101: moved to B.Cu
- J104: footprint Connector_PinSocket_2.54mm:PinSocket_1x02_P2.54mm_Vertical -> Connector_PinHeader_2.54mm:PinHeader_1x02_P2.54mm_Vertical
- moved C503 93.0 mm to (160.6, 55.6), turned to 90 degrees
- moved R101 55.4 mm to (100.2, 71.0)
- moved TP701 51.6 mm to (59.5, 58.0)
- moved R703 48.4 mm to (54.6, 62.2)
- moved Q701 48.4 mm to (55.2, 65.2)
- moved R701 48.4 mm to (54.5, 60.2)
- moved R702 48.4 mm to (58.0, 60.2)
- moved R704 48.4 mm to (59.8, 63.0)
- moved R705 48.4 mm to (59.0, 65.8)
- moved U602 43.3 mm to (167.6, 53.8), turned to 90 degrees
- moved C607 42.3 mm to (172.2, 54.1)
- moved C606 41.9 mm to (163.0, 54.1)
- moved R103 40.7 mm to (55.2, 75.8), turned to -90 degrees
- moved R102 38.3 mm to (57.2, 75.7), turned to -90 degrees
- moved TP602 35.5 mm to (172.4, 56.4)
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Connections:
- net /Controller/DISPLAY1_EN renamed /Display/DISPLAY1_EN
- net /Controller/DISPLAY2_EN renamed /Display/DISPLAY2_EN
- net /Controller/DISPLAY3_EN renamed /Display/DISPLAY3_EN
- net /Controller/DISPLAY4_EN renamed /Display/DISPLAY4_EN
- net /Controller/DISPLAY5_EN renamed /Display/DISPLAY5_EN
- net /Controller/NRST renamed /Host Controller/NRST
- net /Controller/SCT_CLK renamed /Display/SCT_CLK
- net /Controller/SCT_SDI renamed /Display/SCT_SDI
- net /Controller/SWCLK renamed /Host Controller/SWCLK
- net /Controller/SWDIO renamed /Host Controller/SWDIO
- net /Controller/~{SCT_EN} renamed /Display/~{SCT_EN}
- net /Controller/~{SCT_LA} renamed /Display/~{SCT_LA}
- J104 pad 2: Net-(J104-Pin_2) -> /Host Controller/VOLTAGE_SENSE
- J107 pad A4: Net-(J106-Pin_3) -> /Host Controller/VOLTAGE_SENSE
- J107 pad A9: Net-(J106-Pin_3) -> /Host Controller/VOLTAGE_SENSE
- J107 pad B4: Net-(J106-Pin_3) -> /Host Controller/VOLTAGE_SENSE
- J107 pad B9: Net-(J106-Pin_3) -> /Host Controller/VOLTAGE_SENSE
Routing:
- net +3.3V: track 0.00 -> 206.9 mm, vias 0 -> 10
- net /Display/~{SCT_LA}: track 0.00 -> 140.8 mm, vias 0 -> 6
- net /Display/SCT_CLK_F: track 7.45 -> 141.2 mm, vias 0 -> 5
- net /Display/SCT3_SDO: track 0.00 -> 87.8 mm, vias 0 -> 2
- net /Display/~{SCT_EN}: track 53.2 -> 140.7 mm, vias 4 -> 6
- net VBUS: track 5.27 -> 87.4 mm, vias 0 -> 3
- net /Host Controller/UCPD_CC2: track 0.00 -> 62.7 mm, vias 0 -> 2
- net /Display/VDD_DIG1: track 101.3 -> 162.4 mm, vias 1 -> 3
- net /Host Controller/UCPD_CC1: track 0.00 -> 58.1 mm, vias 0 -> 2
- net GND: track 44.5 -> 99.5 mm, vias 11 -> 27
- net /Display/LED_BRIGHTNESS: track 0.00 -> 19.3 mm
- net /Host Controller/VOLTAGE_SENSE: track 0.00 -> 17.4 mm, vias 0 -> 1
- net /Display/DISPLAY1_EN: track 89.5 -> 78.1 mm
- net Net-(Q701-D): track 0.00 -> 7.96 mm
- net /Display/VDD_LED: track 50.6 -> 58.1 mm
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- added copper zone on In4.Cu, net GND
Other:
- board size 185 x 28 mm -> 185 x 30 mm
- copper layers 4 -> 6
