File: KiCad/AstroWeather.kicad_pcb (KiCad board)
At the start: 6 copper layers, 185 x 30 mm, 123 parts, among them J101 OUTPUT, J102 I2C, J103 SWD, J104 AUX_POWER, J105 INPUT, J107 USB, Q501 Si2365EDS, Q502 Si2365EDS, Q503 Si2365EDS, Q504 Si2365EDS, Q505 Si2365EDS, Q506 BC847, Q507 BC847, Q508 BC847, Q509 BC847, Q701 IRLML2502, SW301 Reset, SW302 SW_Push, SW303 SW_Push, SW304 SW_DIP_x03, U101 INA180A2, U201 ST67W611, U301 AT24CS01-STUM, U302 STM32G0B1CETx, U501 SCT2024, U502 LFD028BUE-103A, U503 MCP6006T-E/OT, U504 LFD028BUE-103A, U505 SCT2024, U506 LED Matrix 5x7, U507 MCP6006T-E/OT, U508 LED Matrix 5x7, U509 LED Matrix 5x7, U510 SCT2167, U511 MCP6006T-E/OT, U512 LFD028BUE-103A, U513 SCT2024, U514 LFD028BUE-103A, U515 MCP6006T-E/OT, U601 TPS54302, U602 MCP1825S, Y201 32.768k, Y301 24M

Commit message: KiCad work
Parts:
- removed C204, C205: 5p1, Capacitor_SMD:C_0805_2012Metric
- removed SW301: Reset, Button_Switch_SMD:SW_Tactile_SPST_NO_Straight_CK_PTS636Sx25SMTRLFS
- removed Y201: 32.768k, Crystal:Crystal_SMD_7050-2Pin_7.0x5.0mm
- added TP301: TestPoint, TestPoint:TestPoint_Pad_D1.5mm, F.Cu at (39.5, 71.0)
- R102, R103, R301, R302, U301: moved to B.Cu
- moved D302 22.0 mm to (31.4, 76.2), turned to -90 degrees
- moved SW302 18.6 mm to (56.2, 75.8)
- moved R308 18.5 mm to (33.1, 76.2), turned to 90 degrees
- moved D301 17.0 mm to (37.0, 76.2), turned to -90 degrees
- moved R307 14.5 mm to (35.2, 76.2), turned to 90 degrees
- moved R301 11.3 mm to (53.8, 72.0), turned to 180 degrees
- moved Q701 9.83 mm to (58.5, 56.0), turned to -90 degrees
- moved R705 8.79 mm to (55.8, 57.6), turned to -90 degrees
- moved R302 7.80 mm to (53.8, 77.5), turned to 180 degrees
- moved TP701 7.16 mm to (56.0, 64.2)
- moved U301 6.13 mm to (53.8, 74.8)
- moved R103 4.75 mm to (60.0, 76.0)
- moved R704 3.81 mm to (58.2, 59.5), turned to 90 degrees
- moved C303 3.16 mm to (47.5, 57.0), turned to -90 degrees
- moved C305 2.85 mm to (38.8, 60.8), turned to 90 degrees
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Connections:
- U201 pad 13: Net-(U201-XTAL32K_OUT) -> unconnected-(U201-XTAL32K_OUT-Pad13)
- U201 pad 14: Net-(U201-XTAL32K_IN) -> unconnected-(U201-XTAL32K_IN-Pad14)
- U302 pad 11: unconnected-(U302-PA0-Pad11) -> /Host Controller/ST67_CHIP_EN
- U302 pad 15: unconnected-(U302-PA4-Pad15) -> /Host Controller/ST67_RDY
- U302 pad 16: unconnected-(U302-PA5-Pad16) -> /Host Controller/ST67_CS
- U302 pad 20: unconnected-(U302-PB1-Pad20) -> /Host Controller/ST67_BOOT
- U302 pad 21: /Host Controller/OSC_OUT -> /Host Controller/OSC_OUT_PIN
- U302 pad 45: unconnected-(U302-PB6-Pad45) -> /Display/~{SCT_LA}
- U302 pad 46: unconnected-(U302-PB7-Pad46) -> /Display/~{SCT_EN}
- U302 pad 47: unconnected-(U302-PB8-Pad47) -> /Host Controller/LOW_POWER_ENABLE
Routing:
- net /Host Controller/I2C_SCL: track 0.00 -> 154.1 mm
- net /Host Controller/I2C_SDA: track 0.00 -> 148.1 mm
- net /Display/LED_BRIGHTNESS: track 19.3 -> 156.9 mm, vias 0 -> 3
- net +3.3V: track 206.9 -> 301.9 mm, vias 10 -> 16
- net GND: track 99.5 -> 133.0 mm, vias 27 -> 44
- net /Host Controller/SWDIO: track 0.00 -> 29.8 mm, vias 0 -> 1
- net /Host Controller/SWCLK: track 0.00 -> 26.2 mm, vias 0 -> 1
- net /Host Controller/ST67_SCK: track 0.00 -> 25.9 mm, vias 0 -> 2
- net /Host Controller/ST67_MOSI: track 0.00 -> 24.6 mm, vias 0 -> 2
- net /Host Controller/NRST: track 0.00 -> 24.2 mm
- net /Host Controller/ST67_MISO: track 0.00 -> 24.0 mm, vias 0 -> 2
- net /Host Controller/ST67_CS: track 0.00 -> 23.3 mm, vias 0 -> 2
- net /Host Controller/ST67_RX: track 0.00 -> 23.0 mm, vias 0 -> 2
- net /Host Controller/ST67_TX: track 0.00 -> 21.6 mm, vias 0 -> 2
- net /Host Controller/ST67_RDY: track 0.00 -> 20.7 mm, vias 0 -> 2
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
Commit message: some work
Parts:
- C306, C307, C503, D301, R303, R304, R305, R306: moved to B.Cu
- moved D302 38.7 mm to (60.0, 50.2), turned to 180 degrees
- moved SW303 38.1 mm to (44.9, 76.3), turned to 180 degrees
- moved R304 35.7 mm to (43.0, 76.6), turned to -90 degrees
- moved R305 35.3 mm to (35.8, 76.6), turned to -90 degrees
- moved R306 35.1 mm to (44.5, 76.6), turned to -90 degrees
- moved R308 34.6 mm to (57.0, 51.2), turned to -90 degrees
- moved C307 34.5 mm to (46.0, 76.6), turned to -90 degrees
- moved C306 34.2 mm to (34.2, 76.6), turned to -90 degrees
- moved R303 33.4 mm to (37.2, 76.6), turned to -90 degrees
- moved R307 31.4 mm to (54.2, 51.2), turned to -90 degrees
- moved D301 29.1 mm to (50.0, 50.2), turned to 0 degrees
- moved SW302 20.9 mm to (35.4, 76.3)
- moved J102 18.6 mm to (59.0, 76.5), turned to -90 degrees
- moved R302 5.71 mm to (56.8, 72.7), turned to -90 degrees
- moved R102 3.78 mm to (61.8, 75.5)
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Connections:
- R303 pad 1: +3V3 -> +3.3V
- R304 pad 1: +3V3 -> +3.3V
- U302 pad 1: unconnected-(U302-PC13-Pad1) -> /Host Controller/LED1
- U302 pad 24: unconnected-(U302-PB12-Pad24) -> /Host Controller/SWITCH_2
- U302 pad 25: unconnected-(U302-PB13-Pad25) -> /Host Controller/SWITCH_1
- U302 pad 48: unconnected-(U302-PB9-Pad48) -> /Host Controller/LED2
Routing:
- net VBUS: track 87.4 -> 121.4 mm
- net /Host Controller/LED2: track 0.00 -> 18.0 mm
- net VDD: track 31.0 -> 48.6 mm, vias 0 -> 2
- net /Host Controller/LED1: track 0.00 -> 15.2 mm
- net GND: track 133.0 -> 146.4 mm, vias 44 -> 46
- net /Host Controller/SWITCH_2: track 0.00 -> 10.5 mm, vias 0 -> 1
- net +3.3V: track 301.9 -> 311.7 mm, vias 16 -> 19
- net /Host Controller/SWITCH_1: track 0.00 -> 4.92 mm, vias 0 -> 1
- net Net-(R304-Pad2): track 0.00 -> 4.39 mm, vias 0 -> 1
- net Net-(R303-Pad2): track 0.00 -> 4.39 mm, vias 0 -> 1
- net /Host Controller/I2C_SCL: track 154.1 -> 150.3 mm
- net /Host Controller/I2C_SDA: track 148.1 -> 145.3 mm
- net Net-(Q509-E): track 5.30 -> 7.64 mm
- net Net-(Q509-B): track 0.00 -> 2.16 mm
- net /Display/SCT_SDI: track 21.5 -> 19.5 mm
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
Commit message: KiCad work
Parts:
- removed the J101 at (160.1, 52.1)
- removed the J105 at (160.1, 76.2)
- removed SW304: SW_DIP_x03, Button_Switch_SMD:SW_DIP_SPSTx03_Slide_KingTek_DSHP03TJ_W5.25mm_P1.27mm_JPin
- added C307: 100n, Capacitor_SMD:C_0805_2012Metric, B.Cu at (44.0, 70.2)
- added H101: MountingHole, MountingHole:MountingHole_3.2mm_M3, F.Cu at (25.0, 52.4)
- added H102: MountingHole, MountingHole:MountingHole_3.2mm_M3, F.Cu at (157.0, 52.4)
- added H103: MountingHole, MountingHole:MountingHole_3.2mm_M3, F.Cu at (157.0, 75.6)
- added J102: Conn_01x10, Connector_PinSocket_2.54mm:PinSocket_1x10_P2.54mm_Horizontal, F.Cu at (132.9, 52.0)
- added J104: Conn_01x10, Connector_PinHeader_2.54mm:PinHeader_1x10_P2.54mm_Horizontal, F.Cu at (132.9, 76.1)
- added JP301: A0, Jumper:SolderJumper-3_P1.3mm_Open_RoundedPad1.0x1.5mm, F.Cu at (23.4, 76.3)
- added JP302: A1, Jumper:SolderJumper-3_P1.3mm_Open_RoundedPad1.0x1.5mm, F.Cu at (26.0, 76.3)
- added JP303: A2, Jumper:SolderJumper-3_P1.3mm_Open_RoundedPad1.0x1.5mm, F.Cu at (28.6, 76.3)
- added R305: ?, Resistor_SMD:R_0805_2012Metric, B.Cu at (48.2, 70.2)
- C306: renamed from C308; footprint Capacitor_SMD:C_0603_1608Metric -> Capacitor_SMD:C_0805_2012Metric; moved to B.Cu
- D301: moved to F.Cu
- R304: renamed from R309; value dnp -> ?; moved to B.Cu
- R310: renamed from R307; moved to B.Cu
- moved C306 27.0 mm to (44.0, 68.2), turned to 180 degrees
- moved R304 22.5 mm to (48.2, 68.2)
- moved D301 4.49 mm to (54.4, 51.1), turned to -90 degrees
- moved R310 4.38 mm to (50.0, 50.2), turned to 0 degrees
- moved R311 3.18 mm to (60.0, 50.2), turned to 180 degrees
- moved D302 3.13 mm to (57.0, 51.1), turned to -90 degrees
- moved TP701 1.42 mm to (54.8, 65.0)
- moved R103 1.30 mm to (63.4, 76.8)
- moved TP301 0.83 mm to (38.8, 71.2)
- moved TP602 0.72 mm to (172.0, 57.0)
- moved C201 0.39 mm to (22.2, 56.8)
- moved R102 0.35 mm to (61.4, 75.5)
- moved C308 0.25 mm to (34.0, 76.6)
- moved C309 0.25 mm to (45.8, 76.6)
- moved R306 0.25 mm to (37.0, 76.6)
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- renumbered C206 to C204, C306 to C308, C307 to C309, C506 to C505, C505 to C506, C508 to C507, C507 to C508, C510 to C509, C509 to C510, J102 to J101, J104 to J105, J107 to J106, R310 to R303, R303 to R306, R304 to R307, R305 to R308, R306 to R309, R308 to R311, R504 to R503, R505 to R504, R506 to R505, R508 to R506, R509 to R507, R510 to R508, R512 to R509, R513 to R510, R514 to R511, R516 to R512, R517 to R513, SW302 to SW301, SW303 to SW302
Connections:
- C306 pad 1: Net-(C308-Pad1) -> /Host Controller/VOLTAGE_SENS_FLTR
- D301 pad 1: GND -> Net-(D301-K)
- D301 pad 2: Net-(D301-A) -> /Host Controller/LED1
- D302 pad 1: GND -> Net-(D302-K)
- D302 pad 2: Net-(D302-A) -> /Host Controller/LED2
- R304 pad 1: Net-(C308-Pad1) -> /Host Controller/VOLTAGE_SENS_FLTR
- R304 pad 2: unconnected-(R309-Pad2) -> /Host Controller/VOLTAGE_SENSE
- R310 pad 1: Net-(D301-A) -> GND
- R310 pad 2: /Host Controller/LED1 -> Net-(D301-K)
- R311 pad 1: Net-(D302-A) -> GND
- R311 pad 2: /Host Controller/LED2 -> Net-(D302-K)
- U302 pad 22: unconnected-(U302-PB10-Pad22) -> /Host Controller/ADDR_0
- U302 pad 23: unconnected-(U302-PB11-Pad23) -> /Host Controller/ADDR_1
- U302 pad 26: unconnected-(U302-PB14-Pad26) -> /Host Controller/ADDR_2
- U302 pad 30: unconnected-(U302-PC6-Pad30) -> /Host Controller/CURRENT_SENSE_FLTR
- U302 pad 31: unconnected-(U302-PC7-Pad31) -> /Host Controller/VOLTAGE_SENS_FLTR
Routing:
- net /Host Controller/LOW_POWER_ENABLE: track 18.0 -> 142.3 mm, vias 0 -> 3
- net /Host Controller/CURRENT_SENSE: track 0.00 -> 57.0 mm
- net /Host Controller/VOLTAGE_SENSE: track 15.2 -> 67.7 mm
- net /Display/LED_BRIGHTNESS: track 155.7 -> 191.1 mm
- net /Host Controller/I2C_SDA: track 145.3 -> 114.3 mm
- net /Host Controller/ADDR_0: track 0.00 -> 22.3 mm
- net /Host Controller/I2C_SCL: track 150.3 -> 130.2 mm
- net /Host Controller/ADDR_1: track 0.00 -> 19.5 mm
- net /Host Controller/ADDR_2: track 0.00 -> 19.4 mm
- net +3.3V: track 311.7 -> 330.9 mm, vias 19 -> 21
- net VBUS: track 121.4 -> 131.4 mm, vias 3 -> 2
- net /Host Controller/VOLTAGE_SENS_FLTR: track 0.00 -> 7.01 mm, vias 0 -> 1
- net /Host Controller/CURRENT_SENSE_FLTR: track 0.00 -> 5.34 mm, vias 0 -> 1
- net GND: track 146.4 -> 150.6 mm, vias 46 -> 58
- net /Display/VDD_DIG2: track 175.7 -> 179.5 mm
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- added copper zone on B.Cu, net Net-(U601-SW)
Other:
- board text added: "+3.3V"
- board text added: "BRIG."
- board text added: "BUS INPUT"
- board text added: "BUS OUTPUT"
- board text added: "GND"
- board text added: "I2C"
- board text added: "LOWP"
- board text added: "SCL"
- board text added: "SDA"
- board text added: "SWD"
- board text added: "USB C"
- board text added: "VBUS"
