File: KiCad/AstroWeather.kicad_pcb (KiCad board)
At the start: 6 copper layers, 185 x 30 mm, 127 parts, among them J101 I2C, J102 Conn_01x10, J103 SWD, J104 Conn_01x10, J105 AUX_POWER, J106 USB, Q501 Si2365EDS, Q502 Si2365EDS, Q503 Si2365EDS, Q504 Si2365EDS, Q505 Si2365EDS, Q506 BC847, Q507 BC847, Q508 BC847, Q509 BC847, Q701 IRLML2502, SW301 SW_Push, SW302 SW_Push, U101 INA180A2, U201 ST67W611, U301 AT24CS01-STUM, U302 STM32G0B1CETx, U501 SCT2024, U502 LFD028BUE-103A, U503 MCP6006T-E/OT, U504 LFD028BUE-103A, U505 SCT2024, U506 LED Matrix 5x7, U507 MCP6006T-E/OT, U508 LED Matrix 5x7, U509 LED Matrix 5x7, U510 SCT2167, U511 MCP6006T-E/OT, U512 LFD028BUE-103A, U513 SCT2024, U514 LFD028BUE-103A, U515 MCP6006T-E/OT, U601 TPS54302, U602 MCP1825S, Y301 24M

Commit message: KiCad work
Parts:
- C602: value 10u -> 10u/35V
- D501: moved to B.Cu
- L601: footprint Inductor_SMD:L_Wuerth_MAPI-4020 -> Inductor_SMD:L_Panasonic_PCC-M0630M
- moved R602 7.57 mm to (162.2, 64.0), turned to 180 degrees
- moved C608 6.85 mm to (162.2, 67.0)
- moved R601 6.85 mm to (160.2, 67.0)
- moved D501 6.21 mm to (159.4, 61.0)
- moved TP601 3.98 mm to (162.0, 73.8)
- moved L601 2.26 mm to (168.0, 75.6)
- moved C503 1.83 mm to (160.2, 56.4), turned to 0 degrees
- moved C602 1.64 mm to (170.5, 71.3)
- moved C601 1.59 mm to (166.8, 64.6)
- moved C603 1.59 mm to (170.6, 69.6)
- moved C604 1.59 mm to (167.5, 69.5)
- moved C605 1.59 mm to (165.1, 69.5)
- moved U601 1.59 mm to (170.4, 65.3)
- moved TP602 0.60 mm to (172.0, 57.6)
- moved TP503 0.50 mm to (89.0, 63.0)
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Routing:
- net VDD: track 50.8 -> 38.3 mm
- net /Display/VDD_LED: track 55.3 -> 50.1 mm, vias 1 -> 0
- net Net-(U601-FB): track 9.63 -> 14.3 mm
- net /Display/VDD_DIG2: track 179.5 -> 174.8 mm
- net GND: track 150.6 -> 148.3 mm
- net +3.3V: track 330.9 -> 332.8 mm
- net /Display/LED_BRIGHTNESS: track 191.1 -> 192.6 mm
- net /Display/VDD_DIG1: track 163.4 -> 164.3 mm, vias 3 -> 2
- net Net-(U601-SW): track 31.3 -> 32.2 mm
- net /Display/~{SCT_EN}: track 156.8 -> 157.4 mm
- net /Display/VDD_DIG4: track 160.7 -> 160.1 mm
- net /Display/~{SCT_LA}: track 163.0 -> 163.6 mm
- net /Display/SCT3_SDO: track 88.0 -> 88.5 mm
- net /Display/SCT_CLK_F: track 141.3 -> 141.8 mm
- added copper zone on F.Cu, net Net-(U601-SW)

Commit message: KiCad work
Parts:
- C303, C304: value 10p -> 20p
- C306, C307: value 100n -> 1u
- C603: value 100n -> 100n/35V
- L601: value 6u8 -> SRR6038-33u; footprint Inductor_SMD:L_Panasonic_PCC-M0630M -> Inductor_SMD:L_Bourns_SRP7028A_7.3x6.6mm
- Q501, Q502, Q503, Q504, Q505: value Si2365EDS -> Si2333DDS
- Q701: value IRLML2502 -> Si2374DS
- R304, R305: value ? -> 100k
- U501: value SCT2024 -> SCT2024CSSG
- Y301: value 24M -> Crystal_GND24_Small; footprint Crystal:Crystal_SMD_Abracon_ABM3-2Pin_5.0x3.2mm -> Crystal:Crystal_SMD_Abracon_ABM3B-4Pin_5.0x3.2mm
- moved C305 4.90 mm to (35.6, 57.0), turned to 180 degrees
- moved C303 4.44 mm to (45.2, 60.8)
- moved U601 0.80 mm to (170.4, 64.5)
- moved C602 0.80 mm to (170.5, 70.5)
- moved C603 0.80 mm to (170.6, 68.8)
- moved R303 0.58 mm to (41.7, 60.4)
- moved U302 0.50 mm to (46.5, 69.0)
- moved C301 0.45 mm to (48.2, 62.2)
- moved C302 0.45 mm to (48.5, 60.5)
- moved C608 0.40 mm to (162.2, 66.6)
- moved R601 0.40 mm to (160.2, 66.6)
- moved R602 0.40 mm to (162.2, 63.6)
- moved C601 0.40 mm to (166.8, 64.2)
- moved C604 0.40 mm to (167.5, 69.1)
- moved C605 0.40 mm to (165.1, 69.1)
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Connections:
- Y301 pad 1: Net-(C304-Pad2) -> /Host Controller/OSC_IN
- Y301 pad 2: /Host Controller/OSC_IN -> GND
Routing:
- net GND: track 148.3 -> 179.8 mm, vias 58 -> 71
- net /Host Controller/UCPD_CC2: track 64.5 -> 68.0 mm
- net Net-(U601-SW): track 32.2 -> 29.2 mm
- net +3.3V: track 332.8 -> 335.2 mm
- net /Host Controller/SWCLK: track 25.8 -> 24.0 mm
- net /Host Controller/SWDIO: track 29.4 -> 27.7 mm
- net /Host Controller/OSC_IN: track 10.1 -> 11.6 mm
- net Net-(C304-Pad2): track 6.07 -> 4.68 mm
- net /Host Controller/USB+: track 60.0 -> 58.9 mm
- net /Host Controller/I2C_SCL: track 130.2 -> 129.3 mm
- net /Host Controller/OSC_OUT: track 4.95 -> 5.57 mm
- net /Host Controller/ADDR_2: track 19.4 -> 18.9 mm
- net Net-(U601-FB): track 14.3 -> 14.8 mm
- net /Host Controller/ST67_TX: track 22.6 -> 23.1 mm
- net /Host Controller/LED2: track 18.0 -> 18.5 mm
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Other:
- board text added: "AstroWeater 4x4+3x5x7 v1 JP, 13.06.2026"

Commit message: KiCad work
Parts:
- C504, R502: moved to F.Cu
- moved R502 13.8 mm to (60.1, 67.1)
- moved C504 10.4 mm to (62.8, 64.0)
- moved Q701 0.26 mm to (58.5, 55.7)
- moved TP701 0.20 mm to (54.6, 65.0)
Routing:
- net /Display/SCT_CLK: track 24.4 -> 9.95 mm, vias 1 -> 0
- net /Display/SCT_CLK_F: track 141.7 -> 147.7 mm
- net /Host Controller/SWCLK: track 24.0 -> 26.7 mm
- net /Display/~{SCT_LA}: track 163.8 -> 166.2 mm
- net /Display/VDD_DIG1: track 164.3 -> 165.7 mm
- net GND: track 179.8 -> 181.0 mm, vias 71 -> 80
- net VBUS: track 132.0 -> 133.0 mm
- net /Host Controller/ST67_RX: track 22.9 -> 23.9 mm
- net /Display/SCT_SDI: track 20.4 -> 19.6 mm
- net /Display/DIS1_D: track 18.8 -> 19.6 mm
- net /Display/VDD_DIG2: track 174.8 -> 174.2 mm
- net +3.3V: track 335.2 -> 335.8 mm
- net /Display/SCT1_SDO: track 42.7 -> 43.3 mm
- net /Host Controller/SWDIO: track 27.7 -> 28.3 mm
- net /Display/DIS3_9: track 28.1 -> 27.5 mm
Other:
- board text added: "AstroWeater 4x4+3x5x7 v1 JP, 27.06.2026"
- board text added: "STM32G0B1CET6"
- board text removed: "AstroWeater 4x4+3x5x7 v1 JP, 13.06.2026"

Commit message: KiCad finishing touches, gerber
Parts:
- L601: value SRR6038-33u -> SRR6838-33u
Connections:
- net /Host Controller/VOLTAGE_SENSE renamed /VBUS_IN
Routing:
- net /VBUS_IN: track 67.7 -> 74.0 mm
- net VBUS: track 133.0 -> 134.8 mm, vias 2 -> 6
- net /Display/VDD_DIG4: track 160.1 -> 161.4 mm
- net /Display/DIS3_7: track 28.2 -> 29.5 mm
- net /Display/VDD_DIG3: track 177.5 -> 178.7 mm
- net /Display/VDD_DIG5: track 200.8 -> 201.7 mm
- net /Display/VDD_DIG2: track 174.2 -> 174.9 mm
- net /Display/DIS3_16: track 50.4 -> 49.8 mm
- net /Display/DIS3_3: track 22.2 -> 21.6 mm
- net /Display/~{SCT_EN}: track 157.5 -> 157.0 mm
- net /Display/SCT_CLK_F: track 147.7 -> 148.2 mm
- net GND: track 181.0 -> 181.1 mm, vias 80 -> 85
- added copper zone on B.Cu, net VBUS
- added copper zone on In2.Cu, net VBUS
- added copper zone on In3.Cu, net VBUS
Other:
- board text added: "24MHz"
