File: KiCad/Display.kicad_sch (KiCad schematic)
At the start: 74 parts, among them Q501 IRLML2502, Q502 Si2365EDS, Q503 Si2365EDS, Q504 Si2365EDS, Q505 Si2365EDS, Q506 Si2365EDS, Q507 IRLML2502, U501 SCT2024, U502 MCP6006T-E/OT, U503 LFD028BUE-103A, U504 LFD028BUE-103A, U505 LFD028BUE-103A, U506 LFD028BUE-103A, U507 KW3-281AVA, U508 KW3-281AVA, U509 KW3-281AVA, U510 KW3-281AVA, U511 MCP6006T-E/OT, U512 SCT2024, U513 LED Matrix 5x7, U514 LED Matrix 5x7, U515 LED Matrix 5x7

Commit message: KiCad work
Parts:
- removed D502, D503, D504, D505, D506, D507, D508, D509, D510, D511, D512, D513, D514, D515, D516, D517, D518, D519, D520, D521, D522, D523, D524, D525: LED, LED_THT:LED_D3.0mm, symbol Device:LED
- removed Q501: IRLML2502, Package_TO_SOT_SMD:SOT-23, symbol Transistor_FET:IRLML2060
- removed U505, U506: LFD028BUE-103A, JPDisplays:LFD028BUE-103A, symbol myLib:LFD028BUE-103A
- removed U507, U508, U509, U510: KW3-281AVA, JPDisplays:KW3-281AVA, symbol myLib:KW3-281AVA
- added C508, C510: 4u7, Capacitor_SMD:C_0805_2012Metric, symbol Device:C
- added C509: 1u, Capacitor_SMD:C_0805_2012Metric, symbol Device:C
- added Q501, Q508, Q509, Q510: BC847, Package_TO_SOT_SMD:SOT-23, symbol Transistor_BJT:BC847
- added R520, R521: 10, symbol Device:R
- added TP501, TP502, TP503, TP504, TP505: TestPoint, symbol Connector:TestPoint
- added U505: SCT2167, symbol myLib:SCT2167
- added U506, U509: MCP6006T-E/OT, Package_TO_SOT_SMD:SOT-23-5, symbol Amplifier_Operational:MCP6001-OT
- added U507, U508: LFD028BUE-103A, JPDisplays:LFD028BUE-103A, symbol myLib:LFD028BUE-103A
- added U510: SCT2024, Package_SO:SSOP-24_3.9x8.7mm_P0.635mm, symbol myLib:SCT2024
- C505: value 10p -> 1u
- C506: value 4u7 -> 1u
- C507: value 1u -> 4u7
- D501: value 1.5V-2V -> 1.5V-2V (short)
- R3: value 4k7 -> 1k5
- R502: value 100k -> 470k
- R503, R517: value 1k -> 4k7 / 10k
- R504: value 10k-100k -> 4k-2M
- R509: value dnp -> 3k2
- R510: value 0 -> 1k
- R511: value dnp -> 4k7 / 10k
- R512: value 4k7 -> dnp
- R513: value 4k7 -> 1k
- R514: value 4k7 -> 4k7 / 10k
- R515: value 1k -> dnp
Connections:
- net LINE1_1 is gone; now on net DIS3_1: U512.5 (Out0)
- net LINE1_10 is gone; now on net DIS3_10: U512.14 (Out9)
- net LINE1_11 is gone; now on net DIS3_11: U512.15 (Out10)
- net LINE1_12 is gone; now on net DIS3_12: U512.16 (Out11)
- net LINE1_13 is gone; now on net DIS3_13: U512.17 (Out12)
- net LINE1_14 is gone; now on net DIS3_14: U512.18 (Out13)
- net LINE1_15 is gone; now on net DIS3_15: U512.19 (Out14)
- net LINE1_16 is gone; now on net DIS3_16: U512.20 (Out15)
- net LINE1_2 is gone; now on net DIS3_2: U512.6 (Out1)
- net LINE1_3 is gone; now on net DIS3_3: U512.7 (Out2)
- net LINE1_4 is gone; now on net DIS3_4: U512.8 (Out3)
- net LINE1_5 is gone; now on net DIS3_5: U512.9 (Out4)
- net LINE1_6 is gone; now on net DIS3_6: U512.10 (Out5)
- net LINE1_7 is gone; now on net DIS3_7: U512.11 (Out6)
- net LINE1_8 is gone; now on net DIS3_8: U512.12 (Out7)
- net LINE1_9 is gone; now on net DIS3_9: U512.13 (Out8)
- net !SCT_EN: now also U505.13 (!OE), U510.21 (!OE)
- net !SCT_LA: now also U505.4 (!LA), U510.4 (!LA)
- net +3.3V: now also C505.1, R501.1, U502.5 (V+), U511.5 (V+), C508.1, C509.1, C510.1, R520.1, R521.1, U506.5 (V+), U509.5 (V+); no longer R512.1, R513.1
- net DIS3_17: now also U505.5 (Out0)
- net DIS3_18: now also U505.6 (Out1)
- net DIS3_19: now also U505.7 (Out2)
- net DIS3_20: now also U505.8 (Out3)
- net DIS3_21: now also U505.9 (Out4)
- net GND: now also Q507.2 (S), R509.1, R512.2, R514.2, R515.2, C508.2, C509.2, C510.2, U505.1 (GND), U506.2 (V-), U509.2 (V-), U510.1 (GND); no longer R510.2
- net SCT_CLK: no longer R515.2
- net STC_SDI: no longer U512.2 (SDI)
- net VDD: no longer U502.5 (V+), U511.5 (V+)
- net at U511.1: now also Q508.1 (B); no longer Q507.1 (G)
- net at R516.1, R517.1: now also Q508.2 (E), TP501.1; no longer Q507.2 (S)
- net at R518.1, U512.23 (Rext): now also Q508.3 (C); no longer Q507.3 (D)
- net at U513.1 (COL1): now also Q502.3 (D), U503.1 (Dig1), U504.1 (Dig1), U514.1 (COL1), U515.1 (COL1), U507.1 (Dig1), U508.1 (Dig1)
- net at U513.10 (COL3): now also Q504.3 (D), U503.11 (Dig3), U504.11 (Dig3), U514.10 (COL3), U515.10 (COL3), U507.11 (Dig3), U508.11 (Dig3)
- net at U513.3 (COL2): now also Q503.3 (D), U503.14 (Dig2), U504.14 (Dig2), U514.3 (COL2), U515.3 (COL2), U507.14 (Dig2), U508.14 (Dig2)
- net at U513.7 (COL4): now also Q505.3 (D), U503.8 (Dig4), U504.8 (Dig4), U514.7 (COL4), U515.7 (COL4), U507.8 (Dig4), U508.8 (Dig4)
- net at U513.8 (COL5): now also Q506.3 (D), U503.12 (L), U504.12 (L), U514.8 (COL5), U515.8 (COL5), U507.12 (L), U508.12 (L)
- net at C503.1, R508.1, U501.3 (CLK): now also U512.3 (CLK), U505.3 (CLK), U510.3 (CLK)
- net at R3.2, R509.2: now also Q507.3 (D); no longer R510.1, R511.1
- net at R501.2, R504.1: no longer R514.2
- net at R506.1, U501.23 (Rext): now also Q501.3 (C)
- net at U512.22 (SDO): now also U505.2 (SDI), U510.2 (SDI)
- net at R503.1, R505.1: now also Q501.2 (E), TP502.1
- net at U501.22 (SDO): now also U512.2 (SDI)
- net at U502.1: now also Q501.1 (B)
- net LED_BRIGHT renamed LED_BRIGHTNESS
- net LED_BRIGHTNESS: now also TP505.1, U506.3 (+), U509.3 (+); no longer R509.1
- new net: R520.2, U510.24 (VDD)
- new net: Q509.3 (C), R512.1, U505.15 (Rext)
- new net: R521.2, U505.16 (VDD)
- new net: Q509.2 (E), R510.1, R511.1, TP503.1
- new net: Q510.1 (B), U509.1
- new net: R513.2, U509.4 (-)
- new net: Q509.1 (B), U506.1
- new net: Q510.2 (E), R513.1, R514.1, TP504.1
- new net: Q510.3 (C), R515.1, U510.23 (Rext)
- new net: R510.2, U506.4 (-)
- new net DIS4_A: U507.13 (A), U510.5 (Out0)
- new net DIS4_B: U507.15 (B), U510.6 (Out1)
- new net DIS4_C: U507.2 (C), U510.7 (Out2)
- new net DIS4_D: U507.6 (D), U510.8 (Out3)
- new net DIS4_DP: U507.3 (DP), U510.12 (Out7)
- new net DIS4_E: U507.5 (E), U510.9 (Out4)
- new net DIS4_F: U507.16 (F), U510.10 (Out5)
- new net DIS4_G: U507.7 (G), U510.11 (Out6)
- new net DIS5_A: U508.13 (A), U510.13 (Out8)
- new net DIS5_B: U508.15 (B), U510.14 (Out9)
- new net DIS5_C: U508.2 (C), U510.15 (Out10)
- new net DIS5_D: U508.6 (D), U510.16 (Out11)
- new net DIS5_DP: U508.3 (DP), U510.20 (Out15)
- new net DIS5_E: U508.5 (E), U510.17 (Out12)
- new net DIS5_F: U508.16 (F), U510.18 (Out13)
- new net DIS5_G: U508.7 (G), U510.19 (Out14)
- new net LOW_POWER_ENABLE: Q507.1 (G)
- no-connect marks 0 -> 1
Other:
- note added: "Isense: 0.012mA - 0.262mA Iout: 0.2mA - 4mA Ur:0.06V - 1.2V"
- moved on the sheet: C503, C504, D501, Q502, Q503, Q504, Q505, Q506, Q507, R3, R501, R502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

Commit message: KiCad work
Connections:
- net !SCT_EN renamed ~{SCT_EN}
- net !SCT_LA renamed ~{SCT_LA}
Changed lines of the file:
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@@
 		)
 	)
-	(hierarchical_label "!SCT_EN"
+	(hierarchical_label "~{SCT_EN}"
 		(shape input)
-		(at 82.55 281.94 180)
+		(at 82.55 353.06 180)
 		(effects
 			(font
@@
 		)
 	)
-	(hierarchical_label "Gnd"
+	(hierarchical_label "GND"
 		(shape input)
 		(at 38.1 49.53 180)
@@
 		)
 	)
-	(hierarchical_label "!SCT_EN"
-		(shape input)
-		(at 82.55 209.55 180)
-		(effects
-			(font
-				(size 1.27 1.27)
-			)
-			(justify right)
-		)
-	)
 	(hierarchical_label "DIS2_EN"
 		(shape input)
@@
 		)
 	)
+	(hierarchical_label "~{SCT_EN}"
+		(shape input)
+		(at 82.55 281.94 180)
+		(effects
+			(font
+				(size 1.27 1.27)
+			)
+			(justify right)
+		)
+	)
 	(hierarchical_label "+3.3V"
 		(shape input)
 		(at 38.1 45.72 180)
+		(effects
+			(font
+				(size 1.27 1.27)
+			)
+			(justify right)
+		)
+	)
+	(hierarchical_label "~{SCT_LA}"
+		(shape input)
+		(at 82.55 284.48 180)
+		(effects
+			(font
+				(size 1.27 1.27)
+			)
+			(justify right)
+		)
+	)
+	(hierarchical_label "~{SCT_LA}"
+		(shape input)
+		(at 82.55 212.09 180)
 		(effects
 			(font
@@
 		)
 	)
-	(hierarchical_label "!SCT_LA"
-		(shape input)
-		(at 82.55 212.09 180)
-		(effects
-			(font
-				(size 1.27 1.27)
-			)
-			(justify right)
-		)
-	)
-	(hierarchical_label "!SCT_LA"
+	(hierarchical_label "~{SCT_LA}"
 		(shape input)
 		(at 83.82 130.81 180)
@@
 		)
 	)
-	(hierarchical_label "!SCT_LA"
-		(shape input)
-		(at 82.55 284.48 180)
-		(effects
-			(font
-				(size 1.27 1.27)
-			)
-			(justify right)
-		)
-	)
-	(hierarchical_label "Vdd"
+	(hierarchical_label "VLED"
 		(shape input)
 		(at 38.1 41.91 180)
@@
 		)
 	)
-	(hierarchical_label "!SCT_EN"
+	(hierarchical_label "~{SCT_EN}"
 		(shape input)
-		(at 82.55 353.06 180)
+		(at 82.55 209.55 180)
 		(effects
 			(font
@@
 		)
 	)
-	(hierarchical_label "!SCT_LA"
+	(hierarchical_label "~{SCT_EN}"
 		(shape input)
-		(at 82.55 355.6 180)
+		(at 83.82 128.27 180)
 		(effects
 			(font
@@
 		)
 	)
-	(hierarchical_label "!SCT_EN"
+	(hierarchical_label "~{SCT_LA}"
 		(shape input)
-		(at 83.82 128.27 180)
+		(at 82.55 355.6 180)
 		(effects
 			(font

Commit message: KiCad work
Connections:
- net STC_SDI renamed SCT_SDI
Changed lines of the file:
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@@
 		)
 	)
-	(hierarchical_label "STC_SDI"
+	(hierarchical_label "SCT_SDI"
 		(shape input)
 		(at 87.63 115.57 180)

Commit message: KiCad work
Parts:
- removed Q507: IRLML2502, Package_TO_SOT_SMD:SOT-23, symbol Transistor_FET:IRLML2060
- removed R3: 1k5, symbol Device:R
- removed R501: 4k7, symbol Device:R
- removed R502: 470k, symbol Device:R
- removed R504: 4k-2M, symbol Device:R_Photo
- removed R509: 3k2, symbol Device:R
- removed TP505: TestPoint, symbol Connector:TestPoint
- D501: footprint (none) -> Diode_SMD:D_SMA
- R501: renamed from R507; footprint (none) -> Resistor_SMD:R_0805_2012Metric
- R502: renamed from R508; footprint (none) -> Resistor_SMD:R_0805_2012Metric
- R503: renamed from R506; footprint (none) -> Resistor_SMD:R_0805_2012Metric
- R504: renamed from R505; footprint (none) -> Resistor_SMD:R_0805_2012Metric
- R505: renamed from R503; footprint (none) -> Resistor_SMD:R_0805_2012Metric
- R506: renamed from R519; footprint (none) -> Resistor_SMD:R_0805_2012Metric
- R507: renamed from R518; footprint (none) -> Resistor_SMD:R_0805_2012Metric
- R508: renamed from R516; footprint (none) -> Resistor_SMD:R_0805_2012Metric
- R509: renamed from R517; footprint (none) -> Resistor_SMD:R_0805_2012Metric
- R510: renamed from R521; footprint (none) -> Resistor_SMD:R_0805_2012Metric
- R511: renamed from R512; footprint (none) -> Resistor_SMD:R_0805_2012Metric
- R512: renamed from R510; footprint (none) -> Resistor_SMD:R_0805_2012Metric
- R513: renamed from R511; footprint (none) -> Resistor_SMD:R_0805_2012Metric
- R514: renamed from R520; footprint (none) -> Resistor_SMD:R_0805_2012Metric
- R515: footprint (none) -> Resistor_SMD:R_0805_2012Metric
- R516: renamed from R513; footprint (none) -> Resistor_SMD:R_0805_2012Metric
- R517: renamed from R514; footprint (none) -> Resistor_SMD:R_0805_2012Metric
- TP501: renamed from TP502; footprint (none) -> TestPoint:TestPoint_THTPad_D1.5mm_Drill0.7mm
- TP502: renamed from TP501; footprint (none) -> TestPoint:TestPoint_THTPad_D1.5mm_Drill0.7mm
- TP503, TP504: footprint (none) -> TestPoint:TestPoint_THTPad_D1.5mm_Drill0.7mm
- U506: renamed from U513; footprint (none) -> JPDisplays:FYM-7571A
- U508: renamed from U514; footprint (none) -> JPDisplays:FYM-7571A
- U509: renamed from U515; footprint (none) -> JPDisplays:FYM-7571A
- U510: renamed from U505; footprint (none) -> Package_SO:SSOP-16_3.9x4.9mm_P0.635mm
- renumbered C504 to C503, C503 to C504, C506 to C505, C507 to C506, C509 to C507, C510 to C508, C505 to C509, C508 to C510, Q502 to Q501, Q503 to Q502, Q504 to Q503, Q505 to Q504, Q506 to Q505, Q501 to Q506, Q508 to Q507, Q509 to Q508, Q510 to Q509, U503 to U502, U502 to U503, U512 to U505, U511 to U507, U506 to U511, U507 to U512, U510 to U513, U508 to U514, U509 to U515

Commit message: KiCad work
Connections:
- net +3.3V: no longer C501.1, C502.1
- net SCT1_REXT: now reaches Q506.3 (C), R503.1, U501.23 (Rext)
- net SCT1_VDD: now reaches R501.2, U501.24 (VDD)
- net SCT1_VDD: now also C501.1, C502.1
- net SCT_SDO: now reaches U513.22 (SDO)
- no-connect marks 1 -> 0
Other:
- moved on the sheet: R501
Changed lines of the file:
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@@
 		(color 0 0 0 0)
 	)
-	(no_connect
-		(at 91.44 342.9)
-	)
 	(bus_entry
 		(at 146.05 361.95)
@@
 	(wire
 		(pts
+			(xy 102.87 74.93) (xy 102.87 76.2)
+		)
+		(stroke
+			(width 0)
+			(type default)
+		)
+	)
+	(wire
+		(pts
 			(xy 238.76 132.08) (xy 238.76 120.65)
 		)
@@
 	(wire
 		(pts
-			(xy 102.87 85.09) (xy 102.87 86.36)
-		)
-		(stroke
-			(width 0)
-			(type default)
-		)
-	)
-	(wire
-		(pts
 			(xy 60.96 153.67) (xy 66.04 153.67)
 		)
@@
 	(wire
 		(pts
+			(xy 82.55 342.9) (xy 91.44 342.9)
+		)
+		(stroke
+			(width 0)
+			(type default)
+		)
+	)
+	(wire
+		(pts
 			(xy 82.55 355.6) (xy 91.44 355.6)
 		)
@@
 	(wire
 		(pts
-			(xy 102.87 93.98) (xy 102.87 102.87)
+			(xy 102.87 85.09) (xy 102.87 102.87)
 		)
 		(stroke
@@
 		)
 	)
+	(label "SCT1_REXT"
+		(at 68.58 137.16 0)
+		(effects
+			(font
+				(size 1.27 1.27)
+			)
+			(justify left bottom)
+		)
+	)
 	(label "DIS1_DP"
 		(at 115.57 124.46 0)
@@
 		)
 	)
+	(label "SCT1_VDD"
+		(at 110.49 85.09 0)
+		(effects
+			(font
+				(size 1.27 1.27)
+			)
+			(justify left bottom)
+		)
+	)
 	(label "DIS3_3"
 		(at 123.19 193.04 180)
@@
 		)
 	)
+	(hierarchical_label "SCT_SDO"
+		(shape output)
+		(at 82.55 342.9 180)
+		(effects
+			(font
+				(size 1.27 1.27)
+			)
+			(justify right)
+		)
+	)
 	(hierarchical_label "~{SCT_EN}"
 		(shape input)
@@
 	(symbol
 		(lib_id "power:+3.3V")
-		(at 102.87 83.82 0)
+		(at 102.87 74.93 0)
 		(unit 1)
 		(exclude_from_sim no)
@@
 		(fields_autoplaced yes)
 		(property "Reference" "#PWR0505"
-			(at 102.87 87.63 0)
+			(at 102.87 78.74 0)
 			(effects
 				(font
@@
 		)
 		(property "Value" "+3.3V"
-			(at 102.87 78.74 0)
+			(at 102.87 69.85 0)
 			(effects
 				(font
@@
 		)
 		(property "Footprint" ""
-			(at 102.87 83.82 0)
+			(at 102.87 74.93 0)
 			(effects
 				(font
@@
 		)
 		(property "Datasheet" ""
-			(at 102.87 83.82 0)
+			(at 102.87 74.93 0)
 			(effects
 				(font
@@
 		)
 		(property "Description" "Power symbol creates a global label with name \"+3.3V\""
-			(at 102.87 83.82 0)
+			(at 102.87 74.93 0)
 			(effects
 				(font
@@
 	(symbol
 		(lib_id "Device:R")
-		(at 102.87 90.17 0)
+		(at 102.87 80.01 0)
 		(unit 1)
 		(exclude_from_sim no)
@@
 		(dnp no)
 		(property "Reference" "R501"
-			(at 96.012 88.9 0)
+			(at 96.012 78.74 0)
 			(effects
 				(font
@@
 		)
 		(property "Value" "10"
-			(at 98.552 91.694 0)
+			(at 98.552 81.534 0)
 			(effects
 				(font
@@
 		)
 		(property "Footprint" "Resistor_SMD:R_0805_2012Metric"
-			(at 101.092 90.17 90)
+			(at 101.092 80.01 90)
 			(effects
 				(font
@@
 		)
 		(property "Datasheet" "~"
-			(at 102.87 90.17 0)
+			(at 102.87 80.01 0)
 			(effects
 				(font
@@
 		)
 		(property "Description" "Resistor"
-			(at 102.87 90.17 0)
+			(at 102.87 80.01 0)
 			(effects
 				(font

Commit message: Work
Parts:
- TP501, TP502, TP503, TP504: footprint TestPoint:TestPoint_THTPad_D1.5mm_Drill0.7mm -> TestPoint:TestPoint_Pad_D1.5mm
Connections:
- net +3.3V: no longer C505.1, C506.1, C507.1, C508.1, C509.1, C510.1
- net DIS1_A: now also U501.7 (Out2); no longer U501.5 (Out0)
- net DIS1_C: now also U501.9 (Out4); no longer U501.7 (Out2)
- net DIS1_DP: now also U501.10 (Out5); no longer U501.12 (Out7)
- net DIS1_E: now also U501.11 (Out6); no longer U501.9 (Out4)
- net DIS1_F: now also U501.5 (Out0); no longer U501.10 (Out5)
- net DIS1_G: now also U501.12 (Out7); no longer U501.11 (Out6)
- net DIS2_A: now also U501.18 (Out13); no longer U501.13 (Out8)
- net DIS2_B: now also U501.19 (Out14); no longer U501.14 (Out9)
- net DIS2_C: now also U501.14 (Out9); no longer U501.15 (Out10)
- net DIS2_DP: now also U501.13 (Out8); no longer U501.20 (Out15)
- net DIS2_E: now also U501.15 (Out10); no longer U501.17 (Out12)
- net DIS2_F: now also U501.20 (Out15); no longer U501.18 (Out13)
- net DIS2_G: now also U501.17 (Out12); no longer U501.19 (Out14)
- net DIS4_C: now also U513.8 (Out3); no longer U513.7 (Out2)
- net DIS4_D: now also U513.11 (Out6); no longer U513.8 (Out3)
- net DIS4_DP: now also U513.9 (Out4); no longer U513.12 (Out7)
- net DIS4_E: now also U513.10 (Out5); no longer U513.9 (Out4)
- net DIS4_F: now also U513.7 (Out2); no longer U513.10 (Out5)
- net DIS4_G: now also U513.12 (Out7); no longer U513.11 (Out6)
- net DIS5_C: now also U513.20 (Out15); no longer U513.15 (Out10)
- net DIS5_D: now also U513.17 (Out12); no longer U513.16 (Out11)
- net DIS5_DP: now also U513.19 (Out14); no longer U513.20 (Out15)
- net DIS5_E: now also U513.18 (Out13); no longer U513.17 (Out12)
- net DIS5_F: now also U513.15 (Out10); no longer U513.18 (Out13)
- net DIS5_G: now also U513.16 (Out11); no longer U513.19 (Out14)
- net VDD_DIG1: now reaches Q501.3 (D), U502.1 (Dig1), U504.1 (Dig1), U506.1 (COL1), U508.1 (COL1), U509.1 (COL1), U512.1 (Dig1), U514.1 (Dig1)
- net VDD_DIG3: now reaches Q503.3 (D), U502.11 (Dig3), U504.11 (Dig3), U506.10 (COL3), U508.10 (COL3), U509.10 (COL3), U512.11 (Dig3), U514.11 (Dig3)
- net VDD_DIG2: now reaches Q502.3 (D), U502.14 (Dig2), U504.14 (Dig2), U506.3 (COL2), U508.3 (COL2), U509.3 (COL2), U512.14 (Dig2), U514.14 (Dig2)
- net VDD_DIG4: now reaches Q504.3 (D), U502.8 (Dig4), U504.8 (Dig4), U506.7 (COL4), U508.7 (COL4), U509.7 (COL4), U512.8 (Dig4), U514.8 (Dig4)
- net VDD_DIG5: now reaches Q505.3 (D), U502.12 (L), U504.12 (L), U506.8 (COL5), U508.8 (COL5), U509.8 (COL5), U512.12 (L), U514.12 (L)
- net SCT_CLK_F: now reaches C504.1, R502.1, U501.3 (CLK), U505.3 (CLK), U510.3 (CLK), U513.3 (CLK)
- net SCT4_VDD: now reaches R514.2, U513.24 (VDD)
- net SCT4_VDD: now also C509.1, C510.1
- net VDD_LED: now reaches C503.1, D501.2 (A), Q501.2 (S), Q502.2 (S), Q503.2 (S), Q504.2 (S), Q505.2 (S)
- net SCT3_SDO: now reaches U510.14 (SDO)
- net SCT3_SDO: now also U513.2 (SDI)
- net SCT3_REXT: now reaches Q508.3 (C), R511.1, U510.15 (Rext)
- net SCT3_VDD: now reaches R510.2, U510.16 (VDD)
- net SCT3_VDD: now also C507.1, C508.1
- net SCT2_SDO: now reaches U505.22 (SDO), U510.2 (SDI)
- net SCT2_SDO: no longer U513.2 (SDI)
- net SCT2_REXT: now reaches Q507.3 (C), R507.1, U505.23 (Rext)
- net SCT4_REXT: now reaches Q509.3 (C), R515.1, U513.23 (Rext)
- net SCT1_SDO: now reaches U501.22 (SDO), U505.2 (SDI)
- net SCT2_VDD: now reaches R506.2, U505.24 (VDD)
- net SCT2_VDD: now also C505.1, C506.1
- net DIS1_EN renamed DISPLAY1_EN
- net DIS2_EN renamed DISPLAY2_EN
- net DIS3_EN renamed DISPLAY3_EN
- net DIS4_EN renamed DISPLAY4_EN
- net DIS5_EN renamed DISPLAY5_EN
Other:
- note added: "R=4.7k Isense: 0.012mA - 0.262mA Iout: 0.2mA - 4mA Ur:0.06V - 1.2V"
- note removed: "Isense: 0.012mA - 0.262mA Iout: 0.2mA - 4mA Ur:0.06V - 1.2V"
- moved on the sheet: C505, C506, C507, C508, C509, C510

Commit message: KiCad work
Parts:
- removed R503, R507, R511, R515: dnp, Resistor_SMD:R_0805_2012Metric, symbol Device:R

Commit message: KiCad work
Parts:
- renumbered C506 to C505, C505 to C506, C508 to C507, C507 to C508, C510 to C509, C509 to C510, R504 to R503, R505 to R504, R506 to R505, R508 to R506, R509 to R507, R510 to R508, R512 to R509, R513 to R510, R514 to R511, R516 to R512, R517 to R513
Other:
- note added: "52 Leds * 4mA = 208mA"
