File: KiCad/Display.kicad_sch (KiCad schematic)
At the start: 52 parts, among them Q501 Si2365EDS, Q502 Si2365EDS, Q503 Si2365EDS, Q504 Si2365EDS, Q505 Si2365EDS, Q506 BC847, Q507 BC847, Q508 BC847, Q509 BC847, U501 SCT2024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

Commit message: KiCad work
Parts:
- Q501, Q502, Q503, Q504, Q505: value Si2365EDS -> Si2333DDS
- U501: value SCT2024 -> SCT2024CSSG
Other:
- note added: "Voltage on SCT Vout ~ 1V Iled: 0.2-4mA LEDs on (max) 4*8+3*7=53 Iled(max): 53*4mA = 212mA"
- note removed: "Voltage on SCT Vout ~ 1V"
Changed lines of the file:
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@@
 		)
 	)
-	(text "Voltage on SCT\nVout ~ 1V"
+	(text "Voltage on SCT\nVout ~ 1V\n\nIled: 0.2-4mA\nLEDs on (max) 4*8+3*7=53\nIled(max): 53*4mA = 212mA"
 		(exclude_from_sim no)
-		(at 132.842 107.188 0)
+		(at 142.24 81.28 0)
 		(effects
 			(font
 				(size 1.27 1.27)
 			)
-			(justify left)
+			(justify left top)
 		)
 	)
@@
 			)
 		)
-		(property "Value" "Si2365EDS"
+		(property "Value" "Si2333DDS"
 			(at 214.63 101.5999 0)
 			(effects
@@
 			)
 		)
-		(property "Value" "Si2365EDS"
+		(property "Value" "Si2333DDS"
 			(at 255.27 132.0799 0)
 			(effects
@@
 			)
 		)
-		(property "Value" "SCT2024"
+		(property "Value" "SCT2024CSSG"
 			(at 104.8386 102.87 0)
 			(effects
@@
 			)
 		)
-		(property "Value" "Si2365EDS"
+		(property "Value" "Si2333DDS"
 			(at 245.11 124.4599 0)
 			(effects
@@
 			)
 		)
-		(property "Value" "Si2365EDS"
+		(property "Value" "Si2333DDS"
 			(at 224.79 109.2199 0)
 			(effects
@@
 			)
 		)
-		(property "Value" "Si2365EDS"
+		(property "Value" "Si2333DDS"
 			(at 234.95 116.8399 0)
 			(effects
