File: KiCad/PowerSupply.kicad_sch (KiCad schematic)
At the start: 0 parts

Commit message: KiCad work
Parts:
- added C601, C602: 100n, symbol Device:C
- added C603, C604: 22u, symbol Device:C
- added C605: 10u, symbol Device:C
- added C606: 47p, symbol Device:C
- added C607: 4u7, symbol Device:C
- added C608: 1u, symbol Device:C
- added L601: 6u8, symbol Device:L
- added R601: 511k, symbol Device:R
- added R602, R603, R604: R, symbol Device:R
- added R605: 105k, symbol Device:R
- added TP601, TP602: TestPoint, symbol Connector:TestPoint
- added U601: TPS54302, Package_TO_SOT_SMD:SOT-23-6, symbol Regulator_Switching:TPS54302
- added U603: MCP1825S, symbol Regulator_Linear:MCP1825S
Connections:
- new net: C602.2, L601.1, U601.2 (SW)
- new net: C606.2, R603.2, R604.1, U601.4 (FB)
- new net: R601.1, R605.1, U601.5 (EN)
- new net: C602.1, U601.6 (BOOT)
- new net: C606.1, R602.2, R603.1
- new net +3.3V: C608.1, TP602.1, U603.3 (VO)
- new net +3.7V: C603.1, C604.1, C607.1, L601.2, R602.1, TP601.1, U603.1 (VI)
- new net GND: C601.2, C603.2, C604.2, C605.1, C607.2, C608.2, R604.2, R605.2, U601.1 (GND), U603.2 (GND)
- new net VDD: C601.1, C605.2, R601.2, U601.3 (VIN)

Commit message: KiCad work
Parts:
- removed R601: 511k, symbol Device:R
- removed R602: R, symbol Device:R
- removed R605: 105k, symbol Device:R
- R603: value R -> 100k
- R604: value R -> 19k2
Connections:
- net +3.7V: now also C606.1, R603.1
- no-connect marks 0 -> 1
Other:
- moved on the sheet: C601, C605, C606, R603

Commit message: KiCad work
Parts:
- C601: renamed from C602; footprint (none) -> Capacitor_SMD:C_0201_0603Metric
- C602: renamed from C605; footprint (none) -> Capacitor_SMD:C_0805_2012Metric
- C603: renamed from C601; footprint (none) -> Capacitor_SMD:C_0603_1608Metric
- C604: renamed from C603; footprint (none) -> Capacitor_SMD:C_1206_3216Metric
- C605: renamed from C604; footprint (none) -> Capacitor_SMD:C_1206_3216Metric
- C606: renamed from C607; footprint (none) -> Capacitor_SMD:C_0805_2012Metric
- C607: renamed from C608; footprint (none) -> Capacitor_SMD:C_0805_2012Metric
- C608: renamed from C606; footprint (none) -> Capacitor_SMD:C_0805_2012Metric
- L601: footprint (none) -> Inductor_SMD:L_7.3x7.3_H4.5
- R601: renamed from R603; footprint (none) -> Resistor_SMD:R_0805_2012Metric
- R602: renamed from R604; footprint (none) -> Resistor_SMD:R_0805_2012Metric
- TP601, TP602: footprint (none) -> TestPoint:TestPoint_THTPad_D1.5mm_Drill0.7mm
- U602: renamed from U603; footprint (none) -> Package_TO_SOT_SMD:SOT-223-3_TabPin2
Changed lines of the file:
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@@
 			)
 		)
-		(property "Footprint" ""
+		(property "Footprint" "Inductor_SMD:L_7.3x7.3_H4.5"
 			(at 134.62 93.98 0)
 			(effects
@@
 		(dnp no)
 		(fields_autoplaced yes)
-		(property "Reference" "#PWR0611"
+		(property "Reference" "#PWR0612"
 			(at 191.77 110.49 0)
 			(effects
@@
 			(project "AstroWeather"
 				(path "/8561283c-f5b3-4542-8880-7f435c3a9f7c/50b8a1dd-352e-4a33-913d-a72ec72f4116"
-					(reference "#PWR0611")
+					(reference "#PWR0612")
 					(unit 1)
 				)
@@
 		(dnp no)
 		(fields_autoplaced yes)
-		(property "Reference" "C608"
+		(property "Reference" "C607"
 			(at 226.06 97.7899 0)
 			(effects
@@
 			)
 		)
-		(property "Footprint" ""
+		(property "Footprint" "Capacitor_SMD:C_0805_2012Metric"
 			(at 223.2152 102.87 0)
 			(effects
@@
 			(project "AstroWeather"
 				(path "/8561283c-f5b3-4542-8880-7f435c3a9f7c/50b8a1dd-352e-4a33-913d-a72ec72f4116"
-					(reference "C608")
+					(reference "C607")
 					(unit 1)
 				)
@@
 		(dnp no)
 		(fields_autoplaced yes)
-		(property "Reference" "#PWR0608"
+		(property "Reference" "#PWR0610"
 			(at 140.97 110.49 0)
 			(effects
@@
 			(project "AstroWeather"
 				(path "/8561283c-f5b3-4542-8880-7f435c3a9f7c/50b8a1dd-352e-4a33-913d-a72ec72f4116"
-					(reference "#PWR0608")
+					(reference "#PWR0610")
 					(unit 1)
 				)
@@
 		(dnp no)
 		(fields_autoplaced yes)
-		(property "Reference" "U603"
+		(property "Reference" "U602"
 			(at 208.28 87.63 0)
 			(effects
@@
 			)
 		)
-		(property "Footprint" ""
+		(property "Footprint" "Package_TO_SOT_SMD:SOT-223-3_TabPin2"
 			(at 205.74 90.17 0)
 			(effects
@@
 			(project ""
 				(path "/8561283c-f5b3-4542-8880-7f435c3a9f7c/50b8a1dd-352e-4a33-913d-a72ec72f4116"
-					(reference "U603")
+					(reference "U602")
 					(unit 1)
 				)
@@
 		(dnp no)
 		(fields_autoplaced yes)
-		(property "Reference" "R603"
+		(property "Reference" "R601"
 			(at 176.53 99.0599 0)
 			(effects
@@
 			)
 		)
-		(property "Footprint" ""
+		(property "Footprint" "Resistor_SMD:R_0805_2012Metric"
 			(at 172.212 100.33 90)
 			(effects
@@
 			(project "AstroWeather"
 				(path "/8561283c-f5b3-4542-8880-7f435c3a9f7c/50b8a1dd-352e-4a33-913d-a72ec72f4116"
-					(reference "R603")
+					(reference "R601")
 					(unit 1)
 				)
@@
 		(dnp no)
 		(fields_autoplaced yes)
-		(property "Reference" "C603"
+		(property "Reference" "C604"
 			(at 144.78 97.7899 0)
 			(effects
@@
 			)
 		)
-		(property "Footprint" ""
+		(property "Footprint" "Capacitor_SMD:C_1206_3216Metric"
 			(at 141.9352 102.87 0)
 			(effects
@@
 			(project "AstroWeather"
 				(path "/8561283c-f5b3-4542-8880-7f435c3a9f7c/50b8a1dd-352e-4a33-913d-a72ec72f4116"
-					(reference "C603")
+					(reference "C604")
 					(unit 1)
 				)
@@
 			)
 		)
-		(property "Footprint" ""
+		(property "Footprint" "TestPoint:TestPoint_THTPad_D1.5mm_Drill0.7mm"
 			(at 232.41 92.71 0)
 			(effects
@@
 		(dnp no)
 		(fields_autoplaced yes)
-		(property "Reference" "#PWR0609"
+		(property "Reference" "#PWR0611"
 			(at 152.4 110.49 0)
 			(effects
@@
 			(project "AstroWeather"
 				(path "/8561283c-f5b3-4542-8880-7f435c3a9f7c/50b8a1dd-352e-4a33-913d-a72ec72f4116"
-					(reference "#PWR0609")
+					(reference "#PWR0611")
 					(unit 1)
 				)
@@
 			)
 		)
-		(property "Footprint" ""
+		(property "Footprint" "TestPoint:TestPoint_THTPad_D1.5mm_Drill0.7mm"
 			(at 162.56 91.44 0)
 			(effects
@@
 		(dnp no)
 		(fields_autoplaced yes)
-		(property "Reference" "#PWR0614"
+		(property "Reference" "#PWR0605"
 			(at 242.57 93.98 0)
 			(effects
@@
 			(project ""
 				(path "/8561283c-f5b3-4542-8880-7f435c3a9f7c/50b8a1dd-352e-4a33-913d-a72ec72f4116"
-					(reference "#PWR0614")
+					(reference "#PWR0605")
 					(unit 1)
 				)
@@
 		(dnp no)
 		(fields_autoplaced yes)
-		(property "Reference" "C606"
+		(property "Reference" "C608"
 			(at 170.18 107.9499 0)
 			(effects
@@
 			)
 		)
-		(property "Footprint" ""
+		(property "Footprint" "Capacitor_SMD:C_0805_2012Metric"
 			(at 167.3352 113.03 0)
 			(effects
@@
 			(project "AstroWeather"
 				(path "/8561283c-f5b3-4542-8880-7f435c3a9f7c/50b8a1dd-352e-4a33-913d-a72ec72f4116"
-					(reference "C606")
+					(reference "C608")
 					(unit 1)
 				)
@@
 		(dnp no)
 		(fields_autoplaced yes)
-		(property "Reference" "#PWR0612"
+		(property "Reference" "#PWR0609"
 			(at 208.28 109.22 0)
 			(effects
@@
 			(project "AstroWeather"
 				(path "/8561283c-f5b3-4542-8880-7f435c3a9f7c/50b8a1dd-352e-4a33-913d-a72ec72f4116"
-					(reference "#PWR0612")
+					(reference "#PWR0609")
 					(unit 1)
 				)
@@
 		(dnp no)
 		(fields_autoplaced yes)
-		(property "Reference" "#PWR0603"
+		(property "Reference" "#PWR0602"
 			(at 80.01 67.31 0)
 			(effects
@@
 			(project ""
 				(path "/8561283c-f5b3-4542-8880-7f435c3a9f7c/50b8a1dd-352e-4a33-913d-a72ec72f4116"
-					(reference "#PWR0603")
+					(reference "#PWR0602")
 					(unit 1)
 				)
@@
 		(dnp no)
 		(fields_autoplaced yes)
-		(property "Reference" "#PWR0610"
+		(property "Reference" "#PWR0614"
 			(at 173.99 130.81 0)
 			(effects
@@
 			(project "AstroWeather"
 				(path "/8561283c-f5b3-4542-8880-7f435c3a9f7c/50b8a1dd-352e-4a33-913d-a72ec72f4116"
-					(reference "#PWR0610")
+					(reference "#PWR0614")
 					(unit 1)
 				)
@@
 		(dnp no)
 		(fields_autoplaced yes)
-		(property "Reference" "R604"
+		(property "Reference" "R602"
 			(at 176.53 118.1099 0)
 			(effects
@@
 			)
 		)
-		(property "Footprint" ""
+		(property "Footprint" "Resistor_SMD:R_0805_2012Metric"
 			(at 172.212 119.38 90)
 			(effects
@@
 			(project "AstroWeather"
 				(path "/8561283c-f5b3-4542-8880-7f435c3a9f7c/50b8a1dd-352e-4a33-913d-a72ec72f4116"
-					(reference "R604")
+					(reference "R602")
 					(unit 1)
 				)
@@
 		(dnp no)
 		(fields_autoplaced yes)
-		(property "Reference" "#PWR0605"
+		(property "Reference" "#PWR0604"
 			(at 64.77 93.98 0)
 			(effects
@@
 			(project "AstroWeather"
 				(path "/8561283c-f5b3-4542-8880-7f435c3a9f7c/50b8a1dd-352e-4a33-913d-a72ec72f4116"
-					(reference "#PWR0605")
+					(reference "#PWR0604")
 					(unit 1)
 				)
@@
 		(dnp no)
 		(fields_autoplaced yes)
-		(property "Reference" "#PWR0602"
+		(property "Reference" "#PWR0603"
 			(at 80.01 80.01 0)
 			(effects
@@
 			(project "AstroWeather"
 				(path "/8561283c-f5b3-4542-8880-7f435c3a9f7c/50b8a1dd-352e-4a33-913d-a72ec72f4116"
-					(reference "#PWR0602")
+					(reference "#PWR0603")
 					(unit 1)
 				)
@@
 		(dnp no)
 		(fields_autoplaced yes)
-		(property "Reference" "C607"
+		(property "Reference" "C606"
 			(at 195.58 97.7899 0)
 			(effects
@@
 			)
 		)
-		(property "Footprint" ""
+		(property "Footprint" "Capacitor_SMD:C_0805_2012Metric"
 			(at 192.7352 102.87 0)
 			(effects
@@
 			(project "AstroWeather"
 				(path "/8561283c-f5b3-4542-8880-7f435c3a9f7c/50b8a1dd-352e-4a33-913d-a72ec72f4116"
-					(reference "C607")
+					(reference "C606")
 					(unit 1)
 				)
@@
 		(dnp no)
 		(fields_autoplaced yes)
-		(property "Reference" "C605"
+		(property "Reference" "C602"
 			(at 73.66 95.2499 0)
 			(effects
@@
 			)
 		)
-		(property "Footprint" ""
+		(property "Footprint" "Capacitor_SMD:C_0805_2012Metric"
 			(at 68.8848 92.71 0)
 			(effects
@@
 			(project "AstroWeather"
 				(path "/8561283c-f5b3-4542-8880-7f435c3a9f7c/50b8a1dd-352e-4a33-913d-a72ec72f4116"
-					(reference "C605")
+					(reference "C602")
 					(unit 1)
 				)
@@
 		(dnp no)
 		(fields_autoplaced yes)
-		(property "Reference" "C602"
+		(property "Reference" "C601"
 			(at 124.46 86.3599 0)
 			(effects
@@
 			)
 		)
-		(property "Footprint" ""
+		(property "Footprint" "Capacitor_SMD:C_0201_0603Metric"
 			(at 121.6152 91.44 0)
 			(effects
@@
 			(project "AstroWeather"
 				(path "/8561283c-f5b3-4542-8880-7f435c3a9f7c/50b8a1dd-352e-4a33-913d-a72ec72f4116"
-					(reference "C602")
+					(reference "C601")
 					(unit 1)
 				)
@@
 		(dnp no)
 		(fields_autoplaced yes)
-		(property "Reference" "C601"
+		(property "Reference" "C603"
 			(at 85.09 95.2499 0)
 			(effects
@@
 			)
 		)
-		(property "Footprint" ""
+		(property "Footprint" "Capacitor_SMD:C_0603_1608Metric"
 			(at 82.2452 100.33 0)
 			(effects
@@
 			(project ""
 				(path "/8561283c-f5b3-4542-8880-7f435c3a9f7c/50b8a1dd-352e-4a33-913d-a72ec72f4116"
-					(reference "C601")
+					(reference "C603")
 					(unit 1)
 				)
@@
 		(dnp no)
 		(fields_autoplaced yes)
-		(property "Reference" "#PWR0615"
+		(property "Reference" "#PWR0601"
 			(at 219.71 62.23 0)
 			(effects
@@
 			(project "AstroWeather"
 				(path "/8561283c-f5b3-4542-8880-7f435c3a9f7c/50b8a1dd-352e-4a33-913d-a72ec72f4116"
-					(reference "#PWR0615")
+					(reference "#PWR0601")
 					(unit 1)
 				)
@@
 		(dnp no)
 		(fields_autoplaced yes)
-		(property "Reference" "#PWR0601"
+		(property "Reference" "#PWR0608"
 			(at 102.87 109.22 0)
 			(effects
@@
 			(project ""
 				(path "/8561283c-f5b3-4542-8880-7f435c3a9f7c/50b8a1dd-352e-4a33-913d-a72ec72f4116"
-					(reference "#PWR0601")
+					(reference "#PWR0608")
 					(unit 1)
 				)
@@
 		(dnp no)
 		(fields_autoplaced yes)
-		(property "Reference" "C604"
+		(property "Reference" "C605"
 			(at 156.21 97.7899 0)
 			(effects
@@
 			)
 		)
-		(property "Footprint" ""
+		(property "Footprint" "Capacitor_SMD:C_1206_3216Metric"
 			(at 153.3652 102.87 0)
 			(effects
@@
 			(project "AstroWeather"
 				(path "/8561283c-f5b3-4542-8880-7f435c3a9f7c/50b8a1dd-352e-4a33-913d-a72ec72f4116"
-					(reference "C604")
-					(unit 1)
-				)
+					(reference "C605")
+					(unit 1)
+				)

Commit message: KiCad work
Parts:
- C601: footprint Capacitor_SMD:C_0201_0603Metric -> Capacitor_SMD:C_0805_2012Metric
Other:
- note added: "R=20k -> Vout=3.576V R=19.1k -> Vout=3.716V"
Changed lines of the file:
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@@
 	(generator_version "9.0")
 	(paper "A4")
+	(text "R=20k -> Vout=3.576V\nR=19.1k -> Vout=3.716V"
+		(exclude_from_sim no)
+		(at 186.436 122.936 0)
+		(effects
+			(font
+				(size 1.27 1.27)
+			)
+			(justify left top)
+		)
+	)
 	(junction
 		(at 173.99 93.98)
@@
 			)
 		)
-		(property "Footprint" "Capacitor_SMD:C_0201_0603Metric"
+		(property "Footprint" "Capacitor_SMD:C_0805_2012Metric"
 			(at 121.6152 91.44 0)
 			(effects

Commit message: Work
Parts:
- L601: footprint Inductor_SMD:L_7.3x7.3_H4.5 -> Inductor_SMD:L_Wuerth_MAPI-4020
- TP601, TP602: footprint TestPoint:TestPoint_THTPad_D1.5mm_Drill0.7mm -> TestPoint:TestPoint_Pad_D1.5mm

Commit message: KiCad work
Parts:
- C602: value 10u -> 10u/35V
- L601: footprint Inductor_SMD:L_Wuerth_MAPI-4020 -> Inductor_SMD:L_Panasonic_PCC-M0630M
Changed lines of the file:
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@@
 			)
 		)
-		(property "Footprint" "Inductor_SMD:L_Wuerth_MAPI-4020"
+		(property "Footprint" "Inductor_SMD:L_Panasonic_PCC-M0630M"
 			(at 134.62 93.98 0)
 			(effects
@@
 		(on_board yes)
 		(dnp no)
-		(fields_autoplaced yes)
 		(property "Reference" "C602"
 			(at 73.66 95.2499 0)
@@
 			)
 		)
-		(property "Value" "10u"
-			(at 73.66 97.7899 0)
-			(effects
-				(font
+		(property "Value" "10u/35V"
+			(at 70.866 99.568 0)
+			(effects
+				(font
