File: KiCad/PowerSupply.kicad_sch (KiCad schematic)
At the start: 15 parts, among them U601 TPS54302, U602 MCP1825S

Commit message: KiCad finishing touches, gerber
Parts:
- L601: value SRR6038-33u -> SRR6838-33u
Changed lines of the file:
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@@
 			)
 		)
-		(property "Value" "SRR6038-33u"
+		(property "Value" "SRR6838-33u"
 			(at 134.62 91.44 90)
 			(effects
