File: KiCad/PowerSupply.kicad_sch (KiCad schematic)
At the start: 15 parts, among them U601 TPS54302, U602 MCP1825S

Commit message: KiCad work
Other:
- note added: "47p nie mam, u użyłem 67p"
Changed lines of the file:
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@@
 	(generator_version "9.0")
 	(paper "A4")
+	(text "47p nie mam, u użyłem 67p"
+		(exclude_from_sim no)
+		(at 156.21 120.65 0)
+		(effects
+			(font
+				(size 1.27 1.27)
+			)
+		)
+	)
 	(text "R=20k -> Vout=3.576V\nR=19.1k -> Vout=3.716V"
 		(exclude_from_sim no)
