File: KiCad/ST67W611M1.kicad_sch (KiCad schematic)
At the start: 0 parts

Commit message: KiCad work
Parts:
- added U201: ST67W611, symbol myLib:ST67W611M1A6B
Connections:
- new net GND: U201. (UART_TX)

Commit message: KiCad work
Parts:
- added C201, C202: 5p1, symbol Device:C
- added C203, C204, C205: 10u, symbol Device:C
- added C206: 100n, symbol Device:C
- added R201: 33k, symbol Device:R
- added Y201: 32.768k, symbol Device:Crystal_Small
- U201: footprint (none) -> JPComms:ST67W611M1
Connections:
- net GND: now also U201.10 (GND), U201.15 (GND), U201.18 (GND), U201.26 (GND), U201.30 (GND), U201.32 (GND), C201.1, C202.1, C203.1, C204.2, C205.2, C206.1; no longer U201. (UART_TX)
- net ST67_CLK: now also U201.28 (SPI_CLK)
- net ST67_CS: now also U201.24 (SPI_CS)
- net ST67_MISO: now also U201.29 (SPI_MISO)
- net ST67_MOSI: now also U201.27 (SPI_MOSI)
- net ST67_RDY: now also U201.21 (SPI_RDY)
- net ST67_RX: now also U201.23 (UART_RX)
- net ST67_TX: now also U201.22 (UART_TX)
- new net: C201.2, U201.13 (XTAL32K_OUT), Y201.1
- new net: C202.2, U201.14 (XTAL32K_IN), Y201.2
- new net +3.3V: C203.2, C204.1, C205.1, R201.1, U201.16 (VDD33), U201.25 (VDDIO), U201.9 (VDDIO)
- new net BOOT: U201.3 (BOOT)
- new net CHIP_EN: C206.2, R201.2, U201.17 (CHIP_EN)

Commit message: KiCad work
Parts:
- C201: renamed from C203; footprint (none) -> Capacitor_SMD:C_0805_2012Metric
- C202: renamed from C204; footprint (none) -> Capacitor_SMD:C_0805_2012Metric
- C203: renamed from C205; footprint (none) -> Capacitor_SMD:C_0805_2012Metric
- C204: renamed from C201; footprint (none) -> Capacitor_SMD:C_0805_2012Metric
- C205: renamed from C202; footprint (none) -> Capacitor_SMD:C_0805_2012Metric
- C206: footprint (none) -> Capacitor_SMD:C_0201_0603Metric
- R201: footprint (none) -> Resistor_SMD:R_0805_2012Metric
- Y201: footprint (none) -> Crystal:Crystal_SMD_7050-2Pin_7.0x5.0mm

Commit message: Work
Parts:
- C206: footprint Capacitor_SMD:C_0201_0603Metric -> Capacitor_SMD:C_0805_2012Metric
Changed lines of the file:
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@@
 			)
 		)
-		(property "Footprint" "Capacitor_SMD:C_0201_0603Metric"
+		(property "Footprint" "Capacitor_SMD:C_0805_2012Metric"
 			(at 76.5048 86.36 0)
 			(effects

Commit message: KiCad work
Parts:
- removed C204, C205: 5p1, Capacitor_SMD:C_0805_2012Metric, symbol Device:C
- removed Y201: 32.768k, Crystal:Crystal_SMD_7050-2Pin_7.0x5.0mm, symbol Device:Crystal_Small

Commit message: KiCad work
Parts:
- renumbered C206 to C204
Changed lines of the file:
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@@
 		(dnp no)
 		(fields_autoplaced yes)
-		(property "Reference" "#PWR0210"
+		(property "Reference" "#PWR0208"
 			(at 71.12 83.82 0)
 			(effects
@@
 			(project "AstroWeather"
 				(path "/8561283c-f5b3-4542-8880-7f435c3a9f7c/4e5845db-e9e3-4a64-a835-2e404d8331a5"
-					(reference "#PWR0210")
+					(reference "#PWR0208")
 					(unit 1)
 				)
@@
 		(dnp no)
 		(fields_autoplaced yes)
-		(property "Reference" "#PWR0211"
+		(property "Reference" "#PWR0209"
 			(at 102.87 93.98 0)
 			(effects
@@
 			(project "AstroWeather"
 				(path "/8561283c-f5b3-4542-8880-7f435c3a9f7c/4e5845db-e9e3-4a64-a835-2e404d8331a5"
-					(reference "#PWR0211")
+					(reference "#PWR0209")
 					(unit 1)
 				)
@@
 		(on_board yes)
 		(dnp no)
-		(property "Reference" "C206"
+		(property "Reference" "C204"
 			(at 71.374 87.63 0)
 			(effects
@@
 			(project "AstroWeather"
 				(path "/8561283c-f5b3-4542-8880-7f435c3a9f7c/4e5845db-e9e3-4a64-a835-2e404d8331a5"
-					(reference "C206")
+					(reference "C204")
 					(unit 1)
 				)
@@
 		(dnp no)
 		(fields_autoplaced yes)
-		(property "Reference" "#PWR0212"
+		(property "Reference" "#PWR0210"
 			(at 77.47 101.6 0)
 			(effects
@@
 			(project "AstroWeather"
 				(path "/8561283c-f5b3-4542-8880-7f435c3a9f7c/4e5845db-e9e3-4a64-a835-2e404d8331a5"
-					(reference "#PWR0212")
-					(unit 1)
-				)
+					(reference "#PWR0210")
+					(unit 1)
+				)
