File: KiCad/LightSensor.kicad_sch (KiCad schematic)
At the start: 7 parts, among them Q701 IRLML2502

Commit message: KiCad work
Changed lines of the file:
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@@
 		(dnp no)
 		(property "Reference" "R704"
-			(at 101.6 60.706 0)
+			(at 99.822 60.706 0)
 			(effects
 				(font

Commit message: Work
Parts:
- R703: footprint Resistor_THT:R_Axial_DIN0204_L3.6mm_D1.6mm_P1.90mm_Vertical -> OptoDevice:R_LDR_4.9x4.2mm_P2.54mm_Vertical
- TP701: footprint TestPoint:TestPoint_THTPad_D1.5mm_Drill0.7mm -> TestPoint:TestPoint_Pad_D1.5mm
Changed lines of the file:
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@@
 			)
 		)
-		(property "Footprint" "Resistor_THT:R_Axial_DIN0204_L3.6mm_D1.6mm_P1.90mm_Vertical"
+		(property "Footprint" "OptoDevice:R_LDR_4.9x4.2mm_P2.54mm_Vertical"
 			(at 102.87 55.88 90)
 			(effects
@@
 			)
 		)
-		(property "Footprint" "TestPoint:TestPoint_THTPad_D1.5mm_Drill0.7mm"
+		(property "Footprint" "TestPoint:TestPoint_Pad_D1.5mm"
 			(at 121.92 54.61 0)
 			(effects

Commit message: KiCad work
Parts:
- Q701: value IRLML2502 -> Si2374DS
Changed lines of the file:
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@@
 			)
 		)
-		(property "Value" "IRLML2502"
+		(property "Value" "Si2374DS"
 			(at 95.504 81.788 0)
 			(effects
